File: kicad/imucam/nucleo.sch (KiCad schematic (older format))
At the start: 32 parts

Commit message: Cleaned up footprints
Parts:
- C? (x4): footprint (none) -> Capacitor_SMD:C_0402_1005Metric
- C? (x4): footprint (none) -> Capacitor_SMD:C_0603_1608Metric
- J?: footprint (none) -> Connector_PinHeader_2.54mm:PinHeader_2x08_P2.54mm_Vertical
- J?: footprint (none) -> Connector_PinHeader_2.54mm:PinHeader_2x15_P2.54mm_Vertical
- J?: footprint (none) -> Connector_PinHeader_2.54mm:PinHeader_2x10_P2.54mm_Vertical
- J?: footprint (none) -> Connector_PinHeader_2.54mm:PinHeader_2x17_P2.54mm_Vertical
- STM_LED1: renamed from D?; value LED1 -> RED
- STM_LED2: renamed from D?; value LED2 -> RED
- STM_LED3: renamed from D?; value LED3 -> RED
Changed lines of the file:
@@
 F 0 "J?" H 2300 2717 50  0000 C CNN
 F 1 "NUCLEO_CN8" H 2300 2626 50  0000 C CNN
-F 2 "" H 2250 2200 50  0001 C CNN
+F 2 "Connector_PinHeader_2.54mm:PinHeader_2x08_P2.54mm_Vertical" H 2250 2200 50  0001 C CNN
 F 3 "~" H 2250 2200 50  0001 C CNN
 	1    2250 2200
@@
 F 0 "J?" H 2300 4867 50  0000 C CNN
 F 1 "NUCLEO_CN9" H 2300 4776 50  0000 C CNN
-F 2 "" H 2250 3950 50  0001 C CNN
+F 2 "Connector_PinHeader_2.54mm:PinHeader_2x15_P2.54mm_Vertical" H 2250 3950 50  0001 C CNN
 F 3 "~" H 2250 3950 50  0001 C CNN
 	1    2250 3950
@@
 F 0 "J?" H 4500 2917 50  0000 C CNN
 F 1 "NUCLEO_CN7" H 4500 2826 50  0000 C CNN
-F 2 "" H 4450 2300 50  0001 C CNN
+F 2 "Connector_PinHeader_2.54mm:PinHeader_2x10_P2.54mm_Vertical" H 4450 2300 50  0001 C CNN
 F 3 "~" H 4450 2300 50  0001 C CNN
 	1    4450 2300
@@
 F 0 "J?" H 4500 5067 50  0000 C CNN
 F 1 "NUCLEO_CN10" H 4500 4976 50  0000 C CNN
-F 2 "" H 4450 4050 50  0001 C CNN
+F 2 "Connector_PinHeader_2.54mm:PinHeader_2x17_P2.54mm_Vertical" H 4450 4050 50  0001 C CNN
 F 3 "~" H 4450 4050 50  0001 C CNN
 	1    4450 4050
@@
 F 0 "C?" H 7065 1896 50  0000 L CNN
 F 1 "100nF" H 7065 1805 50  0000 L CNN
-F 2 "" H 6988 1700 50  0001 C CNN
+F 2 "Capacitor_SMD:C_0402_1005Metric" H 6988 1700 50  0001 C CNN
 F 3 "~" H 6950 1850 50  0001 C CNN
 	1    6950 1850
@@
 F 0 "C?" V 8650 1550 50  0000 C CNN
 F 1 "100nF" V 8750 1550 50  0000 C CNN
-F 2 "" H 8538 1400 50  0001 C CNN
+F 2 "Capacitor_SMD:C_0402_1005Metric" H 8538 1400 50  0001 C CNN
 F 3 "~" H 8500 1550 50  0001 C CNN
 	1    8500 1550
@@
 F 0 "C?" H 9715 1896 50  0000 L CNN
 F 1 "22uF" H 9715 1805 50  0000 L CNN
-F 2 "" H 9638 1700 50  0001 C CNN
+F 2 "Capacitor_SMD:C_0603_1608Metric" H 9638 1700 50  0001 C CNN
 F 3 "~" H 9600 1850 50  0001 C CNN
 	1    9600 1850
@@
 F 0 "C?" H 6615 1896 50  0000 L CNN
 F 1 "10uF" H 6615 1805 50  0000 L CNN
-F 2 "" H 6538 1700 50  0001 C CNN
+F 2 "Capacitor_SMD:C_0603_1608Metric" H 6538 1700 50  0001 C CNN
 F 3 "~" H 6500 1850 50  0001 C CNN
 	1    6500 1850
@@
 F 0 "C?" H 7065 3396 50  0000 L CNN
 F 1 "100nF" H 7065 3305 50  0000 L CNN
-F 2 "" H 6988 3200 50  0001 C CNN
+F 2 "Capacitor_SMD:C_0402_1005Metric" H 6988 3200 50  0001 C CNN
 F 3 "~" H 6950 3350 50  0001 C CNN
 	1    6950 3350
@@
 F 0 "C?" V 8650 3050 50  0000 C CNN
 F 1 "100nF" V 8750 3050 50  0000 C CNN
-F 2 "" H 8538 2900 50  0001 C CNN
+F 2 "Capacitor_SMD:C_0402_1005Metric" H 8538 2900 50  0001 C CNN
 F 3 "~" H 8500 3050 50  0001 C CNN
 	1    8500 3050
@@
 F 0 "C?" H 9715 3396 50  0000 L CNN
 F 1 "22uF" H 9715 3305 50  0000 L CNN
-F 2 "" H 9638 3200 50  0001 C CNN
+F 2 "Capacitor_SMD:C_0603_1608Metric" H 9638 3200 50  0001 C CNN
 F 3 "~" H 9600 3350 50  0001 C CNN
 	1    9600 3350
@@
 F 0 "C?" H 6615 3396 50  0000 L CNN
 F 1 "10uF" H 6615 3305 50  0000 L CNN
-F 2 "" H 6538 3200 50  0001 C CNN
+F 2 "Capacitor_SMD:C_0603_1608Metric" H 6538 3200 50  0001 C CNN
 F 3 "~" H 6500 3350 50  0001 C CNN
 	1    6500 3350
@@
 P 3800 6400
 AR Path="/6108B368/61E31E2A" Ref="D?"  Part="1"
-AR Path="/617746AB/61E31E2A" Ref="D?"  Part="1"
-F 0 "D?" V 3839 6282 50  0000 R CNN
-F 1 "LED1" V 3748 6282 50  0000 R CNN
+AR Path="/617746AB/61E31E2A" Ref="STM_LED1"  Part="1"
+F 0 "STM_LED1" V 3900 6800 50  0000 R CNN
+F 1 "RED" V 3748 6282 50  0001 R CNN
 F 2 "LED_SMD:LED_0805_2012Metric" H 3800 6400 50  0001 C CNN
 F 3 "~" H 3800 6400 50  0001 C CNN
@@
 L Device:LED D?
 U 1 1 61E3D14D
-P 4200 6400
+P 4300 6400
 AR Path="/6108B368/61E3D14D" Ref="D?"  Part="1"
-AR Path="/617746AB/61E3D14D" Ref="D?"  Part="1"
-F 0 "D?" V 4239 6282 50  0000 R CNN
-F 1 "LED2" V 4148 6282 50  0000 R CNN
-F 2 "LED_SMD:LED_0805_2012Metric" H 4200 6400 50  0001 C CNN
-F 3 "~" H 4200 6400 50  0001 C CNN
-	1    4200 6400
+AR Path="/617746AB/61E3D14D" Ref="STM_LED2"  Part="1"
+F 0 "STM_LED2" V 4400 6800 50  0000 R CNN
+F 1 "RED" V 4248 6282 50  0001 R CNN
+F 2 "LED_SMD:LED_0805_2012Metric" H 4300 6400 50  0001 C CNN
+F 3 "~" H 4300 6400 50  0001 C CNN
+	1    4300 6400
 	0    -1   -1   0
 $EndComp
@@
 L Device:R R?
 U 1 1 61E3D153
-P 4200 6100
+P 4300 6100
 AR Path="/6108B368/61E3D153" Ref="R?"  Part="1"
 AR Path="/617746AB/61E3D153" Ref="R?"  Part="1"
-F 0 "R?" H 4270 6146 50  0000 L CNN
-F 1 "1k" H 4270 6055 50  0000 L CNN
-F 2 "Resistor_SMD:R_0402_1005Metric" V 4130 6100 50  0001 C CNN
-F 3 "~" H 4200 6100 50  0001 C CNN
-	1    4200 6100
+F 0 "R?" H 4370 6146 50  0000 L CNN
+F 1 "1k" H 4370 6055 50  0000 L CNN
+F 2 "Resistor_SMD:R_0402_1005Metric" V 4230 6100 50  0001 C CNN
+F 3 "~" H 4300 6100 50  0001 C CNN
+	1    4300 6100
 	1    0    0    -1
 $EndComp
@@
 L Device:LED D?
 U 1 1 61E42BC7
-P 4600 6400
+P 4800 6400
 AR Path="/6108B368/61E42BC7" Ref="D?"  Part="1"
-AR Path="/617746AB/61E42BC7" Ref="D?"  Part="1"
-F 0 "D?" V 4639 6282 50  0000 R CNN
-F 1 "LED3" V 4548 6282 50  0000 R CNN
-F 2 "LED_SMD:LED_0805_2012Metric" H 4600 6400 50  0001 C CNN
-F 3 "~" H 4600 6400 50  0001 C CNN
-	1    4600 6400
+AR Path="/617746AB/61E42BC7" Ref="STM_LED3"  Part="1"
+F 0 "STM_LED3" V 4900 6800 50  0000 R CNN
+F 1 "RED" V 4748 6282 50  0001 R CNN
+F 2 "LED_SMD:LED_0805_2012Metric" H 4800 6400 50  0001 C CNN
+F 3 "~" H 4800 6400 50  0001 C CNN
+	1    4800 6400
 	0    -1   -1   0
 $EndComp
@@
 L Device:R R?
 U 1 1 61E42BCD
-P 4600 6100
+P 4800 6100
 AR Path="/6108B368/61E42BCD" Ref="R?"  Part="1"
 AR Path="/617746AB/61E42BCD" Ref="R?"  Part="1"
-F 0 "R?" H 4670 6146 50  0000 L CNN
-F 1 "1k" H 4670 6055 50  0000 L CNN
-F 2 "Resistor_SMD:R_0402_1005Metric" V 4530 6100 50  0001 C CNN
-F 3 "~" H 4600 6100 50  0001 C CNN
-	1    4600 6100
-	1    0    0    -1
-$EndComp
-Wire Wire Line
-	3800 6600 4200 6600
-Wire Wire Line
-	4600 6600 4600 6550
-Wire Wire Line
-	4200 6550 4200 6600
-Connection ~ 4200 6600
-Wire Wire Line
-	4200 6600 4600 6600
+F 0 "R?" H 4870 6146 50  0000 L CNN
+F 1 "1k" H 4870 6055 50  0000 L CNN
+F 2 "Resistor_SMD:R_0402_1005Metric" V 4730 6100 50  0001 C CNN
+F 3 "~" H 4800 6100 50  0001 C CNN
+	1    4800 6100
+	1    0    0    -1
+$EndComp
+Wire Wire Line
+	4800 6600 4800 6550
+Wire Wire Line
+	4300 6550 4300 6600
 Wire Wire Line
 	3800 6550 3800 6600
@@
 	1    0    0    -1
 $EndComp
-Connection ~ 3800 6600
 Wire Wire Line
 	3800 5950 3800 5900
@@
 LED1
 Wire Wire Line
-	4200 5950 4200 5900
-Wire Wire Line
-	4200 5900 3950 5900
-Text Label 3950 5900 0    50   ~ 0
+	4300 5950 4300 5900
+Wire Wire Line
+	4300 5900 4050 5900
+Text Label 4050 5900 0    50   ~ 0
 LED2
 Wire Wire Line
-	4600 5950 4600 5900
-Wire Wire Line
-	4600 5900 4350 5900
-Text Label 4350 5900 0    50   ~ 0
+	4800 5950 4800 5900
+Wire Wire Line
+	4800 5900 4550 5900
+Text Label 4550 5900 0    50   ~ 0
 LED3
 Wire Wire Line
@@
 Wire Wire Line
 	2550 4550 2650 4550
+Connection ~ 3800 6600
+Wire Wire Line
+	3800 6600 4300 6600
+Wire Wire Line
+	4300 6600 4800 6600
+Connection ~ 4300 6600
 $EndSCHEMATC

Commit message: All components have footprints!
Parts:
- L? (x2): footprint (none) -> Inductor_SMD:L_Coilcraft_XxL4020
Changed lines of the file:
@@
 F 0 "L?" V 8719 1450 50  0000 C CNN
 F 1 "3.3uH" V 8810 1450 50  0000 C CNN
-F 2 "" H 8900 1450 50  0001 C CNN
+F 2 "Inductor_SMD:L_Coilcraft_XxL4020" H 8900 1450 50  0001 C CNN
 F 3 "https://www.coilcraft.com/getmedia/50632d43-da1b-4cdb-8ab4-3029cab51df3/xfl4020.pdf" H 8900 1450 50  0001 C CNN
 	1    8900 1450
@@
 F 0 "L?" V 8719 2950 50  0000 C CNN
 F 1 "3.3uH" V 8810 2950 50  0000 C CNN
-F 2 "" H 8900 2950 50  0001 C CNN
+F 2 "Inductor_SMD:L_Coilcraft_XxL4020" H 8900 2950 50  0001 C CNN
 F 3 "https://www.coilcraft.com/getmedia/50632d43-da1b-4cdb-8ab4-3029cab51df3/xfl4020.pdf" H 8900 2950 50  0001 C CNN
 	1    8900 2950

Commit message: Annotated schematic
Parts:
- gave numbers to parts that had none: 29

Commit message: Lots of schematic work
Parts:
- added R23, R24, R25, R28, R29, R30: 10k, Resistor_SMD:R_0402_1005Metric, symbol Device:R
- renumbered R23 to R26, R24 to R27, R25 to R31, R26 to R32, R27 to R33, R28 to R34, R29 to R35
Connections:
- net labels added: IMU_CS_3V3, IMU_SCK_3V3, IMU_SI_3V3
- wire segments 134 -> 140

Commit message: Added 3.3v power LED
Parts:
- added PWR1: RED, LED_SMD:LED_0805_2012Metric, symbol Device:LED
- added R45: 1k, Resistor_SMD:R_0402_1005Metric, symbol Device:R
Connections:
- wire segments 140 -> 143
Changed lines of the file:
@@
+	1    0    0    -1
+$EndComp
+$Comp
+L Device:LED STM_LED?
+U 1 1 60F9FF97
+P 5300 6400
+AR Path="/6108B368/60F9FF97" Ref="STM_LED?"  Part="1"
+AR Path="/617746AB/60F9FF97" Ref="PWR1"  Part="1"
+F 0 "PWR1" V 5400 6600 50  0000 R CNN
+F 1 "RED" V 5248 6282 50  0001 R CNN
+F 2 "LED_SMD:LED_0805_2012Metric" H 5300 6400 50  0001 C CNN
+F 3 "~" H 5300 6400 50  0001 C CNN
+	1    5300 6400
+	0    -1   -1   0
+$EndComp
+$Comp
+L Device:R R?
+U 1 1 60F9FF9D
+P 5300 6100
+AR Path="/6108B368/60F9FF9D" Ref="R?"  Part="1"
+AR Path="/617746AB/60F9FF9D" Ref="R45"  Part="1"
+F 0 "R45" H 5370 6146 50  0000 L CNN
+F 1 "1k" H 5370 6055 50  0000 L CNN
+F 2 "Resistor_SMD:R_0402_1005Metric" V 5230 6100 50  0001 C CNN
+F 3 "~" H 5300 6100 50  0001 C CNN
+	1    5300 6100
+	1    0    0    -1
+$EndComp
+Wire Wire Line
+	5300 6600 5300 6550
+Wire Wire Line
+	5300 5950 5300 5900
+Wire Wire Line
+	4800 6600 5300 6600
+Connection ~ 4800 6600
+$Comp
+L power:+3.3V #PWR091
+U 1 1 60FB7AC2
+P 5300 5900
+F 0 "#PWR091" H 5300 5750 50  0001 C CNN
+F 1 "+3.3V" H 5315 6073 50  0000 C CNN
+F 2 "" H 5300 5900 50  0001 C CNN
+F 3 "" H 5300 5900 50  0001 C CNN
+	1    5300 5900
 	1    0    0    -1
 $EndComp

Commit message: Switched FSYNC to use TRIGGER, lots of PCB work
Parts:
- added R32, R37: 10k, Resistor_SMD:R_0402_1005Metric, symbol Device:R
- renumbered J4 to J3, J5 to J4, J6 to J5, J7 to J6, R19 to R18, R20 to R19, R21 to R20, R22 to R21, R23 to R22, R24 to R23, R25 to R24, R26 to R25, R27 to R26, R28 to R27, R29 to R28, R30 to R29, R31 to R30, R32 to R31, R45 to R36, PWR1 to STM_LED4
Connections:
- net labels added: CAM_TRIGGER_3V3, IMU_FSYNC_EN, IMU_FSYNC_SEL
- wire segments 143 -> 148

Commit message: More PCB work, began current sense
Parts:
- added R?: R_US, symbol Device:R_US
- added U?: INA219AxDCN, Package_TO_SOT_SMD:SOT-23-8, symbol Analog_ADC:INA219AxDCN
Connections:
- net labels added: 5V_IN
- wire segments 148 -> 154
Changed lines of the file:
@@
 	1    0    0    -1
 $EndComp
-Wire Wire Line
-	2050 2300 2000 2300
 $Comp
 L power:GND #PWR067
@@
 L power:+5V #PWR066
 U 1 1 61ABC972
-P 2000 2300
-F 0 "#PWR066" H 2000 2150 50  0001 C CNN
-F 1 "+5V" V 2015 2428 50  0000 L CNN
-F 2 "" H 2000 2300 50  0001 C CNN
-F 3 "" H 2000 2300 50  0001 C CNN
-	1    2000 2300
-	0    -1   -1   0
+P 1700 5550
+F 0 "#PWR066" H 1700 5400 50  0001 C CNN
+F 1 "+5V" V 1715 5678 50  0000 L CNN
+F 2 "" H 1700 5550 50  0001 C CNN
+F 3 "" H 1700 5550 50  0001 C CNN
+	1    1700 5550
+	0    1    1    0
 $EndComp
 $Comp
@@
 	1    0    0    -1
 $EndComp
+$Comp
+L Analog_ADC:INA219AxDCN U?
+U 1 1 61570FAE
+P 2150 6300
+F 0 "U?" H 1900 6650 50  0000 C CNN
+F 1 "INA219AxDCN" H 2450 6650 50  0000 C CNN
+F 2 "Package_TO_SOT_SMD:SOT-23-8" H 2800 5950 50  0001 C CNN
+F 3 "http://www.ti.com/lit/ds/symlink/ina219.pdf" H 2500 6200 50  0001 C CNN
+	1    2150 6300
+	1    0    0    -1
+$EndComp
+Text Label 1700 2300 0    50   ~ 0
+5V_IN
+Wire Wire Line
+	2050 2300 1700 2300
+$Comp
+L Device:R_US R?
+U 1 1 6158B83B
+P 1500 5550
+F 0 "R?" V 1295 5550 50  0000 C CNN
+F 1 "R_US" V 1386 5550 50  0000 C CNN
+F 2 "" V 1540 5540 50  0001 C CNN
+F 3 "~" H 1500 5550 50  0001 C CNN
+	1    1500 5550
+	0    1    1    0
+$EndComp
+Wire Wire Line
+	1650 5550 1700 5550
+Text Label 1050 5550 0    50   ~ 0
+5V_IN
+Wire Wire Line
+	1750 6200 1350 6200
+Wire Wire Line
+	1350 6200 1350 5550
+Connection ~ 1350 5550
+Wire Wire Line
+	1350 5550 1050 5550
+Wire Wire Line
+	1650 5550 1650 6400
+Wire Wire Line
+	1650 6400 1750 6400
+Connection ~ 1650 5550
+$Comp
+L power:GND #PWR?
+U 1 1 615B9113
+P 2150 6700
+F 0 "#PWR?" H 2150 6450 50  0001 C CNN
+F 1 "GND" H 2155 6527 50  0000 C CNN
+F 2 "" H 2150 6700 50  0001 C CNN
+F 3 "" H 2150 6700 50  0001 C CNN
+	1    2150 6700
+	1    0    0    -1
+$EndComp
+$Comp
+L power:+3.3V #PWR?
+U 1 1 615B9C16
+P 2150 5900
+F 0 "#PWR?" H 2150 5750 50  0001 C CNN
+F 1 "+3.3V" H 2165 6073 50  0000 C CNN
+F 2 "" H 2150 5900 50  0001 C CNN
+F 3 "" H 2150 5900 50  0001 C CNN
+	1    2150 5900
+	1    0    0    -1
+$EndComp

Commit message: Slightly more progress on current measurement
Parts:
- added C57: 100nF, Capacitor_SMD:C_0402_1005Metric, symbol Device:C
- R18: renamed from R?; value R_US -> .05; footprint (none) -> Resistor_SMD:R_0805_2012Metric
- gave numbers to parts that had none: 1
- renumbered C62 to C59, C59 to C60, C63 to C61, C57 to C62, C61 to C63, C60 to C64, C64 to C65, J5 to J4, J4 to J5, R33 to R19, R34 to R20, R35 to R21, R36 to R22, R25 to R23, R30 to R24, R26 to R25, R31 to R26, R22 to R27, R27 to R28, R32 to R29, R37 to R30, R18 to R31, R19 to R32, R20 to R33, R21 to R34, R23 to R35, R28 to R36, R24 to R37, R29 to R38, U7 to U8, U8 to U9
Connections:
- wire segments 154 -> 165
