File: kicad/imucam/nucleo.sch (KiCad schematic (older format))
At the start: 45 parts, among them J3 NUCLEO_CN8, J4 NUCLEO_CN9, J5 NUCLEO_CN7, J6 NUCLEO_CN10, Q5 BSS214NW, Q6 BSS214NW, U7 INA219AxDCN, U8 TPS562200, U9 TPS562200

Commit message: Turns out, we need level translators
Parts:
- removed Q5, Q6: BSS214NW, Package_TO_SOT_SMD:SOT-323_SC-70, symbol Transistor_FET:BSS214NW
- removed R23, R24, R25, R26: 4.7k, Resistor_SMD:R_0402_1005Metric, symbol Device:R
- removed R27, R28, R29, R30, R35, R36, R37, R38: 10k, Resistor_SMD:R_0402_1005Metric, symbol Device:R
- added C55, C56, C57, C58, C59, C60: 100nF, Capacitor_SMD:C_0402_1005Metric, symbol Device:C
- added R17, R18, R19, R20: 4.7k, Resistor_SMD:R_0402_1005Metric, symbol Device:R
- added U11, U7, U8: NTS0104PW, Package_SO:TSSOP-14_4.4x5mm_P0.65mm, symbol Logic_LevelTranslator:TXB0104PW
- R26: renamed from R19; value 1k -> 100
- R27: renamed from R20; value 1k -> 100
- R28: renamed from R21; value 1k -> 100
- R29: renamed from R22; value 1k -> 100
- renumbered C63 to C61, C59 to C63, C61 to C64, C58 to C66, C60 to C67, C64 to C68, C57 to C69, J5 to J4, J4 to J5, L2 to L1, L1 to L2, STM_LED4 to PWR1, R33 to R21, R31 to R22, R34 to R23, R32 to R24, R18 to R25, U8 to U10, U7 to U12
Connections:
- net labels added: +3V3, CAM_FLASH_3V3, CAM_RESET_BAR_3V3, CAM_SHUTTER, CAM_SHUTTER_3V3, IMU_INT_3V3, IMU_SO_3V3
- net labels removed: +3.3V, IMU_FSYNC_EN, IMU_FSYNC_SEL
- wire segments 165 -> 204
Other:
- note removed: "Open Collector"

Commit message: WIP of remapping nucleo pinout for pcb routing
Parts:
- removed C55, C56, C57, C58, C59, C60: 100nF, Capacitor_SMD:C_0402_1005Metric, symbol Device:C
- removed R17, R18, R19, R20: 4.7k, Resistor_SMD:R_0402_1005Metric, symbol Device:R
- removed U11, U7, U8: NTS0104PW, Package_SO:TSSOP-14_4.4x5mm_P0.65mm, symbol Logic_LevelTranslator:TXB0104PW
- added C62, C65: 100nF, Capacitor_SMD:C_0402_1005Metric, symbol Device:C
- added R25, R26, R29, R30: 4.7k, Resistor_SMD:R_0402_1005Metric, symbol Device:R
- added U10: NTS0308E, Package_SO:TSSOP-20_4.4x6.5mm_P0.65mm, symbol imucam:NTS0308E
- renumbered C63 to C55, C64 to C56, C61 to C57, C69 to C58, C65 to C59, C66 to C60, C67 to C61, C62 to C63, C68 to C64, J5 to J4, J4 to J5, R25 to R18, R21 to R19, R23 to R20, R26 to R21, R27 to R22, R28 to R23, R29 to R24, R22 to R27, R24 to R28, U9 to U7, U12 to U8, U10 to U9
Connections:
- net labels removed: CAM_FLASH, CAM_FLASH_3V3, CAM_RESET_BAR_3V3, CAM_SHUTTER, CAM_SHUTTER_3V3
- wire segments 204 -> 186
Other:
- note added: "EXTI3"
- note added: "Open Drain"
- note removed: "EXTI5"
- note removed: "EXTI6"

Commit message: Ready to begin routing differential pairs
Connections:
- wire segments 186 -> 172
- no-connect marks 0 -> 62
Other:
- note removed: "EXTI7"

Commit message: More routing
Connections:
- no-connect marks 62 -> 61
Changed lines of the file:
@@
 Text Notes 4750 1750 0    50   ~ 0
 EXTI15\n
+Text GLabel 3500 3350 0    50   Output ~ 0
+HDMI_OE
+Text GLabel 3500 3150 0    50   Input ~ 0
+HDMI_HPD
+Text GLabel 3500 2950 0    50   Output ~ 0
+HDMI_EQ1
 Text GLabel 3500 2850 0    50   Output ~ 0
-HDMI_OE
-Text GLabel 3500 3250 0    50   Input ~ 0
-HDMI_HPD
-Text GLabel 3500 3350 0    50   Output ~ 0
-HDMI_EQ1
-Text GLabel 3500 3150 0    50   Output ~ 0
 HDMI_EQ0
 Text GLabel 4150 2350 2    50   Output ~ 0
@@
 Text Label 5000 6600 0    50   ~ 0
 LED3
-Text GLabel 3500 2950 0    50   Output ~ 0
+Text GLabel 3500 3250 0    50   Output ~ 0
 HDMI_DDC_EN
 Connection ~ 4250 7300
@@
 Text Label 8600 2200 0    50   ~ 0
 IMU_INT_3V3
-Text Label 8600 2600 0    50   ~ 0
+Text Label 8600 2300 0    50   ~ 0
 IMU_SI_3V3
 Text Label 2000 3250 0    50   ~ 0
@@
 Text Label 2000 3050 0    50   ~ 0
 IMU_SO_3V3
+Text GLabel 6950 2100 0    50   BiDi ~ 0
+SCL_1V8
+Text GLabel 9350 2100 2    50   BiDi ~ 0
+SCL_3V3
+Text GLabel 9350 2000 2    50   BiDi ~ 0
+SDA_3V3
 Text GLabel 6950 2000 0    50   BiDi ~ 0
-SCL_1V8
-Text GLabel 9350 2000 2    50   BiDi ~ 0
-SCL_3V3
-Text GLabel 9350 2100 2    50   BiDi ~ 0
-SDA_3V3
-Text GLabel 6900 2100 0    50   BiDi ~ 0
 SDA_1V8
 Text GLabel 7650 2200 0    50   Input ~ 0
 IMU_INT
+Text GLabel 7650 2300 0    50   Output ~ 0
+IMU_SI
+Text Label 8600 2400 0    50   ~ 0
+IMU_SO_3V3
 Text GLabel 7650 2600 0    50   Output ~ 0
-IMU_SI
+IMU_SCK
+Text GLabel 7650 2500 0    50   Output ~ 0
+IMU_CS
+Wire Wire Line
+	7700 2300 7650 2300
+Wire Wire Line
+	7700 2400 7650 2400
+Text GLabel 7650 2400 0    50   Input ~ 0
+IMU_SO
+Wire Wire Line
+	7700 2500 7650 2500
+Text Label 8600 2600 0    50   ~ 0
+IMU_SCK_3V3
 Text Label 8600 2500 0    50   ~ 0
-IMU_SO_3V3
-Text GLabel 7650 2300 0    50   Output ~ 0
-IMU_SCK
-Text GLabel 7650 2400 0    50   Output ~ 0
-IMU_CS
-Wire Wire Line
-	7700 2300 7650 2300
-Wire Wire Line
-	7700 2400 7650 2400
-Text GLabel 7650 2500 0    50   Input ~ 0
-IMU_SO
-Wire Wire Line
-	7700 2500 7650 2500
-Text Label 8600 2300 0    50   ~ 0
-IMU_SCK_3V3
-Text Label 8600 2400 0    50   ~ 0
 IMU_CS_3V3
 Text GLabel 4150 2250 2    50   Output ~ 0
@@
 	8550 2200 9300 2200
 Wire Wire Line
+	8550 2600 9300 2600
+Wire Wire Line
+	8550 2500 9300 2500
+Wire Wire Line
+	8550 2400 9300 2400
+Wire Wire Line
 	8550 2300 9300 2300
-Wire Wire Line
-	8550 2400 9300 2400
-Wire Wire Line
-	8550 2500 9300 2500
-Wire Wire Line
-	8550 2600 9300 2600
 Wire Wire Line
 	8550 2700 9300 2700
@@
 	6950 2000 7550 2000
 Wire Wire Line
-	6900 2100 7200 2100
+	6950 2100 7200 2100
 Wire Wire Line
 	7550 2000 7550 1800
@@
 Wire Wire Line
 	1900 3250 2500 3250
-Text Notes 2600 3250 0    50   ~ 0
+Text Notes 2550 3250 0    50   ~ 0
 EXTI3
 Wire Wire Line
@@
 NoConn ~ 3600 3650
 NoConn ~ 3600 3450
-NoConn ~ 3600 2750
 NoConn ~ 3600 2650
 NoConn ~ 3600 2550
