File: kicad/imucam/cam.sch (KiCad schematic (older format))
At the start: 20 parts

Commit message: All components have footprints!
Parts:
- removed J?: EXTCAM, symbol Connector_Generic:Conn_01x22
- added J?: EXTCAM, imucam:Molex_545482271, symbol imucam:54548-2271
- U?: footprint (none) -> imucam:CLCC48
Changed lines of the file:
@@
 F 0 "U?" H 5300 3550 50  0000 C CNN
 F 1 "AR0330CM1C00" H 6600 3550 50  0000 C CNN
-F 2 "" H 6200 700 50  0001 C CNN
+F 2 "imucam:CLCC48" H 6200 700 50  0001 C CNN
 F 3 "" H 6450 2050 50  0001 C CNN
 	1    6050 2400
@@
 	7750 3100 8000 3100
 $Comp
-L Connector_Generic:Conn_01x22 J?
-U 1 1 615777DB
-P 4550 5550
-AR Path="/6108B368/615777DB" Ref="J?"  Part="1"
-AR Path="/6136B1E7/615777DB" Ref="J?"  Part="1"
-F 0 "J?" H 4630 5542 50  0000 L CNN
-F 1 "EXTCAM" H 4630 5451 50  0000 L CNN
-F 2 "" H 4550 5550 50  0001 C CNN
-F 3 "~" H 4550 5550 50  0001 C CNN
-	1    4550 5550
-	1    0    0    -1
-$EndComp
-$Comp
 L power:GND #PWR?
 U 1 1 615777E1
@@
 Text GLabel 4150 5950 0    50   Output ~ 0
 EXTCAM_D3_P
+$Comp
+L imucam:54548-2271 J?
+U 1 1 60CE4657
+P 4550 4450
+F 0 "J?" H 4630 3346 50  0000 L CNN
+F 1 "EXTCAM" H 4630 3255 50  0000 L CNN
+F 2 "imucam:Molex_545482271" H 4550 4450 50  0001 C CNN
+F 3 "" H 4550 4450 50  0001 C CNN
+	1    4550 4450
+	1    0    0    -1
+$EndComp
 $EndSCHEMATC

Commit message: Annotated schematic
Parts:
- gave numbers to parts that had none: 20
Changed lines of the file:
@@
 $EndDescr
 $Comp
-L imucam:AR0330CM1C00 U?
+L imucam:AR0330CM1C00 U5
 U 1 1 6136CF1D
 P 6050 2400
-F 0 "U?" H 5300 3550 50  0000 C CNN
+F 0 "U5" H 5300 3550 50  0000 C CNN
 F 1 "AR0330CM1C00" H 6600 3550 50  0000 C CNN
 F 2 "imucam:CLCC48" H 6200 700 50  0001 C CNN
@@
 $EndComp
 $Comp
-L power:GND #PWR?
+L power:GND #PWR0145
 U 1 1 61370FCE
 P 6050 3650
-F 0 "#PWR?" H 6050 3400 50  0001 C CNN
+F 0 "#PWR0145" H 6050 3400 50  0001 C CNN
 F 1 "GND" H 6055 3477 50  0000 C CNN
 F 2 "" H 6050 3650 50  0001 C CNN
@@
 	6350 3600 6350 3650
 $Comp
-L Device:C C?
+L Device:C C51
 U 1 1 61372F35
 P 8900 2200
-F 0 "C?" H 9015 2246 50  0000 L CNN
+F 0 "C51" H 9015 2246 50  0000 L CNN
 F 1 "1uF" H 9015 2155 50  0000 L CNN
 F 2 "Capacitor_SMD:C_0402_1005Metric" H 8938 2050 50  0001 C CNN
@@
 $EndComp
 $Comp
-L Device:C C?
+L Device:C C49
 U 1 1 613752DC
 P 8000 2200
-F 0 "C?" H 8115 2246 50  0000 L CNN
+F 0 "C49" H 8115 2246 50  0000 L CNN
 F 1 "100nF" H 8115 2155 50  0000 L CNN
 F 2 "Capacitor_SMD:C_0402_1005Metric" H 8038 2050 50  0001 C CNN
@@
 	7000 2100 7050 2100
 $Comp
-L power:+2V8 #PWR?
+L power:+2V8 #PWR0146
 U 1 1 61379194
 P 7200 2050
-F 0 "#PWR?" H 7200 1900 50  0001 C CNN
+F 0 "#PWR0146" H 7200 1900 50  0001 C CNN
 F 1 "+2V8" H 7215 2223 50  0000 C CNN
 F 2 "" H 7200 2050 50  0001 C CNN
@@
 $EndComp
 $Comp
-L Device:C C?
+L Device:C C50
 U 1 1 61387529
 P 8450 2200
-F 0 "C?" H 8565 2246 50  0000 L CNN
+F 0 "C50" H 8565 2246 50  0000 L CNN
 F 1 "1uF" H 8565 2155 50  0000 L CNN
 F 2 "Capacitor_SMD:C_0402_1005Metric" H 8488 2050 50  0001 C CNN
@@
 $EndComp
 $Comp
-L Device:C C?
+L Device:C C48
 U 1 1 6138752F
 P 7550 2200
-F 0 "C?" H 7665 2246 50  0000 L CNN
+F 0 "C48" H 7665 2246 50  0000 L CNN
 F 1 "100nF" H 7665 2155 50  0000 L CNN
 F 2 "Capacitor_SMD:C_0402_1005Metric" H 7588 2050 50  0001 C CNN
@@
 	7050 1900 7050 1800
 $Comp
-L power:+1V8 #PWR?
+L power:+1V8 #PWR0147
 U 1 1 61397BEE
 P 7200 950
-F 0 "#PWR?" H 7200 800 50  0001 C CNN
+F 0 "#PWR0147" H 7200 800 50  0001 C CNN
 F 1 "+1V8" H 7215 1123 50  0000 C CNN
 F 2 "" H 7200 950 50  0001 C CNN
@@
 Connection ~ 7550 2050
 $Comp
-L Device:C C?
+L Device:C C43
 U 1 1 613A452F
 P 7550 1650
-F 0 "C?" H 7665 1696 50  0000 L CNN
+F 0 "C43" H 7665 1696 50  0000 L CNN
 F 1 "100nF" H 7665 1605 50  0000 L CNN
 F 2 "Capacitor_SMD:C_0402_1005Metric" H 7588 1500 50  0001 C CNN
@@
 $EndComp
 $Comp
-L Device:C C?
+L Device:C C44
 U 1 1 613A4CD0
 P 8000 1650
-F 0 "C?" H 8115 1696 50  0000 L CNN
+F 0 "C44" H 8115 1696 50  0000 L CNN
 F 1 "100nF" H 8115 1605 50  0000 L CNN
 F 2 "Capacitor_SMD:C_0402_1005Metric" H 8038 1500 50  0001 C CNN
@@
 $EndComp
 $Comp
-L Device:C C?
+L Device:C C45
 U 1 1 613A4F84
 P 8450 1650
-F 0 "C?" H 8565 1696 50  0000 L CNN
+F 0 "C45" H 8565 1696 50  0000 L CNN
 F 1 "100nF" H 8565 1605 50  0000 L CNN
 F 2 "Capacitor_SMD:C_0402_1005Metric" H 8488 1500 50  0001 C CNN
@@
 $EndComp
 $Comp
-L Device:C C?
+L Device:C C46
 U 1 1 613A54C1
 P 8900 1650
-F 0 "C?" H 9015 1696 50  0000 L CNN
+F 0 "C46" H 9015 1696 50  0000 L CNN
 F 1 "100nF" H 9015 1605 50  0000 L CNN
 F 2 "Capacitor_SMD:C_0402_1005Metric" H 8938 1500 50  0001 C CNN
@@
 	8450 2050 8900 2050
 $Comp
-L Device:C C?
+L Device:C C47
 U 1 1 613A733B
 P 9350 1650
-F 0 "C?" H 9465 1696 50  0000 L CNN
+F 0 "C47" H 9465 1696 50  0000 L CNN
 F 1 "100nF" H 9465 1605 50  0000 L CNN
 F 2 "Capacitor_SMD:C_0402_1005Metric" H 9388 1500 50  0001 C CNN
@@
 	8900 1800 8450 1800
 $Comp
-L power:GND #PWR?
+L power:GND #PWR0148
 U 1 1 613A900D
 P 8900 1800
-F 0 "#PWR?" H 8900 1550 50  0001 C CNN
+F 0 "#PWR0148" H 8900 1550 50  0001 C CNN
 F 1 "GND" H 8905 1627 50  0000 C CNN
 F 2 "" H 8900 1800 50  0001 C CNN
@@
 $EndComp
 $Comp
-L Device:C C?
+L Device:C C38
 U 1 1 613A9295
 P 7550 1100
-F 0 "C?" H 7665 1146 50  0000 L CNN
+F 0 "C38" H 7665 1146 50  0000 L CNN
 F 1 "1uF" H 7665 1055 50  0000 L CNN
 F 2 "Capacitor_SMD:C_0402_1005Metric" H 7588 950 50  0001 C CNN
@@
 $EndComp
 $Comp
-L Device:C C?
+L Device:C C39
 U 1 1 613A95E2
 P 8000 1100
-F 0 "C?" H 8115 1146 50  0000 L CNN
+F 0 "C39" H 8115 1146 50  0000 L CNN
 F 1 "1uF" H 8115 1055 50  0000 L CNN
 F 2 "Capacitor_SMD:C_0402_1005Metric" H 8038 950 50  0001 C CNN
@@
 $EndComp
 $Comp
-L Device:C C?
+L Device:C C40
 U 1 1 613A9A71
 P 8450 1100
-F 0 "C?" H 8565 1146 50  0000 L CNN
+F 0 "C40" H 8565 1146 50  0000 L CNN
 F 1 "1uF" H 8565 1055 50  0000 L CNN
 F 2 "Capacitor_SMD:C_0402_1005Metric" H 8488 950 50  0001 C CNN
@@
 $EndComp
 $Comp
-L Device:C C?
+L Device:C C41
 U 1 1 613A9D53
 P 8900 1100
-F 0 "C?" H 9015 1146 50  0000 L CNN
+F 0 "C41" H 9015 1146 50  0000 L CNN
 F 1 "1uF" H 9015 1055 50  0000 L CNN
 F 2 "Capacitor_SMD:C_0402_1005Metric" H 8938 950 50  0001 C CNN
@@
 $EndComp
 $Comp
-L Device:C C?
+L Device:C C42
 U 1 1 613AA142
 P 9350 1100
-F 0 "C?" H 9465 1146 50  0000 L CNN
+F 0 "C42" H 9465 1146 50  0000 L CNN
 F 1 "1uF" H 9465 1055 50  0000 L CNN
 F 2 "Capacitor_SMD:C_0402_1005Metric" H 9388 950 50  0001 C CNN
@@
 	8900 1250 8450 1250
 $Comp
-L power:GND #PWR?
+L power:GND #PWR0149
 U 1 1 613AB8E0
 P 8900 1250
-F 0 "#PWR?" H 8900 1000 50  0001 C CNN
+F 0 "#PWR0149" H 8900 1000 50  0001 C CNN
 F 1 "GND" H 8905 1077 50  0000 C CNN
 F 2 "" H 8900 1250 50  0001 C CNN
@@
 	7000 2500 7050 2500
 $Comp
-L power:GND #PWR?
+L power:GND #PWR0150
 U 1 1 613CAEB7
 P 7050 3400
-F 0 "#PWR?" H 7050 3150 50  0001 C CNN
+F 0 "#PWR0150" H 7050 3150 50  0001 C CNN
 F 1 "GND" H 7055 3227 50  0000 C CNN
 F 2 "" H 7050 3400 50  0001 C CNN
@@
 NoConn ~ 5150 2300
 $Comp
-L Regulator_Linear:MIC5365-3.3YD5 U?
+L Regulator_Linear:MIC5365-3.3YD5 U4
 U 1 1 613FD667
 P 3050 2400
-F 0 "U?" H 3050 2767 50  0000 C CNN
+F 0 "U4" H 3050 2767 50  0000 C CNN
 F 1 "MIC5365-2.8YD5" H 3050 2676 50  0000 C CNN
 F 2 "Package_TO_SOT_SMD:SOT-23-5" H 3050 2750 50  0001 C CNN
@@
 Connection ~ 2600 2300
 $Comp
-L Device:C C?
+L Device:C C53
 U 1 1 61405D62
 P 2300 2500
-F 0 "C?" H 2415 2546 50  0000 L CNN
+F 0 "C53" H 2415 2546 50  0000 L CNN
 F 1 "1uF" H 2415 2455 50  0000 L CNN
 F 2 "Capacitor_SMD:C_0402_1005Metric" H 2338 2350 50  0001 C CNN
@@
 $EndComp
 $Comp
-L power:+3.3V #PWR?
+L power:+3.3V #PWR0151
 U 1 1 614078C8
 P 2300 2150
-F 0 "#PWR?" H 2300 2000 50  0001 C CNN
+F 0 "#PWR0151" H 2300 2000 50  0001 C CNN
 F 1 "+3.3V" H 2315 2323 50  0000 C CNN
 F 2 "" H 2300 2150 50  0001 C CNN
@@
 Connection ~ 2300 2300
 $Comp
-L power:GND #PWR?
+L power:GND #PWR0152
 U 1 1 6140EDD3
 P 2300 2700
-F 0 "#PWR?" H 2300 2450 50  0001 C CNN
+F 0 "#PWR0152" H 2300 2450 50  0001 C CNN
 F 1 "GND" H 2305 2527 50  0000 C CNN
 F 2 "" H 2300 2700 50  0001 C CNN
@@
 	2300 2650 2300 2700
 $Comp
-L power:+2V8 #PWR?
+L power:+2V8 #PWR0153
 U 1 1 6141426A
 P 3650 2150
-F 0 "#PWR?" H 3650 2000 50  0001 C CNN
+F 0 "#PWR0153" H 3650 2000 50  0001 C CNN
 F 1 "+2V8" H 3665 2323 50  0000 C CNN
 F 2 "" H 3650 2150 50  0001 C CNN
@@
 Connection ~ 6150 3650
 $Comp
-L power:GND #PWR?
+L power:GND #PWR0154
 U 1 1 61419A0E
 P 8900 2350
-F 0 "#PWR?" H 8900 2100 50  0001 C CNN
+F 0 "#PWR0154" H 8900 2100 50  0001 C CNN
 F 1 "GND" H 8905 2177 50  0000 C CNN
 F 2 "" H 8900 2350 50  0001 C CNN
@@
 	3450 2300 3650 2300
 $Comp
-L Device:C C?
+L Device:C C52
 U 1 1 6141FC67
 P 3650 2450
-F 0 "C?" H 3765 2496 50  0000 L CNN
+F 0 "C52" H 3765 2496 50  0000 L CNN
 F 1 "1uF" H 3765 2405 50  0000 L CNN
 F 2 "Capacitor_SMD:C_0402_1005Metric" H 3688 2300 50  0001 C CNN
@@
 Connection ~ 3050 2700
 $Comp
-L power:+1V8 #PWR?
+L power:+1V8 #PWR0155
 U 1 1 613CD932
 P 7750 2800
-F 0 "#PWR?" H 7750 2650 50  0001 C CNN
+F 0 "#PWR0155" H 7750 2650 50  0001 C CNN
 F 1 "+1V8" H 7765 2973 50  0000 C CNN
 F 2 "" H 7750 2800 50  0001 C CNN
@@
 $EndComp
 $Comp
-L Device:R R?
+L Device:R R17
 U 1 1 613CB6A4
 P 7750 2950
-F 0 "R?" H 7820 2996 50  0000 L CNN
+F 0 "R17" H 7820 2996 50  0000 L CNN
 F 1 "4.7k" H 7820 2905 50  0000 L CNN
 F 2 "Resistor_SMD:R_0402_1005Metric" V 7680 2950 50  0001 C CNN
@@
 P 4300 6700
 AR Path="/6108B368/615777E1" Ref="#PWR?"  Part="1"
-AR Path="/6136B1E7/615777E1" Ref="#PWR?"  Part="1"
-F 0 "#PWR?" H 4300 6450 50  0001 C CNN
+AR Path="/6136B1E7/615777E1" Ref="#PWR0156"  Part="1"
+F 0 "#PWR0156" H 4300 6450 50  0001 C CNN
 F 1 "GND" H 4305 6527 50  0000 C CNN
 F 2 "" H 4300 6700 50  0001 C CNN
@@
 P 4150 6650
 AR Path="/6108B368/61577817" Ref="#PWR?"  Part="1"
-AR Path="/6136B1E7/61577817" Ref="#PWR?"  Part="1"
-F 0 "#PWR?" H 4150 6500 50  0001 C CNN
+AR Path="/6136B1E7/61577817" Ref="#PWR0157"  Part="1"
+F 0 "#PWR0157" H 4150 6500 50  0001 C CNN
 F 1 "+3.3V" V 4165 6778 50  0000 L CNN
 F 2 "" H 4150 6650 50  0001 C CNN
@@
 EXTCAM_D3_P
 $Comp
-L imucam:54548-2271 J?
+L imucam:54548-2271 J2
 U 1 1 60CE4657
 P 4550 4450
-F 0 "J?" H 4630 3346 50  0000 L CNN
+F 0 "J2" H 4630 3346 50  0000 L CNN
 F 1 "EXTCAM" H 4630 3255 50  0000 L CNN
 F 2 "imucam:Molex_545482271" H 4550 4450 50  0001 C CNN

Commit message: Final schematic rev?
Parts:
- added H1, H2, H3, H4: MountingHole, symbol Mechanical:MountingHole
Changed lines of the file:
@@
+	1    0    0    -1
+$EndComp
+$Comp
+L Mechanical:MountingHole H1
+U 1 1 60D095D3
+P 5500 5000
+F 0 "H1" H 5600 5046 50  0000 L CNN
+F 1 "MountingHole" H 5600 4955 50  0000 L CNN
+F 2 "" H 5500 5000 50  0001 C CNN
+F 3 "~" H 5500 5000 50  0001 C CNN
+	1    5500 5000
+	1    0    0    -1
+$EndComp
+$Comp
+L Mechanical:MountingHole H2
+U 1 1 60D098E1
+P 5500 5200
+F 0 "H2" H 5600 5246 50  0000 L CNN
+F 1 "MountingHole" H 5600 5155 50  0000 L CNN
+F 2 "" H 5500 5200 50  0001 C CNN
+F 3 "~" H 5500 5200 50  0001 C CNN
+	1    5500 5200
+	1    0    0    -1
+$EndComp
+$Comp
+L Mechanical:MountingHole H3
+U 1 1 60D09D87
+P 5500 5400
+F 0 "H3" H 5600 5446 50  0000 L CNN
+F 1 "MountingHole" H 5600 5355 50  0000 L CNN
+F 2 "" H 5500 5400 50  0001 C CNN
+F 3 "~" H 5500 5400 50  0001 C CNN
+	1    5500 5400
+	1    0    0    -1
+$EndComp
+$Comp
+L Mechanical:MountingHole H4
+U 1 1 60D0A1B1
+P 5500 5600
+F 0 "H4" H 5600 5646 50  0000 L CNN
+F 1 "MountingHole" H 5600 5555 50  0000 L CNN
+F 2 "" H 5500 5600 50  0001 C CNN
+F 3 "~" H 5500 5600 50  0001 C CNN
+	1    5500 5600
 	1    0    0    -1
 $EndComp

Commit message: Lots of schematic work
Parts:
- H1, H2, H3, H4: footprint (none) -> MountingHole:MountingHole_2.5mm
Changed lines of the file:
@@
 $EndComp
 $Comp
-L power:GND #PWR0145
+L power:GND #PWR055
 U 1 1 61370FCE
 P 6050 3650
-F 0 "#PWR0145" H 6050 3400 50  0001 C CNN
+F 0 "#PWR055" H 6050 3400 50  0001 C CNN
 F 1 "GND" H 6055 3477 50  0000 C CNN
 F 2 "" H 6050 3650 50  0001 C CNN
@@
 	7000 2100 7050 2100
 $Comp
-L power:+2V8 #PWR0146
+L power:+2V8 #PWR048
 U 1 1 61379194
 P 7200 2050
-F 0 "#PWR0146" H 7200 1900 50  0001 C CNN
+F 0 "#PWR048" H 7200 1900 50  0001 C CNN
 F 1 "+2V8" H 7215 2223 50  0000 C CNN
 F 2 "" H 7200 2050 50  0001 C CNN
@@
 	7050 1900 7050 1800
 $Comp
-L power:+1V8 #PWR0147
+L power:+1V8 #PWR045
 U 1 1 61397BEE
 P 7200 950
-F 0 "#PWR0147" H 7200 800 50  0001 C CNN
+F 0 "#PWR045" H 7200 800 50  0001 C CNN
 F 1 "+1V8" H 7215 1123 50  0000 C CNN
 F 2 "" H 7200 950 50  0001 C CNN
@@
 	8900 1800 8450 1800
 $Comp
-L power:GND #PWR0148
+L power:GND #PWR047
 U 1 1 613A900D
 P 8900 1800
-F 0 "#PWR0148" H 8900 1550 50  0001 C CNN
+F 0 "#PWR047" H 8900 1550 50  0001 C CNN
 F 1 "GND" H 8905 1627 50  0000 C CNN
 F 2 "" H 8900 1800 50  0001 C CNN
@@
 	8900 1250 8450 1250
 $Comp
-L power:GND #PWR0149
+L power:GND #PWR046
 U 1 1 613AB8E0
 P 8900 1250
-F 0 "#PWR0149" H 8900 1000 50  0001 C CNN
+F 0 "#PWR046" H 8900 1000 50  0001 C CNN
 F 1 "GND" H 8905 1077 50  0000 C CNN
 F 2 "" H 8900 1250 50  0001 C CNN
@@
 	7000 2500 7050 2500
 $Comp
-L power:GND #PWR0150
+L power:GND #PWR054
 U 1 1 613CAEB7
 P 7050 3400
-F 0 "#PWR0150" H 7050 3150 50  0001 C CNN
+F 0 "#PWR054" H 7050 3150 50  0001 C CNN
 F 1 "GND" H 7055 3227 50  0000 C CNN
 F 2 "" H 7050 3400 50  0001 C CNN
@@
 $EndComp
 $Comp
-L power:+3.3V #PWR0151
+L power:+3.3V #PWR049
 U 1 1 614078C8
 P 2300 2150
-F 0 "#PWR0151" H 2300 2000 50  0001 C CNN
+F 0 "#PWR049" H 2300 2000 50  0001 C CNN
 F 1 "+3.3V" H 2315 2323 50  0000 C CNN
 F 2 "" H 2300 2150 50  0001 C CNN
@@
 Connection ~ 2300 2300
 $Comp
-L power:GND #PWR0152
+L power:GND #PWR052
 U 1 1 6140EDD3
 P 2300 2700
-F 0 "#PWR0152" H 2300 2450 50  0001 C CNN
+F 0 "#PWR052" H 2300 2450 50  0001 C CNN
 F 1 "GND" H 2305 2527 50  0000 C CNN
 F 2 "" H 2300 2700 50  0001 C CNN
@@
 	2300 2650 2300 2700
 $Comp
-L power:+2V8 #PWR0153
+L power:+2V8 #PWR050
 U 1 1 6141426A
 P 3650 2150
-F 0 "#PWR0153" H 3650 2000 50  0001 C CNN
+F 0 "#PWR050" H 3650 2000 50  0001 C CNN
 F 1 "+2V8" H 3665 2323 50  0000 C CNN
 F 2 "" H 3650 2150 50  0001 C CNN
@@
 Connection ~ 6150 3650
 $Comp
-L power:GND #PWR0154
+L power:GND #PWR051
 U 1 1 61419A0E
 P 8900 2350
-F 0 "#PWR0154" H 8900 2100 50  0001 C CNN
+F 0 "#PWR051" H 8900 2100 50  0001 C CNN
 F 1 "GND" H 8905 2177 50  0000 C CNN
 F 2 "" H 8900 2350 50  0001 C CNN
@@
 Connection ~ 3050 2700
 $Comp
-L power:+1V8 #PWR0155
+L power:+1V8 #PWR053
 U 1 1 613CD932
 P 7750 2800
-F 0 "#PWR0155" H 7750 2650 50  0001 C CNN
+F 0 "#PWR053" H 7750 2650 50  0001 C CNN
 F 1 "+1V8" H 7765 2973 50  0000 C CNN
 F 2 "" H 7750 2800 50  0001 C CNN
@@
 P 4300 6700
 AR Path="/6108B368/615777E1" Ref="#PWR?"  Part="1"
-AR Path="/6136B1E7/615777E1" Ref="#PWR0156"  Part="1"
-F 0 "#PWR0156" H 4300 6450 50  0001 C CNN
+AR Path="/6136B1E7/615777E1" Ref="#PWR057"  Part="1"
+F 0 "#PWR057" H 4300 6450 50  0001 C CNN
 F 1 "GND" H 4305 6527 50  0000 C CNN
 F 2 "" H 4300 6700 50  0001 C CNN
@@
 P 4150 6650
 AR Path="/6108B368/61577817" Ref="#PWR?"  Part="1"
-AR Path="/6136B1E7/61577817" Ref="#PWR0157"  Part="1"
-F 0 "#PWR0157" H 4150 6500 50  0001 C CNN
+AR Path="/6136B1E7/61577817" Ref="#PWR056"  Part="1"
+F 0 "#PWR056" H 4150 6500 50  0001 C CNN
 F 1 "+3.3V" V 4165 6778 50  0000 L CNN
 F 2 "" H 4150 6650 50  0001 C CNN
@@
 F 0 "H1" H 5600 5046 50  0000 L CNN
 F 1 "MountingHole" H 5600 4955 50  0000 L CNN
-F 2 "" H 5500 5000 50  0001 C CNN
+F 2 "MountingHole:MountingHole_2.5mm" H 5500 5000 50  0001 C CNN
 F 3 "~" H 5500 5000 50  0001 C CNN
 	1    5500 5000
@@
 F 0 "H2" H 5600 5246 50  0000 L CNN
 F 1 "MountingHole" H 5600 5155 50  0000 L CNN
-F 2 "" H 5500 5200 50  0001 C CNN
+F 2 "MountingHole:MountingHole_2.5mm" H 5500 5200 50  0001 C CNN
 F 3 "~" H 5500 5200 50  0001 C CNN
 	1    5500 5200
@@
 F 0 "H3" H 5600 5446 50  0000 L CNN
 F 1 "MountingHole" H 5600 5355 50  0000 L CNN
-F 2 "" H 5500 5400 50  0001 C CNN
+F 2 "MountingHole:MountingHole_2.5mm" H 5500 5400 50  0001 C CNN
 F 3 "~" H 5500 5400 50  0001 C CNN
 	1    5500 5400
@@
 F 0 "H4" H 5600 5646 50  0000 L CNN
 F 1 "MountingHole" H 5600 5555 50  0000 L CNN
-F 2 "" H 5500 5600 50  0001 C CNN
+F 2 "MountingHole:MountingHole_2.5mm" H 5500 5600 50  0001 C CNN
 F 3 "~" H 5500 5600 50  0001 C CNN
 	1    5500 5600

Commit message: More work on PCB
Parts:
- removed H1, H2, H3, H4: MountingHole, MountingHole:MountingHole_2.5mm, symbol Mechanical:MountingHole
Changed lines of the file:
@@
-	1    0    0    -1
-$EndComp
-$Comp
-L Mechanical:MountingHole H1
-U 1 1 60D095D3
-P 5500 5000
-F 0 "H1" H 5600 5046 50  0000 L CNN
-F 1 "MountingHole" H 5600 4955 50  0000 L CNN
-F 2 "MountingHole:MountingHole_2.5mm" H 5500 5000 50  0001 C CNN
-F 3 "~" H 5500 5000 50  0001 C CNN
-	1    5500 5000
-	1    0    0    -1
-$EndComp
-$Comp
-L Mechanical:MountingHole H2
-U 1 1 60D098E1
-P 5500 5200
-F 0 "H2" H 5600 5246 50  0000 L CNN
-F 1 "MountingHole" H 5600 5155 50  0000 L CNN
-F 2 "MountingHole:MountingHole_2.5mm" H 5500 5200 50  0001 C CNN
-F 3 "~" H 5500 5200 50  0001 C CNN
-	1    5500 5200
-	1    0    0    -1
-$EndComp
-$Comp
-L Mechanical:MountingHole H3
-U 1 1 60D09D87
-P 5500 5400
-F 0 "H3" H 5600 5446 50  0000 L CNN
-F 1 "MountingHole" H 5600 5355 50  0000 L CNN
-F 2 "MountingHole:MountingHole_2.5mm" H 5500 5400 50  0001 C CNN
-F 3 "~" H 5500 5400 50  0001 C CNN
-	1    5500 5400
-	1    0    0    -1
-$EndComp
-$Comp
-L Mechanical:MountingHole H4
-U 1 1 60D0A1B1
-P 5500 5600
-F 0 "H4" H 5600 5646 50  0000 L CNN
-F 1 "MountingHole" H 5600 5555 50  0000 L CNN
-F 2 "MountingHole:MountingHole_2.5mm" H 5500 5600 50  0001 C CNN
-F 3 "~" H 5500 5600 50  0001 C CNN
-	1    5500 5600
 	1    0    0    -1
 $EndComp

Commit message: Switched FSYNC to use TRIGGER, lots of PCB work
Parts:
- added H1: M12Lens, imucam:M12_Lens_20mm, symbol imucam:M12Lens
- added H2: EXTCAM, imucam:Arducam_module_40mm, symbol imucam:Arducam_Module
Connections:
- net labels added: CAM_TRIGGER
- net labels removed: CAM_FLASH, CAM_SHUTTER
- wire segments 117 -> 116
Changed lines of the file:
@@
 $EndComp
-Wire Wire Line
-	7000 3000 7050 3000
 Wire Wire Line
 	7000 3300 7050 3300
-Connection ~ 7050 3300
 Wire Wire Line
 	7050 3300 7050 3400
@@
 Text GLabel 8000 3200 2    50   Input ~ 0
 CLK_24MHZ
-Text GLabel 7050 2800 2    50   Input ~ 0
-CAM_FLASH
-Text GLabel 7050 2900 2    50   Input ~ 0
-CAM_SHUTTER
 Wire Wire Line
 	7000 2800 7050 2800
 Wire Wire Line
 	7000 2900 7050 2900
-Wire Wire Line
-	7050 3000 7050 3300
 Wire Wire Line
 	7000 3100 7750 3100
@@
 	1    0    0    -1
 $EndComp
+$Comp
+L imucam:M12Lens H1
+U 1 1 61429870
+P 4750 1000
+F 0 "H1" H 4500 1300 50  0000 L CNN
+F 1 "M12Lens" H 4750 700 50  0001 C CNN
+F 2 "imucam:M12_Lens_20mm" H 4750 600 50  0001 C CNN
+F 3 "" H 4750 1000 50  0001 C CNN
+	1    4750 1000
+	1    0    0    -1
+$EndComp
+$Comp
+L imucam:Arducam_Module H2
+U 1 1 61438A5A
+P 5350 5650
+F 0 "H2" H 5100 6000 50  0000 L CNN
+F 1 "EXTCAM" H 5250 5300 50  0000 C CNN
+F 2 "imucam:Arducam_module_40mm" H 5350 5200 50  0001 C CNN
+F 3 "" H 5350 5650 50  0001 C CNN
+	1    5350 5650
+	1    0    0    -1
+$EndComp
+Text GLabel 7100 3000 2    50   Input ~ 0
+CAM_TRIGGER
+Wire Wire Line
+	7000 3000 7100 3000
 $EndSCHEMATC
