File: kicad/imucam/cam.sch (KiCad schematic (older format))
At the start: 22 parts, among them J2 EXTCAM, U4 MIC5365-2.8YD5, U5 AR0330CM1C00

Commit message: Slightly more progress on current measurement
Parts:
- renumbered C53 to C38, C52 to C39, C38 to C40, C43 to C41, C48 to C42, C39 to C43, C49 to C45, C40 to C46, C45 to C47, C50 to C48, C41 to C49, C46 to C50, C42 to C52, C47 to C53
Changed lines of the file:
@@
 $EndComp
 $Comp
-L power:GND #PWR055
+L power:GND #PWR050
 U 1 1 61370FCE
 P 6050 3650
-F 0 "#PWR055" H 6050 3400 50  0001 C CNN
+F 0 "#PWR050" H 6050 3400 50  0001 C CNN
 F 1 "GND" H 6055 3477 50  0000 C CNN
 F 2 "" H 6050 3650 50  0001 C CNN
@@
 $EndComp
 $Comp
-L Device:C C49
+L Device:C C45
 U 1 1 613752DC
 P 8000 2200
-F 0 "C49" H 8115 2246 50  0000 L CNN
+F 0 "C45" H 8115 2246 50  0000 L CNN
 F 1 "100nF" H 8115 2155 50  0000 L CNN
 F 2 "Capacitor_SMD:C_0402_1005Metric" H 8038 2050 50  0001 C CNN
@@
 	7000 2100 7050 2100
 $Comp
-L power:+2V8 #PWR048
+L power:+2V8 #PWR053
 U 1 1 61379194
 P 7200 2050
-F 0 "#PWR048" H 7200 1900 50  0001 C CNN
+F 0 "#PWR053" H 7200 1900 50  0001 C CNN
 F 1 "+2V8" H 7215 2223 50  0000 C CNN
 F 2 "" H 7200 2050 50  0001 C CNN
@@
 $EndComp
 $Comp
-L Device:C C50
+L Device:C C48
 U 1 1 61387529
 P 8450 2200
-F 0 "C50" H 8565 2246 50  0000 L CNN
+F 0 "C48" H 8565 2246 50  0000 L CNN
 F 1 "1uF" H 8565 2155 50  0000 L CNN
 F 2 "Capacitor_SMD:C_0402_1005Metric" H 8488 2050 50  0001 C CNN
@@
 $EndComp
 $Comp
-L Device:C C48
+L Device:C C42
 U 1 1 6138752F
 P 7550 2200
-F 0 "C48" H 7665 2246 50  0000 L CNN
+F 0 "C42" H 7665 2246 50  0000 L CNN
 F 1 "100nF" H 7665 2155 50  0000 L CNN
 F 2 "Capacitor_SMD:C_0402_1005Metric" H 7588 2050 50  0001 C CNN
@@
 	7050 1900 7050 1800
 $Comp
-L power:+1V8 #PWR045
+L power:+1V8 #PWR052
 U 1 1 61397BEE
 P 7200 950
-F 0 "#PWR045" H 7200 800 50  0001 C CNN
+F 0 "#PWR052" H 7200 800 50  0001 C CNN
 F 1 "+1V8" H 7215 1123 50  0000 C CNN
 F 2 "" H 7200 950 50  0001 C CNN
@@
 Connection ~ 7550 2050
 $Comp
-L Device:C C43
+L Device:C C41
 U 1 1 613A452F
 P 7550 1650
-F 0 "C43" H 7665 1696 50  0000 L CNN
+F 0 "C41" H 7665 1696 50  0000 L CNN
 F 1 "100nF" H 7665 1605 50  0000 L CNN
 F 2 "Capacitor_SMD:C_0402_1005Metric" H 7588 1500 50  0001 C CNN
@@
 $EndComp
 $Comp
-L Device:C C45
+L Device:C C47
 U 1 1 613A4F84
 P 8450 1650
-F 0 "C45" H 8565 1696 50  0000 L CNN
+F 0 "C47" H 8565 1696 50  0000 L CNN
 F 1 "100nF" H 8565 1605 50  0000 L CNN
 F 2 "Capacitor_SMD:C_0402_1005Metric" H 8488 1500 50  0001 C CNN
@@
 $EndComp
 $Comp
-L Device:C C46
+L Device:C C50
 U 1 1 613A54C1
 P 8900 1650
-F 0 "C46" H 9015 1696 50  0000 L CNN
+F 0 "C50" H 9015 1696 50  0000 L CNN
 F 1 "100nF" H 9015 1605 50  0000 L CNN
 F 2 "Capacitor_SMD:C_0402_1005Metric" H 8938 1500 50  0001 C CNN
@@
 	8450 2050 8900 2050
 $Comp
-L Device:C C47
+L Device:C C53
 U 1 1 613A733B
 P 9350 1650
-F 0 "C47" H 9465 1696 50  0000 L CNN
+F 0 "C53" H 9465 1696 50  0000 L CNN
 F 1 "100nF" H 9465 1605 50  0000 L CNN
 F 2 "Capacitor_SMD:C_0402_1005Metric" H 9388 1500 50  0001 C CNN
@@
 	8900 1800 8450 1800
 $Comp
-L power:GND #PWR047
+L power:GND #PWR056
 U 1 1 613A900D
 P 8900 1800
-F 0 "#PWR047" H 8900 1550 50  0001 C CNN
+F 0 "#PWR056" H 8900 1550 50  0001 C CNN
 F 1 "GND" H 8905 1627 50  0000 C CNN
 F 2 "" H 8900 1800 50  0001 C CNN
@@
 $EndComp
 $Comp
-L Device:C C38
+L Device:C C40
 U 1 1 613A9295
 P 7550 1100
-F 0 "C38" H 7665 1146 50  0000 L CNN
+F 0 "C40" H 7665 1146 50  0000 L CNN
 F 1 "1uF" H 7665 1055 50  0000 L CNN
 F 2 "Capacitor_SMD:C_0402_1005Metric" H 7588 950 50  0001 C CNN
@@
 $EndComp
 $Comp
-L Device:C C39
+L Device:C C43
 U 1 1 613A95E2
 P 8000 1100
-F 0 "C39" H 8115 1146 50  0000 L CNN
+F 0 "C43" H 8115 1146 50  0000 L CNN
 F 1 "1uF" H 8115 1055 50  0000 L CNN
 F 2 "Capacitor_SMD:C_0402_1005Metric" H 8038 950 50  0001 C CNN
@@
 $EndComp
 $Comp
-L Device:C C40
+L Device:C C46
 U 1 1 613A9A71
 P 8450 1100
-F 0 "C40" H 8565 1146 50  0000 L CNN
+F 0 "C46" H 8565 1146 50  0000 L CNN
 F 1 "1uF" H 8565 1055 50  0000 L CNN
 F 2 "Capacitor_SMD:C_0402_1005Metric" H 8488 950 50  0001 C CNN
@@
 $EndComp
 $Comp
-L Device:C C41
+L Device:C C49
 U 1 1 613A9D53
 P 8900 1100
-F 0 "C41" H 9015 1146 50  0000 L CNN
+F 0 "C49" H 9015 1146 50  0000 L CNN
 F 1 "1uF" H 9015 1055 50  0000 L CNN
 F 2 "Capacitor_SMD:C_0402_1005Metric" H 8938 950 50  0001 C CNN
@@
 $EndComp
 $Comp
-L Device:C C42
+L Device:C C52
 U 1 1 613AA142
 P 9350 1100
-F 0 "C42" H 9465 1146 50  0000 L CNN
+F 0 "C52" H 9465 1146 50  0000 L CNN
 F 1 "1uF" H 9465 1055 50  0000 L CNN
 F 2 "Capacitor_SMD:C_0402_1005Metric" H 9388 950 50  0001 C CNN
@@
 	8900 1250 8450 1250
 $Comp
-L power:GND #PWR046
+L power:GND #PWR055
 U 1 1 613AB8E0
 P 8900 1250
-F 0 "#PWR046" H 8900 1000 50  0001 C CNN
+F 0 "#PWR055" H 8900 1000 50  0001 C CNN
 F 1 "GND" H 8905 1077 50  0000 C CNN
 F 2 "" H 8900 1250 50  0001 C CNN
@@
 	7000 2500 7050 2500
 $Comp
-L power:GND #PWR054
+L power:GND #PWR051
 U 1 1 613CAEB7
 P 7050 3400
-F 0 "#PWR054" H 7050 3150 50  0001 C CNN
+F 0 "#PWR051" H 7050 3150 50  0001 C CNN
 F 1 "GND" H 7055 3227 50  0000 C CNN
 F 2 "" H 7050 3400 50  0001 C CNN
@@
 Connection ~ 2600 2300
 $Comp
-L Device:C C53
+L Device:C C38
 U 1 1 61405D62
 P 2300 2500
-F 0 "C53" H 2415 2546 50  0000 L CNN
+F 0 "C38" H 2415 2546 50  0000 L CNN
 F 1 "1uF" H 2415 2455 50  0000 L CNN
 F 2 "Capacitor_SMD:C_0402_1005Metric" H 2338 2350 50  0001 C CNN
@@
 $EndComp
 $Comp
-L power:+3.3V #PWR049
+L power:+3.3V #PWR045
 U 1 1 614078C8
 P 2300 2150
-F 0 "#PWR049" H 2300 2000 50  0001 C CNN
+F 0 "#PWR045" H 2300 2000 50  0001 C CNN
 F 1 "+3.3V" H 2315 2323 50  0000 C CNN
 F 2 "" H 2300 2150 50  0001 C CNN
@@
 Connection ~ 2300 2300
 $Comp
-L power:GND #PWR052
+L power:GND #PWR046
 U 1 1 6140EDD3
 P 2300 2700
-F 0 "#PWR052" H 2300 2450 50  0001 C CNN
+F 0 "#PWR046" H 2300 2450 50  0001 C CNN
 F 1 "GND" H 2305 2527 50  0000 C CNN
 F 2 "" H 2300 2700 50  0001 C CNN
@@
 	2300 2650 2300 2700
 $Comp
-L power:+2V8 #PWR050
+L power:+2V8 #PWR047
 U 1 1 6141426A
 P 3650 2150
-F 0 "#PWR050" H 3650 2000 50  0001 C CNN
+F 0 "#PWR047" H 3650 2000 50  0001 C CNN
 F 1 "+2V8" H 3665 2323 50  0000 C CNN
 F 2 "" H 3650 2150 50  0001 C CNN
@@
 Connection ~ 6150 3650
 $Comp
-L power:GND #PWR051
+L power:GND #PWR057
 U 1 1 61419A0E
 P 8900 2350
-F 0 "#PWR051" H 8900 2100 50  0001 C CNN
+F 0 "#PWR057" H 8900 2100 50  0001 C CNN
 F 1 "GND" H 8905 2177 50  0000 C CNN
 F 2 "" H 8900 2350 50  0001 C CNN
@@
 	3450 2300 3650 2300
 $Comp
-L Device:C C52
+L Device:C C39
 U 1 1 6141FC67
 P 3650 2450
-F 0 "C52" H 3765 2496 50  0000 L CNN
+F 0 "C39" H 3765 2496 50  0000 L CNN
 F 1 "1uF" H 3765 2405 50  0000 L CNN
 F 2 "Capacitor_SMD:C_0402_1005Metric" H 3688 2300 50  0001 C CNN
@@
 Connection ~ 3050 2700
 $Comp
-L power:+1V8 #PWR053
+L power:+1V8 #PWR054
 U 1 1 613CD932
 P 7750 2800
-F 0 "#PWR053" H 7750 2650 50  0001 C CNN
+F 0 "#PWR054" H 7750 2650 50  0001 C CNN
 F 1 "+1V8" H 7765 2973 50  0000 C CNN
 F 2 "" H 7750 2800 50  0001 C CNN
@@
 P 4300 6700
 AR Path="/6108B368/615777E1" Ref="#PWR?"  Part="1"
-AR Path="/6136B1E7/615777E1" Ref="#PWR057"  Part="1"
-F 0 "#PWR057" H 4300 6450 50  0001 C CNN
+AR Path="/6136B1E7/615777E1" Ref="#PWR049"  Part="1"
+F 0 "#PWR049" H 4300 6450 50  0001 C CNN
 F 1 "GND" H 4305 6527 50  0000 C CNN
 F 2 "" H 4300 6700 50  0001 C CNN
@@
 P 4150 6650
 AR Path="/6108B368/61577817" Ref="#PWR?"  Part="1"
-AR Path="/6136B1E7/61577817" Ref="#PWR056"  Part="1"
-F 0 "#PWR056" H 4150 6500 50  0001 C CNN
+AR Path="/6136B1E7/61577817" Ref="#PWR048"  Part="1"
+F 0 "#PWR048" H 4150 6500 50  0001 C CNN
 F 1 "+3.3V" V 4165 6778 50  0000 L CNN
 F 2 "" H 4150 6650 50  0001 C CNN

Commit message: Turns out, we need level translators
Parts:
- removed C50, C53: 100nF, Capacitor_SMD:C_0402_1005Metric, symbol Device:C
- removed C51, C52: 1uF, Capacitor_SMD:C_0402_1005Metric, symbol Device:C
- removed R17: 4.7k, Resistor_SMD:R_0402_1005Metric, symbol Device:R
- added C38: 1uF, Capacitor_SMD:C_0402_1005Metric, symbol Device:C
- added C39: 100nF, Capacitor_SMD:C_0402_1005Metric, symbol Device:C
- C42, C44: value 100nF -> 1uF
- C43, C49: value 1uF -> 100nF
- renumbered C39 to C50, C38 to C51
Connections:
- net labels added: CAM_FLASH, CAM_SHUTTER
- wire segments 116 -> 111
