File: kicad/imucam/cam.sch (KiCad schematic (older format))
At the start: 19 parts, among them J2 EXTCAM, U4 MIC5365-2.8YD5, U5 AR0330CM1C00

Commit message: WIP of remapping nucleo pinout for pcb routing
Parts:
- added R17: 4.7k, Resistor_SMD:R_0402_1005Metric, symbol Device:R
- renumbered C51 to C38, C50 to C39, C38 to C40, C42 to C41, C39 to C42, C40 to C44, C44 to C45, C41 to C46, C45 to C47, C46 to C48, C47 to C49, C48 to C50, C49 to C51
Connections:
- net labels added: +3V3
- net labels removed: CAM_FLASH, CAM_SHUTTER
- wire segments 111 -> 113
- no-connect marks 10 -> 12
Changed lines of the file:
@@
 $EndDescr
 $Comp
-L power:GND #PWR052
+L power:GND #PWR048
 U 1 1 61370FCE
 P 6050 3650
-F 0 "#PWR052" H 6050 3400 50  0001 C CNN
+F 0 "#PWR048" H 6050 3400 50  0001 C CNN
 F 1 "GND" H 6055 3477 50  0000 C CNN
 F 2 "" H 6050 3650 50  0001 C CNN
@@
 Wire Wire Line
 	6350 3600 6350 3650
-Text GLabel 7050 2400 2    50   BiDi ~ 0
+Text GLabel 7400 2400 2    50   BiDi ~ 0
 SCL_1V8
-Text GLabel 7050 2500 2    50   BiDi ~ 0
+Text GLabel 7400 2500 2    50   BiDi ~ 0
 SDA_1V8
 Wire Wire Line
-	7000 2400 7050 2400
-Wire Wire Line
-	7000 2500 7050 2500
+	7000 2400 7400 2400
+Wire Wire Line
+	7000 2500 7400 2500
 Wire Wire Line
 	7000 3300 7050 3300
@@
 Connection ~ 2600 2300
 $Comp
-L Device:C C51
+L Device:C C38
 U 1 1 61405D62
 P 2300 2500
-F 0 "C51" H 2415 2546 50  0000 L CNN
+F 0 "C38" H 2415 2546 50  0000 L CNN
 F 1 "1uF" H 2415 2455 50  0000 L CNN
 F 2 "Capacitor_SMD:C_0402_1005Metric" H 2338 2350 50  0001 C CNN
@@
 	1    0    0    -1
 $EndComp
-$Comp
-L power:+3.3V #PWR049
-U 1 1 614078C8
-P 2300 2150
-F 0 "#PWR049" H 2300 2000 50  0001 C CNN
-F 1 "+3.3V" H 2315 2323 50  0000 C CNN
-F 2 "" H 2300 2150 50  0001 C CNN
-F 3 "" H 2300 2150 50  0001 C CNN
-	1    2300 2150
-	1    0    0    -1
-$EndComp
 Wire Wire Line
 	2300 2300 2300 2350
 Connection ~ 2300 2300
 $Comp
-L power:GND #PWR051
+L power:GND #PWR044
 U 1 1 6140EDD3
 P 2300 2700
-F 0 "#PWR051" H 2300 2450 50  0001 C CNN
+F 0 "#PWR044" H 2300 2450 50  0001 C CNN
 F 1 "GND" H 2305 2527 50  0000 C CNN
 F 2 "" H 2300 2700 50  0001 C CNN
@@
 	2300 2650 2300 2700
 $Comp
-L power:+2V8 #PWR050
+L power:+2V8 #PWR045
 U 1 1 6141426A
 P 3650 2150
-F 0 "#PWR050" H 3650 2000 50  0001 C CNN
+F 0 "#PWR045" H 3650 2000 50  0001 C CNN
 F 1 "+2V8" H 3665 2323 50  0000 C CNN
 F 2 "" H 3650 2150 50  0001 C CNN
@@
 	3450 2300 3650 2300
 $Comp
-L Device:C C50
+L Device:C C39
 U 1 1 6141FC67
 P 3650 2450
-F 0 "C50" H 3765 2496 50  0000 L CNN
+F 0 "C39" H 3765 2496 50  0000 L CNN
 F 1 "1uF" H 3765 2405 50  0000 L CNN
 F 2 "Capacitor_SMD:C_0402_1005Metric" H 3688 2300 50  0001 C CNN
@@
 	3650 2700 3650 2600
 Connection ~ 3050 2700
-Text GLabel 7050 3100 2    50   Input ~ 0
+Text GLabel 7400 3100 2    50   Input ~ 0
 CAM_RESET_BAR
-Text GLabel 7050 3200 2    50   Input ~ 0
+Text GLabel 7400 3200 2    50   Input ~ 0
 CLK_24MHZ
 Wire Wire Line
@@
 	7000 2900 7050 2900
 Wire Wire Line
-	7000 3200 7050 3200
+	7000 3200 7400 3200
 $Comp
 L power:GND #PWR?
@@
 P 4300 6700
 AR Path="/6108B368/615777E1" Ref="#PWR?"  Part="1"
-AR Path="/6136B1E7/615777E1" Ref="#PWR054"  Part="1"
-F 0 "#PWR054" H 4300 6450 50  0001 C CNN
+AR Path="/6136B1E7/615777E1" Ref="#PWR047"  Part="1"
+F 0 "#PWR047" H 4300 6450 50  0001 C CNN
 F 1 "GND" H 4305 6527 50  0000 C CNN
 F 2 "" H 4300 6700 50  0001 C CNN
@@
 P 4150 6650
 AR Path="/6108B368/61577817" Ref="#PWR?"  Part="1"
-AR Path="/6136B1E7/61577817" Ref="#PWR053"  Part="1"
-F 0 "#PWR053" H 4150 6500 50  0001 C CNN
+AR Path="/6136B1E7/61577817" Ref="#PWR046"  Part="1"
+F 0 "#PWR046" H 4150 6500 50  0001 C CNN
 F 1 "+3.3V" V 4165 6778 50  0000 L CNN
 F 2 "" H 4150 6650 50  0001 C CNN
@@
 	1    0    0    -1
 $EndComp
-Text GLabel 7050 3000 2    50   Input ~ 0
+Text GLabel 7400 3000 2    50   Input ~ 0
 CAM_TRIGGER
 Wire Wire Line
-	7000 3000 7050 3000
+	7000 3000 7400 3000
 Wire Wire Line
 	7000 1900 7050 1900
@@
 	7050 1400 7050 1150
 $Comp
-L power:+1V8 #PWR045
+L power:+1V8 #PWR049
 U 1 1 6147C370
 P 7050 1100
-F 0 "#PWR045" H 7050 950 50  0001 C CNN
+F 0 "#PWR049" H 7050 950 50  0001 C CNN
 F 1 "+1V8" H 7065 1273 50  0000 C CNN
 F 2 "" H 7050 1100 50  0001 C CNN
@@
 Connection ~ 7050 1400
 $Comp
-L power:+2V8 #PWR046
+L power:+2V8 #PWR051
 U 1 1 61486FE0
 P 7300 1100
-F 0 "#PWR046" H 7300 950 50  0001 C CNN
+F 0 "#PWR051" H 7300 950 50  0001 C CNN
 F 1 "+2V8" H 7315 1273 50  0000 C CNN
 F 2 "" H 7300 1100 50  0001 C CNN
@@
 Connection ~ 7300 2100
 $Comp
-L Device:C C38
+L Device:C C40
 U 1 1 614AE316
 P 7800 1300
-F 0 "C38" H 7915 1346 50  0000 L CNN
+F 0 "C40" H 7915 1346 50  0000 L CNN
 F 1 "1uF" H 7915 1255 50  0000 L CNN
 F 2 "Capacitor_SMD:C_0402_1005Metric" H 7838 1150 50  0001 C CNN
@@
 $EndComp
 $Comp
-L Device:C C39
+L Device:C C42
 U 1 1 614AF4C7
 P 8200 1300
-F 0 "C39" H 8315 1346 50  0000 L CNN
+F 0 "C42" H 8315 1346 50  0000 L CNN
 F 1 "100nF" H 8315 1255 50  0000 L CNN
 F 2 "Capacitor_SMD:C_0402_1005Metric" H 8238 1150 50  0001 C CNN
@@
 $EndComp
 $Comp
-L Device:C C40
+L Device:C C44
 U 1 1 614AF9BD
 P 8650 1300
-F 0 "C40" H 8765 1346 50  0000 L CNN
+F 0 "C44" H 8765 1346 50  0000 L CNN
 F 1 "1uF" H 8765 1255 50  0000 L CNN
 F 2 "Capacitor_SMD:C_0402_1005Metric" H 8688 1150 50  0001 C CNN
@@
 $EndComp
 $Comp
-L Device:C C41
+L Device:C C46
 U 1 1 614B0284
 P 9050 1300
-F 0 "C41" H 9165 1346 50  0000 L CNN
+F 0 "C46" H 9165 1346 50  0000 L CNN
 F 1 "100nF" H 9165 1255 50  0000 L CNN
 F 2 "Capacitor_SMD:C_0402_1005Metric" H 9088 1150 50  0001 C CNN
@@
 	8650 1450 9050 1450
 $Comp
-L power:GND #PWR047
+L power:GND #PWR052
 U 1 1 614B5F27
 P 7800 1450
-F 0 "#PWR047" H 7800 1200 50  0001 C CNN
+F 0 "#PWR052" H 7800 1200 50  0001 C CNN
 F 1 "GND" H 7805 1277 50  0000 C CNN
 F 2 "" H 7800 1450 50  0001 C CNN
@@
 Connection ~ 7800 1450
 $Comp
-L Device:C C42
+L Device:C C41
 U 1 1 614B68CC
 P 7800 1850
-F 0 "C42" H 7915 1896 50  0000 L CNN
+F 0 "C41" H 7915 1896 50  0000 L CNN
 F 1 "1uF" H 7915 1805 50  0000 L CNN
 F 2 "Capacitor_SMD:C_0402_1005Metric" H 7838 1700 50  0001 C CNN
@@
 $EndComp
 $Comp
-L Device:C C44
+L Device:C C45
 U 1 1 614B6EDD
 P 8650 1850
-F 0 "C44" H 8765 1896 50  0000 L CNN
+F 0 "C45" H 8765 1896 50  0000 L CNN
 F 1 "1uF" H 8765 1805 50  0000 L CNN
 F 2 "Capacitor_SMD:C_0402_1005Metric" H 8688 1700 50  0001 C CNN
@@
 $EndComp
 $Comp
-L Device:C C46
+L Device:C C48
 U 1 1 614B71F7
 P 9500 1850
-F 0 "C46" H 9615 1896 50  0000 L CNN
+F 0 "C48" H 9615 1896 50  0000 L CNN
 F 1 "1uF" H 9615 1805 50  0000 L CNN
 F 2 "Capacitor_SMD:C_0402_1005Metric" H 9538 1700 50  0001 C CNN
@@
 $EndComp
 $Comp
-L Device:C C48
+L Device:C C50
 U 1 1 614B73A0
 P 10350 1850
-F 0 "C48" H 10465 1896 50  0000 L CNN
+F 0 "C50" H 10465 1896 50  0000 L CNN
 F 1 "1uF" H 10465 1805 50  0000 L CNN
 F 2 "Capacitor_SMD:C_0402_1005Metric" H 10388 1700 50  0001 C CNN
@@
 $EndComp
 $Comp
-L Device:C C45
+L Device:C C47
 U 1 1 614B77E5
 P 9050 1850
-F 0 "C45" H 9165 1896 50  0000 L CNN
+F 0 "C47" H 9165 1896 50  0000 L CNN
 F 1 "100nF" H 9165 1805 50  0000 L CNN
 F 2 "Capacitor_SMD:C_0402_1005Metric" H 9088 1700 50  0001 C CNN
@@
 $EndComp
 $Comp
-L Device:C C47
+L Device:C C49
 U 1 1 614BA230
 P 9900 1850
-F 0 "C47" H 10015 1896 50  0000 L CNN
+F 0 "C49" H 10015 1896 50  0000 L CNN
 F 1 "100nF" H 10015 1805 50  0000 L CNN
 F 2 "Capacitor_SMD:C_0402_1005Metric" H 9938 1700 50  0001 C CNN
@@
 $EndComp
 $Comp
-L Device:C C49
+L Device:C C51
 U 1 1 614BAEA4
 P 10750 1850
-F 0 "C49" H 10865 1896 50  0000 L CNN
+F 0 "C51" H 10865 1896 50  0000 L CNN
 F 1 "100nF" H 10865 1805 50  0000 L CNN
 F 2 "Capacitor_SMD:C_0402_1005Metric" H 10788 1700 50  0001 C CNN
@@
 	10350 2000 10750 2000
 $Comp
-L power:GND #PWR048
+L power:GND #PWR053
 U 1 1 614C1D2C
 P 7800 2000
-F 0 "#PWR048" H 7800 1750 50  0001 C CNN
+F 0 "#PWR053" H 7800 1750 50  0001 C CNN
 F 1 "GND" H 7805 1827 50  0000 C CNN
 F 2 "" H 7800 2000 50  0001 C CNN
@@
 $EndComp
 Connection ~ 7800 2000
-Text GLabel 7050 2900 2    50   Output ~ 0
-CAM_SHUTTER
-Text GLabel 7050 2800 2    50   Output ~ 0
-CAM_FLASH
 Wire Wire Line
 	6350 3650 7050 3650
@@
 Wire Wire Line
 	7050 3300 7050 3650
-Wire Wire Line
-	7000 3100 7050 3100
+NoConn ~ 7050 2800
+NoConn ~ 7050 2900
+$Comp
+L Device:R R?
+U 1 1 6160EF60
+P 7250 2800
+AR Path="/6108B368/6160EF60" Ref="R?"  Part="1"
+AR Path="/6136B1E7/6160EF60" Ref="R17"  Part="1"
+F 0 "R17" H 7320 2846 50  0000 L CNN
+F 1 "4.7k" H 7320 2755 50  0000 L CNN
+F 2 "Resistor_SMD:R_0402_1005Metric" V 7180 2800 50  0001 C CNN
+F 3 "~" H 7250 2800 50  0001 C CNN
+	1    7250 2800
+	1    0    0    -1
+$EndComp
+Wire Wire Line
+	7000 3100 7250 3100
+Wire Wire Line
+	7250 3100 7250 2950
+Connection ~ 7250 3100
+Wire Wire Line
+	7250 3100 7400 3100
+$Comp
+L power:+1V8 #PWR050
+U 1 1 61625268
+P 7250 2650
+F 0 "#PWR050" H 7250 2500 50  0001 C CNN
+F 1 "+1V8" H 7100 2700 50  0000 C CNN
+F 2 "" H 7250 2650 50  0001 C CNN
+F 3 "" H 7250 2650 50  0001 C CNN
+	1    7250 2650
+	1    0    0    -1
+$EndComp
+$Comp
+L power:+3V3 #PWR043
+U 1 1 6162D84F
+P 2300 2150
+F 0 "#PWR043" H 2300 2000 50  0001 C CNN
+F 1 "+3V3" H 2315 2323 50  0000 C CNN
+F 2 "" H 2300 2150 50  0001 C CNN
+F 3 "" H 2300 2150 50  0001 C CNN
+	1    2300 2150
+	1    0    0    -1
+$EndComp
 $EndSCHEMATC

Commit message: More routing
Parts:
- J2: symbol imucam:54548-2271 -> imucam-rescue:54548-2271-imucam
- U5: symbol imucam:AR0330CM1C00 -> imucam-rescue:AR0330CM1C00-imucam
Changed lines of the file:
@@
 EXTCAM_D3_P
 $Comp
-L imucam:54548-2271 J2
+L imucam-rescue:54548-2271-imucam J2
 U 1 1 60CE4657
 P 4550 4450
+AR Path="/60CE4657" Ref="J2"  Part="1"
+AR Path="/6136B1E7/60CE4657" Ref="J2"  Part="1"
 F 0 "J2" H 4630 3346 50  0000 L CNN
 F 1 "EXTCAM" H 4630 3255 50  0000 L CNN
@@
 	7000 2000 7050 2000
 $Comp
-L imucam:AR0330CM1C00 U5
+L imucam-rescue:AR0330CM1C00-imucam U5
 U 1 1 6136CF1D
 P 6050 2400
