File: kicad/imucam/fpga.sch (KiCad schematic (older format))
At the start: 72 parts

Commit message: Cleaned up footprints
Parts:
- D?: footprint (none) -> Diode_SMD:D_0402_1005Metric
- DONE: renamed from D?; value DONE -> RED
- FB? (x5): footprint (none) -> Inductor_SMD:L_0402_1005Metric
- FPGA_LED1: renamed from D?; value LED0 -> RED
- FPGA_LED2: renamed from D?; value LED1 -> RED
- FPGA_LED3: renamed from D?; value LED2 -> RED
- J?: footprint (none) -> Connector_PinHeader_1.27mm:PinHeader_2x04_P1.27mm_Vertical_SMD
- U?: footprint (none) -> Package_DFN_QFN:QFN-72-1EP_10x10mm_P0.5mm_EP6x6mm_ThermalVias
Connections:
- net labels added: LED3
- net labels removed: LED0
Changed lines of the file:
@@
 F 0 "U?" H 4600 -1250 50  0000 C CNN
 F 1 "LIFCL-17-xSG72" H 5700 -1250 50  0000 C CNN
-F 2 "" H 4550 3000 50  0001 C CNN
+F 2 "Package_DFN_QFN:QFN-72-1EP_10x10mm_P0.5mm_EP6x6mm_ThermalVias" H 4550 3000 50  0001 C CNN
 F 3 "" H 4550 3000 50  0001 C CNN
 	1    5200 3050
@@
 F 0 "FB?" H 5600 1096 50  0000 L CNN
 F 1 "120" H 5600 1005 50  0000 L CNN
-F 2 "" V 5430 1050 50  0001 C CNN
+F 2 "Inductor_SMD:L_0402_1005Metric" V 5430 1050 50  0001 C CNN
 F 3 "~" H 5500 1050 50  0001 C CNN
 	1    5500 1050
@@
 F 0 "FB?" H 4300 6146 50  0000 L CNN
 F 1 "120" H 4300 6055 50  0000 L CNN
-F 2 "" V 4130 6100 50  0001 C CNN
+F 2 "Inductor_SMD:L_0402_1005Metric" V 4130 6100 50  0001 C CNN
 F 3 "~" H 4200 6100 50  0001 C CNN
 	1    4200 6100
@@
 F 0 "FB?" H 3950 6146 50  0000 L CNN
 F 1 "120" H 3950 6055 50  0000 L CNN
-F 2 "" V 3780 6100 50  0001 C CNN
+F 2 "Inductor_SMD:L_0402_1005Metric" V 3780 6100 50  0001 C CNN
 F 3 "~" H 3850 6100 50  0001 C CNN
 	1    3850 6100
@@
 F 0 "FB?" H 3600 6146 50  0000 L CNN
 F 1 "120" H 3600 6055 50  0000 L CNN
-F 2 "" V 3430 6100 50  0001 C CNN
+F 2 "Inductor_SMD:L_0402_1005Metric" V 3430 6100 50  0001 C CNN
 F 3 "~" H 3500 6100 50  0001 C CNN
 	1    3500 6100
@@
 $EndComp
 $Comp
-L Device:LED D?
+L Device:LED DONE
 U 1 1 60F31EC2
 P 7850 5550
-F 0 "D?" V 7889 5432 50  0000 R CNN
-F 1 "DONE" V 7798 5432 50  0000 R CNN
+F 0 "DONE" V 7889 5432 50  0000 R CNN
+F 1 "RED" V 7798 5432 50  0001 R CNN
 F 2 "LED_SMD:LED_0805_2012Metric" H 7850 5550 50  0001 C CNN
 F 3 "~" H 7850 5550 50  0001 C CNN
@@
 F 0 "FB?" H 10000 1046 50  0000 L CNN
 F 1 "120" H 10000 955 50  0000 L CNN
-F 2 "" V 9830 1000 50  0001 C CNN
+F 2 "Inductor_SMD:L_0402_1005Metric" V 9830 1000 50  0001 C CNN
 F 3 "~" H 9900 1000 50  0001 C CNN
 	1    9900 1000
@@
 F 0 "J?" H 10950 5950 50  0000 R CNN
 F 1 "JTAG" H 10350 5950 50  0000 R CNN
-F 2 "" H 10550 5400 50  0001 C CNN
+F 2 "Connector_PinHeader_1.27mm:PinHeader_2x04_P1.27mm_Vertical_SMD" H 10550 5400 50  0001 C CNN
 F 3 "http://infocenter.arm.com/help/topic/com.arm.doc.ddi0314h/DDI0314H_coresight_components_trm.pdf" V 10200 4150 50  0001 C CNN
 	1    10550 5400
@@
 	6100 4100 6600 4100
 Text Label 6200 3800 0    50   ~ 0
-LED0
+LED1
 Text Label 6200 3900 0    50   ~ 0
-LED1
+LED2
 Text Label 6200 4100 0    50   ~ 0
-LED2
+LED3
 $Comp
 L power:GND #PWR?
@@
 $EndComp
 $Comp
-L Device:LED D?
+L Device:LED FPGA_LED1
 U 1 1 61D666BC
 P 1200 4100
-F 0 "D?" V 1239 3982 50  0000 R CNN
-F 1 "LED0" V 1148 3982 50  0000 R CNN
+F 0 "FPGA_LED1" V 1239 3982 50  0000 R CNN
+F 1 "RED" V 1148 3982 50  0001 R CNN
 F 2 "LED_SMD:LED_0805_2012Metric" H 1200 4100 50  0001 C CNN
 F 3 "~" H 1200 4100 50  0001 C CNN
@@
 	550  4450 800  4450
 Text Label 550  4450 0    50   ~ 0
-LED0
+LED1
 $Comp
 L Device:R R?
@@
 $EndComp
 $Comp
-L Device:LED D?
+L Device:LED FPGA_LED2
 U 1 1 61DCEDA1
 P 2150 4100
-F 0 "D?" V 2189 3982 50  0000 R CNN
-F 1 "LED1" V 2098 3982 50  0000 R CNN
+F 0 "FPGA_LED2" V 2189 3982 50  0000 R CNN
+F 1 "RED" V 2098 3982 50  0001 R CNN
 F 2 "LED_SMD:LED_0805_2012Metric" H 2150 4100 50  0001 C CNN
 F 3 "~" H 2150 4100 50  0001 C CNN
@@
 	1500 4450 1750 4450
 Text Label 1500 4450 0    50   ~ 0
-LED1
+LED2
 $Comp
 L Device:R R?
@@
 $EndComp
 $Comp
-L Device:LED D?
+L Device:LED FPGA_LED3
 U 1 1 61DF00D3
 P 3100 4100
-F 0 "D?" V 3139 3982 50  0000 R CNN
-F 1 "LED2" V 3048 3982 50  0000 R CNN
+F 0 "FPGA_LED3" V 3139 3982 50  0000 R CNN
+F 1 "RED" V 3048 3982 50  0001 R CNN
 F 2 "LED_SMD:LED_0805_2012Metric" H 3100 4100 50  0001 C CNN
 F 3 "~" H 3100 4100 50  0001 C CNN
@@
 	2450 4450 2700 4450
 Text Label 2450 4450 0    50   ~ 0
-LED2
+LED3
 $Comp
 L Device:R R?
@@
 F 0 "D?" H 1750 5325 50  0000 C CNN
 F 1 "D_Schottky" H 1750 5324 50  0001 C CNN
-F 2 "" H 1750 5450 50  0001 C CNN
+F 2 "Diode_SMD:D_0402_1005Metric" H 1750 5450 50  0001 C CNN
 F 3 "~" H 1750 5450 50  0001 C CNN
 	1    1750 5450

Commit message: Annotated schematic
Parts:
- gave numbers to parts that had none: 68
- renumbered DONE to DONE1

Commit message: Lots of schematic work
Parts:
- J1: footprint Connector_PinHeader_1.27mm:PinHeader_2x04_P1.27mm_Vertical_SMD -> Connector_PinHeader_1.27mm:PinHeader_2x05_P1.27mm_Vertical_SMD

Commit message: More work on PCB
Parts:
- R14, R2, R3, R4: value 1k -> 100
Changed lines of the file:
@@
 P 7850 5250
 F 0 "R14" H 7920 5296 50  0000 L CNN
-F 1 "1k" H 7920 5205 50  0000 L CNN
+F 1 "100" H 7920 5205 50  0000 L CNN
 F 2 "Resistor_SMD:R_0402_1005Metric" V 7780 5250 50  0001 C CNN
 F 3 "~" H 7850 5250 50  0001 C CNN
@@
 P 1200 3800
 F 0 "R2" H 1270 3846 50  0000 L CNN
-F 1 "1k" H 1270 3755 50  0000 L CNN
+F 1 "100" H 1270 3755 50  0000 L CNN
 F 2 "Resistor_SMD:R_0402_1005Metric" V 1130 3800 50  0001 C CNN
 F 3 "~" H 1200 3800 50  0001 C CNN
@@
 P 2150 3800
 F 0 "R3" H 2220 3846 50  0000 L CNN
-F 1 "1k" H 2220 3755 50  0000 L CNN
+F 1 "100" H 2220 3755 50  0000 L CNN
 F 2 "Resistor_SMD:R_0402_1005Metric" V 2080 3800 50  0001 C CNN
 F 3 "~" H 2150 3800 50  0001 C CNN
@@
 P 3100 3800
 F 0 "R4" H 3170 3846 50  0000 L CNN
-F 1 "1k" H 3170 3755 50  0000 L CNN
+F 1 "100" H 3170 3755 50  0000 L CNN
 F 2 "Resistor_SMD:R_0402_1005Metric" V 3030 3800 50  0001 C CNN
 F 3 "~" H 3100 3800 50  0001 C CNN

Commit message: Through-hole JTAG
Parts:
- J1: footprint Connector_PinHeader_1.27mm:PinHeader_2x05_P1.27mm_Vertical_SMD -> Connector_PinHeader_1.27mm:PinHeader_2x05_P1.27mm_Vertical
Changed lines of the file:
@@
 F 0 "J1" H 10950 5950 50  0000 R CNN
 F 1 "JTAG" H 10350 5950 50  0000 R CNN
-F 2 "Connector_PinHeader_1.27mm:PinHeader_2x05_P1.27mm_Vertical_SMD" H 10550 5400 50  0001 C CNN
+F 2 "Connector_PinHeader_1.27mm:PinHeader_2x05_P1.27mm_Vertical" H 10550 5400 50  0001 C CNN
 F 3 "http://infocenter.arm.com/help/topic/com.arm.doc.ddi0314h/DDI0314H_coresight_components_trm.pdf" V 10200 4150 50  0001 C CNN
 	1    10550 5400

Commit message: Slightly more progress on current measurement
Parts:
- renumbered C6 to C1, C34 to C11, C1 to C12, C11 to C13, C24 to C14, C35 to C15, C36 to C16, C2 to C17, C12 to C18, C23 to C2, C25 to C20, C27 to C21, C29 to C22, C37 to C23, C3 to C24, C13 to C25, C20 to C26, C26 to C27, C30 to C29, C7 to C3, C14 to C30, C15 to C31, C16 to C32, C17 to C33, C18 to C34, C4 to C35, C5 to C36, C21 to C37, C31 to C4, C8 to C5, C32 to C6, C9 to C7, C22 to C8, C33 to C9, FB3 to FB1, FB4 to FB2, FB5 to FB3, FB2 to FB4, FB1 to FB5, R6 to R1, R1 to R11, R5 to R12, R11 to R13, R12 to R14, R13 to R15, R7 to R3, R3 to R4, R8 to R5, R4 to R6, R9 to R7, R15 to R8, R14 to R9

Commit message: Turns out, we need level translators
Parts:
- renumbered C12 to C1, C13 to C11, C18 to C12, C25 to C13, C30 to C14, C31 to C15, C32 to C16, C33 to C17, C34 to C18, C17 to C2, C26 to C20, C37 to C21, C8 to C22, C2 to C23, C14 to C24, C20 to C25, C27 to C26, C21 to C27, C22 to C29, C24 to C3, C29 to C30, C4 to C31, C6 to C32, C9 to C33, C11 to C34, C15 to C35, C16 to C36, C23 to C37, C35 to C4, C36 to C5, C1 to C6, C3 to C7, C5 to C8, C7 to C9, FB5 to FB1, FB4 to FB2, FB1 to FB3, FB2 to FB4, FB3 to FB5, R11 to R1, R13 to R11, R14 to R12, R15 to R13, R9 to R14, R8 to R15, R4 to R3, R6 to R4, R12 to R5, R1 to R6, R3 to R7, R5 to R8, R7 to R9

Commit message: WIP of remapping nucleo pinout for pcb routing
Parts:
- renumbered C6 to C1, C34 to C11, C1 to C12, C11 to C13, C24 to C14, C35 to C15, C36 to C16, C2 to C17, C12 to C18, C23 to C2, C25 to C20, C27 to C21, C29 to C22, C37 to C23, C3 to C24, C13 to C25, C20 to C26, C26 to C27, C30 to C29, C7 to C3, C14 to C30, C15 to C31, C16 to C32, C17 to C33, C18 to C34, C21 to C35, C4 to C36, C5 to C37, C31 to C4, C8 to C5, C32 to C6, C9 to C7, C22 to C8, C33 to C9, FB3 to FB1, FB4 to FB2, FB5 to FB3, FB2 to FB4, FB1 to FB5, R6 to R1, R1 to R11, R5 to R12, R11 to R13, R12 to R14, R13 to R15, R7 to R3, R3 to R4, R8 to R5, R4 to R6, R9 to R7, R15 to R8, R14 to R9
Connections:
- net labels added: +3V3
- net labels removed: +3.3V
- wire segments 213 -> 216
