File: kicad/imucam/hdmi.sch (KiCad schematic (older format))
At the start: 24 parts

Commit message: Cleaned up footprints
Parts:
- C?: footprint (none) -> Capacitor_SMD:C_0603_1608Metric
- C? (x11): footprint (none) -> Capacitor_SMD:C_0402_1005Metric
- J?: footprint (none) -> Connector_HDMI:HDMI_A_Contact_Technology_HDMI-19APL2_Horizontal
- R? (x9): footprint (none) -> Resistor_SMD:R_0402_1005Metric
- U?: footprint (none) -> Package_DFN_QFN:QFN-32-1EP_5x5mm_P0.5mm_EP3.6x3.6mm
Changed lines of the file:
@@
 F 0 "U?" H 6650 5250 50  0000 C CNN
 F 1 "PTN3366" H 5800 5250 50  0000 C CNN
-F 2 "" H 6350 4250 50  0001 C CNN
+F 2 "Package_DFN_QFN:QFN-32-1EP_5x5mm_P0.5mm_EP3.6x3.6mm" H 6350 4250 50  0001 C CNN
 F 3 "" H 6350 4250 50  0001 C CNN
 	1    6200 4150
@@
 F 0 "C?" H 5465 2796 50  0000 L CNN
 F 1 "10uF" H 5465 2705 50  0000 L CNN
-F 2 "" H 5388 2600 50  0001 C CNN
+F 2 "Capacitor_SMD:C_0603_1608Metric" H 5388 2600 50  0001 C CNN
 F 3 "~" H 5350 2750 50  0001 C CNN
 	1    5350 2750
@@
 F 0 "C?" H 5915 2796 50  0000 L CNN
 F 1 "100nF" H 5915 2705 50  0000 L CNN
-F 2 "" H 5838 2600 50  0001 C CNN
+F 2 "Capacitor_SMD:C_0402_1005Metric" H 5838 2600 50  0001 C CNN
 F 3 "~" H 5800 2750 50  0001 C CNN
 	1    5800 2750
@@
 F 0 "R?" H 7120 4796 50  0000 L CNN
 F 1 "12.4k 1%" H 7120 4705 50  0000 L CNN
-F 2 "" V 6980 4750 50  0001 C CNN
+F 2 "Resistor_SMD:R_0402_1005Metric" V 6980 4750 50  0001 C CNN
 F 3 "~" H 7050 4750 50  0001 C CNN
 	1    7050 4750
@@
 F 0 "C?" V 4650 3150 50  0000 C CNN
 F 1 "100nF" V 4750 3100 50  0000 C CNN
-F 2 "" H 4738 3100 50  0001 C CNN
+F 2 "Capacitor_SMD:C_0402_1005Metric" H 4738 3100 50  0001 C CNN
 F 3 "~" H 4700 3250 50  0001 C CNN
 	1    4700 3250
@@
 F 0 "C?" V 5000 3250 50  0000 C CNN
 F 1 "100nF" V 5100 3200 50  0000 C CNN
-F 2 "" H 5088 3200 50  0001 C CNN
+F 2 "Capacitor_SMD:C_0402_1005Metric" H 5088 3200 50  0001 C CNN
 F 3 "~" H 5050 3350 50  0001 C CNN
 	1    5050 3350
@@
 F 0 "C?" V 4650 3350 50  0000 C CNN
 F 1 "100nF" V 4750 3300 50  0000 C CNN
-F 2 "" H 4738 3300 50  0001 C CNN
+F 2 "Capacitor_SMD:C_0402_1005Metric" H 4738 3300 50  0001 C CNN
 F 3 "~" H 4700 3450 50  0001 C CNN
 	1    4700 3450
@@
 F 0 "C?" V 5000 3450 50  0000 C CNN
 F 1 "100nF" V 5100 3400 50  0000 C CNN
-F 2 "" H 5088 3400 50  0001 C CNN
+F 2 "Capacitor_SMD:C_0402_1005Metric" H 5088 3400 50  0001 C CNN
 F 3 "~" H 5050 3550 50  0001 C CNN
 	1    5050 3550
@@
 F 0 "C?" V 4650 3550 50  0000 C CNN
 F 1 "100nF" V 4750 3500 50  0000 C CNN
-F 2 "" H 4738 3500 50  0001 C CNN
+F 2 "Capacitor_SMD:C_0402_1005Metric" H 4738 3500 50  0001 C CNN
 F 3 "~" H 4700 3650 50  0001 C CNN
 	1    4700 3650
@@
 F 0 "C?" V 5000 3650 50  0000 C CNN
 F 1 "100nF" V 5100 3600 50  0000 C CNN
-F 2 "" H 5088 3600 50  0001 C CNN
+F 2 "Capacitor_SMD:C_0402_1005Metric" H 5088 3600 50  0001 C CNN
 F 3 "~" H 5050 3750 50  0001 C CNN
 	1    5050 3750
@@
 F 0 "C?" V 4650 3750 50  0000 C CNN
 F 1 "100nF" V 4750 3700 50  0000 C CNN
-F 2 "" H 4738 3700 50  0001 C CNN
+F 2 "Capacitor_SMD:C_0402_1005Metric" H 4738 3700 50  0001 C CNN
 F 3 "~" H 4700 3850 50  0001 C CNN
 	1    4700 3850
@@
 F 0 "C?" V 5000 3850 50  0000 C CNN
 F 1 "100nF" V 5100 3800 50  0000 C CNN
-F 2 "" H 5088 3800 50  0001 C CNN
+F 2 "Capacitor_SMD:C_0402_1005Metric" H 5088 3800 50  0001 C CNN
 F 3 "~" H 5050 3950 50  0001 C CNN
 	1    5050 3950
@@
 F 0 "R?" H 8120 4196 50  0000 L CNN
 F 1 "4.7k" H 8120 4105 50  0000 L CNN
-F 2 "" V 7980 4150 50  0001 C CNN
+F 2 "Resistor_SMD:R_0402_1005Metric" V 7980 4150 50  0001 C CNN
 F 3 "~" H 8050 4150 50  0001 C CNN
 	1    8050 4150
@@
 F 0 "R?" H 7820 4196 50  0000 L CNN
 F 1 "4.7k" H 7820 4105 50  0000 L CNN
-F 2 "" V 7680 4150 50  0001 C CNN
+F 2 "Resistor_SMD:R_0402_1005Metric" V 7680 4150 50  0001 C CNN
 F 3 "~" H 7750 4150 50  0001 C CNN
 	1    7750 4150
@@
 F 0 "J?" H 9180 4096 50  0000 L CNN
 F 1 "HDMI" H 9180 4005 50  0000 L CNN
-F 2 "" H 8775 4050 50  0001 C CNN
+F 2 "Connector_HDMI:HDMI_A_Contact_Technology_HDMI-19APL2_Horizontal" H 8775 4050 50  0001 C CNN
 F 3 "https://en.wikipedia.org/wiki/HDMI" H 8775 4050 50  0001 C CNN
 	1    8750 4050
@@
 F 0 "R?" H 3470 4446 50  0000 L CNN
 F 1 "4.7k" H 3470 4355 50  0000 L CNN
-F 2 "" V 3330 4400 50  0001 C CNN
+F 2 "Resistor_SMD:R_0402_1005Metric" V 3330 4400 50  0001 C CNN
 F 3 "~" H 3400 4400 50  0001 C CNN
 	1    3400 4400
@@
 F 0 "R?" H 3170 4446 50  0000 L CNN
 F 1 "4.7k" H 3170 4355 50  0000 L CNN
-F 2 "" V 3030 4400 50  0001 C CNN
+F 2 "Resistor_SMD:R_0402_1005Metric" V 3030 4400 50  0001 C CNN
 F 3 "~" H 3100 4400 50  0001 C CNN
 	1    3100 4400
@@
 F 0 "C?" H 6665 2396 50  0000 L CNN
 F 1 "100nF" H 6665 2305 50  0000 L CNN
-F 2 "" H 6588 2200 50  0001 C CNN
+F 2 "Capacitor_SMD:C_0402_1005Metric" H 6588 2200 50  0001 C CNN
 F 3 "~" H 6550 2350 50  0001 C CNN
 	1    6550 2350
@@
 F 0 "C?" H 7765 2396 50  0000 L CNN
 F 1 "100nF" H 7765 2305 50  0000 L CNN
-F 2 "" H 7688 2200 50  0001 C CNN
+F 2 "Capacitor_SMD:C_0402_1005Metric" H 7688 2200 50  0001 C CNN
 F 3 "~" H 7650 2350 50  0001 C CNN
 	1    7650 2350
@@
 F 0 "R?" H 4370 4446 50  0000 L CNN
 F 1 "10k" H 4370 4355 50  0000 L CNN
-F 2 "" V 4230 4400 50  0001 C CNN
+F 2 "Resistor_SMD:R_0402_1005Metric" V 4230 4400 50  0001 C CNN
 F 3 "~" H 4300 4400 50  0001 C CNN
 	1    4300 4400
@@
 F 0 "R?" H 4070 4446 50  0000 L CNN
 F 1 "10k" H 4070 4355 50  0000 L CNN
-F 2 "" V 3930 4400 50  0001 C CNN
+F 2 "Resistor_SMD:R_0402_1005Metric" V 3930 4400 50  0001 C CNN
 F 3 "~" H 4000 4400 50  0001 C CNN
 	1    4000 4400
@@
 F 0 "R?" H 3770 5446 50  0000 L CNN
 F 1 "10k" H 3770 5355 50  0000 L CNN
-F 2 "" V 3630 5400 50  0001 C CNN
+F 2 "Resistor_SMD:R_0402_1005Metric" V 3630 5400 50  0001 C CNN
 F 3 "~" H 3700 5400 50  0001 C CNN
 	1    3700 5400
@@
 F 0 "R?" H 4670 4446 50  0000 L CNN
 F 1 "10k" H 4670 4355 50  0000 L CNN
-F 2 "" V 4530 4400 50  0001 C CNN
+F 2 "Resistor_SMD:R_0402_1005Metric" V 4530 4400 50  0001 C CNN
 F 3 "~" H 4600 4400 50  0001 C CNN
 	1    4600 4400

Commit message: Annotated schematic
Parts:
- gave numbers to parts that had none: 24
Changed lines of the file:
@@
 $EndDescr
 $Comp
-L imucam:PTN3366 U?
+L imucam:PTN3366 U10
 U 1 1 61A33450
 P 6200 4150
-F 0 "U?" H 6650 5250 50  0000 C CNN
+F 0 "U10" H 6650 5250 50  0000 C CNN
 F 1 "PTN3366" H 5800 5250 50  0000 C CNN
 F 2 "Package_DFN_QFN:QFN-32-1EP_5x5mm_P0.5mm_EP3.6x3.6mm" H 6350 4250 50  0001 C CNN
@@
 $EndComp
 $Comp
-L power:GND #PWR?
+L power:GND #PWR0180
 U 1 1 61A343C7
 P 6200 5050
-F 0 "#PWR?" H 6200 4800 50  0001 C CNN
+F 0 "#PWR0180" H 6200 4800 50  0001 C CNN
 F 1 "GND" H 6205 4877 50  0000 C CNN
 F 2 "" H 6200 5050 50  0001 C CNN
@@
 $EndComp
 $Comp
-L power:+3.3V #PWR?
+L power:+3.3V #PWR0181
 U 1 1 61A34AA9
 P 6200 2600
-F 0 "#PWR?" H 6200 2450 50  0001 C CNN
+F 0 "#PWR0181" H 6200 2450 50  0001 C CNN
 F 1 "+3.3V" H 6215 2773 50  0000 C CNN
 F 2 "" H 6200 2600 50  0001 C CNN
@@
 $EndComp
 $Comp
-L Device:C C?
+L Device:C C67
 U 1 1 61A3662C
 P 5350 2750
-F 0 "C?" H 5465 2796 50  0000 L CNN
+F 0 "C67" H 5465 2796 50  0000 L CNN
 F 1 "10uF" H 5465 2705 50  0000 L CNN
 F 2 "Capacitor_SMD:C_0603_1608Metric" H 5388 2600 50  0001 C CNN
@@
 $EndComp
 $Comp
-L Device:C C?
+L Device:C C68
 U 1 1 61A3695C
 P 5800 2750
-F 0 "C?" H 5915 2796 50  0000 L CNN
+F 0 "C68" H 5915 2796 50  0000 L CNN
 F 1 "100nF" H 5915 2705 50  0000 L CNN
 F 2 "Capacitor_SMD:C_0402_1005Metric" H 5838 2600 50  0001 C CNN
@@
 	5800 2900 5350 2900
 $Comp
-L power:GND #PWR?
+L power:GND #PWR0182
 U 1 1 61A38134
 P 5350 2900
-F 0 "#PWR?" H 5350 2650 50  0001 C CNN
+F 0 "#PWR0182" H 5350 2650 50  0001 C CNN
 F 1 "GND" H 5355 2727 50  0000 C CNN
 F 2 "" H 5350 2900 50  0001 C CNN
@@
 Connection ~ 6200 2600
 $Comp
-L Device:R R?
+L Device:R R37
 U 1 1 61A397D5
 P 7050 4750
-F 0 "R?" H 7120 4796 50  0000 L CNN
+F 0 "R37" H 7120 4796 50  0000 L CNN
 F 1 "12.4k 1%" H 7120 4705 50  0000 L CNN
 F 2 "Resistor_SMD:R_0402_1005Metric" V 6980 4750 50  0001 C CNN
@@
 HDMI_HPD
 $Comp
-L Device:C C?
+L Device:C C69
 U 1 1 61A78AD4
 P 4700 3250
-F 0 "C?" V 4650 3150 50  0000 C CNN
+F 0 "C69" V 4650 3150 50  0000 C CNN
 F 1 "100nF" V 4750 3100 50  0000 C CNN
 F 2 "Capacitor_SMD:C_0402_1005Metric" H 4738 3100 50  0001 C CNN
@@
 $EndComp
 $Comp
-L Device:C C?
+L Device:C C70
 U 1 1 61A797BD
 P 5050 3350
-F 0 "C?" V 5000 3250 50  0000 C CNN
+F 0 "C70" V 5000 3250 50  0000 C CNN
 F 1 "100nF" V 5100 3200 50  0000 C CNN
 F 2 "Capacitor_SMD:C_0402_1005Metric" H 5088 3200 50  0001 C CNN
@@
 $EndComp
 $Comp
-L Device:C C?
+L Device:C C71
 U 1 1 61A7A48F
 P 4700 3450
-F 0 "C?" V 4650 3350 50  0000 C CNN
+F 0 "C71" V 4650 3350 50  0000 C CNN
 F 1 "100nF" V 4750 3300 50  0000 C CNN
 F 2 "Capacitor_SMD:C_0402_1005Metric" H 4738 3300 50  0001 C CNN
@@
 $EndComp
 $Comp
-L Device:C C?
+L Device:C C72
 U 1 1 61A7AA31
 P 5050 3550
-F 0 "C?" V 5000 3450 50  0000 C CNN
+F 0 "C72" V 5000 3450 50  0000 C CNN
 F 1 "100nF" V 5100 3400 50  0000 C CNN
 F 2 "Capacitor_SMD:C_0402_1005Metric" H 5088 3400 50  0001 C CNN
@@
 $EndComp
 $Comp
-L Device:C C?
+L Device:C C73
 U 1 1 61A7AEB6
 P 4700 3650
-F 0 "C?" V 4650 3550 50  0000 C CNN
+F 0 "C73" V 4650 3550 50  0000 C CNN
 F 1 "100nF" V 4750 3500 50  0000 C CNN
 F 2 "Capacitor_SMD:C_0402_1005Metric" H 4738 3500 50  0001 C CNN
@@
 $EndComp
 $Comp
-L Device:C C?
+L Device:C C74
 U 1 1 61A7B399
 P 5050 3750
-F 0 "C?" V 5000 3650 50  0000 C CNN
+F 0 "C74" V 5000 3650 50  0000 C CNN
 F 1 "100nF" V 5100 3600 50  0000 C CNN
 F 2 "Capacitor_SMD:C_0402_1005Metric" H 5088 3600 50  0001 C CNN
@@
 $EndComp
 $Comp
-L Device:C C?
+L Device:C C75
 U 1 1 61A7BB72
 P 4700 3850
-F 0 "C?" V 4650 3750 50  0000 C CNN
+F 0 "C75" V 4650 3750 50  0000 C CNN
 F 1 "100nF" V 4750 3700 50  0000 C CNN
 F 2 "Capacitor_SMD:C_0402_1005Metric" H 4738 3700 50  0001 C CNN
@@
 $EndComp
 $Comp
-L Device:C C?
+L Device:C C76
 U 1 1 61A7C0F4
 P 5050 3950
-F 0 "C?" V 5000 3850 50  0000 C CNN
+F 0 "C76" V 5000 3850 50  0000 C CNN
 F 1 "100nF" V 5100 3800 50  0000 C CNN
 F 2 "Capacitor_SMD:C_0402_1005Metric" H 5088 3800 50  0001 C CNN
@@
 	7750 4350 7750 4300
 $Comp
-L Device:R R?
+L Device:R R31
 U 1 1 61AEEAD1
 P 8050 4150
-F 0 "R?" H 8120 4196 50  0000 L CNN
+F 0 "R31" H 8120 4196 50  0000 L CNN
 F 1 "4.7k" H 8120 4105 50  0000 L CNN
 F 2 "Resistor_SMD:R_0402_1005Metric" V 7980 4150 50  0001 C CNN
@@
 $EndComp
 $Comp
-L Device:R R?
+L Device:R R30
 U 1 1 61AEDD4D
 P 7750 4150
-F 0 "R?" H 7820 4196 50  0000 L CNN
+F 0 "R30" H 7820 4196 50  0000 L CNN
 F 1 "4.7k" H 7820 4105 50  0000 L CNN
 F 2 "Resistor_SMD:R_0402_1005Metric" V 7680 4150 50  0001 C CNN
@@
 	8550 5150 8550 5200
 $Comp
-L power:GND #PWR?
+L power:GND #PWR0183
 U 1 1 61A6FC85
 P 8750 5200
-F 0 "#PWR?" H 8750 4950 50  0001 C CNN
+F 0 "#PWR0183" H 8750 4950 50  0001 C CNN
 F 1 "GND" H 8755 5027 50  0000 C CNN
 F 2 "" H 8750 5200 50  0001 C CNN
@@
 $EndComp
 $Comp
-L Connector:HDMI_A J?
+L Connector:HDMI_A J8
 U 1 1 61A5E9CE
 P 8750 4050
-F 0 "J?" H 9180 4096 50  0000 L CNN
+F 0 "J8" H 9180 4096 50  0000 L CNN
 F 1 "HDMI" H 9180 4005 50  0000 L CNN
 F 2 "Connector_HDMI:HDMI_A_Contact_Technology_HDMI-19APL2_Horizontal" H 8775 4050 50  0001 C CNN
@@
 HDMI_OE
 $Comp
-L Device:R R?
+L Device:R R33
 U 1 1 61B50DA8
 P 3400 4400
-F 0 "R?" H 3470 4446 50  0000 L CNN
+F 0 "R33" H 3470 4446 50  0000 L CNN
 F 1 "4.7k" H 3470 4355 50  0000 L CNN
 F 2 "Resistor_SMD:R_0402_1005Metric" V 3330 4400 50  0001 C CNN
@@
 $EndComp
 $Comp
-L Device:R R?
+L Device:R R32
 U 1 1 61B511BB
 P 3100 4400
-F 0 "R?" H 3170 4446 50  0000 L CNN
+F 0 "R32" H 3170 4446 50  0000 L CNN
 F 1 "4.7k" H 3170 4355 50  0000 L CNN
 F 2 "Resistor_SMD:R_0402_1005Metric" V 3030 4400 50  0001 C CNN
@@
 Connection ~ 3400 4750
 $Comp
-L power:+3.3V #PWR?
+L power:+3.3V #PWR0184
 U 1 1 61B620D7
 P 3100 4250
-F 0 "#PWR?" H 3100 4100 50  0001 C CNN
+F 0 "#PWR0184" H 3100 4100 50  0001 C CNN
 F 1 "+3.3V" H 3115 4423 50  0000 C CNN
 F 2 "" H 3100 4250 50  0001 C CNN
@@
 	5150 4500 5150 4850
 $Comp
-L imucam:AP2331 U?
+L imucam:AP2331 U9
 U 1 1 61B93326
 P 7200 2250
-F 0 "U?" H 7200 2665 50  0000 C CNN
+F 0 "U9" H 7200 2665 50  0000 C CNN
 F 1 "AP2331" H 7200 2574 50  0000 C CNN
 F 2 "Package_TO_SOT_SMD:SOT-23" H 7200 1800 50  0001 C CNN
@@
 $EndComp
 $Comp
-L power:+5V #PWR?
+L power:+5V #PWR0185
 U 1 1 61B94788
 P 6550 2150
-F 0 "#PWR?" H 6550 2000 50  0001 C CNN
+F 0 "#PWR0185" H 6550 2000 50  0001 C CNN
 F 1 "+5V" H 6565 2323 50  0000 C CNN
 F 2 "" H 6550 2150 50  0001 C CNN
@@
 	6850 2150 6550 2150
 $Comp
-L power:GND #PWR?
+L power:GND #PWR0186
 U 1 1 61B984B1
 P 7200 2550
-F 0 "#PWR?" H 7200 2300 50  0001 C CNN
+F 0 "#PWR0186" H 7200 2300 50  0001 C CNN
 F 1 "GND" H 7205 2377 50  0000 C CNN
 F 2 "" H 7200 2550 50  0001 C CNN
@@
 	8050 2150 8050 2850
 $Comp
-L Device:C C?
+L Device:C C65
 U 1 1 61B9C87B
 P 6550 2350
-F 0 "C?" H 6665 2396 50  0000 L CNN
+F 0 "C65" H 6665 2396 50  0000 L CNN
 F 1 "100nF" H 6665 2305 50  0000 L CNN
 F 2 "Capacitor_SMD:C_0402_1005Metric" H 6588 2200 50  0001 C CNN
@@
 $EndComp
 $Comp
-L Device:C C?
+L Device:C C66
 U 1 1 61B9D2E1
 P 7650 2350
-F 0 "C?" H 7765 2396 50  0000 L CNN
+F 0 "C66" H 7765 2396 50  0000 L CNN
 F 1 "100nF" H 7765 2305 50  0000 L CNN
 F 2 "Capacitor_SMD:C_0402_1005Metric" H 7688 2200 50  0001 C CNN
@@
 Connection ~ 6550 2150
 $Comp
-L Device:R R?
+L Device:R R35
 U 1 1 61C43F79
 P 4300 4400
-F 0 "R?" H 4370 4446 50  0000 L CNN
+F 0 "R35" H 4370 4446 50  0000 L CNN
 F 1 "10k" H 4370 4355 50  0000 L CNN
 F 2 "Resistor_SMD:R_0402_1005Metric" V 4230 4400 50  0001 C CNN
@@
 $EndComp
 $Comp
-L Device:R R?
+L Device:R R34
 U 1 1 61C443EB
 P 4000 4400
-F 0 "R?" H 4070 4446 50  0000 L CNN
+F 0 "R34" H 4070 4446 50  0000 L CNN
 F 1 "10k" H 4070 4355 50  0000 L CNN
 F 2 "Resistor_SMD:R_0402_1005Metric" V 3930 4400 50  0001 C CNN
@@
 	3400 4250 4000 4250
 $Comp
-L Device:R R?
+L Device:R R38
 U 1 1 61FD3CEB
 P 3700 5400
-F 0 "R?" H 3770 5446 50  0000 L CNN
+F 0 "R38" H 3770 5446 50  0000 L CNN
 F 1 "10k" H 3770 5355 50  0000 L CNN
 F 2 "Resistor_SMD:R_0402_1005Metric" V 3630 5400 50  0001 C CNN
@@
 $EndComp
 $Comp
-L power:GND #PWR?
+L power:GND #PWR0187
 U 1 1 61FD40D4
 P 3700 5550
-F 0 "#PWR?" H 3700 5300 50  0001 C CNN
+F 0 "#PWR0187" H 3700 5300 50  0001 C CNN
 F 1 "GND" H 3705 5377 50  0000 C CNN
 F 2 "" H 3700 5550 50  0001 C CNN
@@
 Connection ~ 4300 5050
 $Comp
-L Device:R R?
+L Device:R R36
 U 1 1 6200261D
 P 4600 4400
-F 0 "R?" H 4670 4446 50  0000 L CNN
+F 0 "R36" H 4670 4446 50  0000 L CNN
 F 1 "10k" H 4670 4355 50  0000 L CNN
 F 2 "Resistor_SMD:R_0402_1005Metric" V 4530 4400 50  0001 C CNN

Commit message: Lots of schematic work
Parts:
- J8: footprint Connector_HDMI:HDMI_A_Contact_Technology_HDMI-19APL2_Horizontal -> imucam:CnC_2000-1-2-41-00-BK; symbol Connector:HDMI_A -> Connector:HDMI_A_1.4
- renumbered R30 to R36, R31 to R37, R32 to R38, R33 to R39, R34 to R40, R35 to R41, R36 to R42, R37 to R43, R38 to R44
Connections:
- net labels added: CK_N, CK_P, D0_N, D0_P, D1_N, D1_P, D2_N, D2_P
Changed lines of the file:
@@
 $EndComp
 $Comp
-L power:GND #PWR0180
+L power:GND #PWR088
 U 1 1 61A343C7
 P 6200 5050
-F 0 "#PWR0180" H 6200 4800 50  0001 C CNN
+F 0 "#PWR088" H 6200 4800 50  0001 C CNN
 F 1 "GND" H 6205 4877 50  0000 C CNN
 F 2 "" H 6200 5050 50  0001 C CNN
@@
 $EndComp
 $Comp
-L power:+3.3V #PWR0181
+L power:+3.3V #PWR085
 U 1 1 61A34AA9
 P 6200 2600
-F 0 "#PWR0181" H 6200 2450 50  0001 C CNN
+F 0 "#PWR085" H 6200 2450 50  0001 C CNN
 F 1 "+3.3V" H 6215 2773 50  0000 C CNN
 F 2 "" H 6200 2600 50  0001 C CNN
@@
 	5800 2900 5350 2900
 $Comp
-L power:GND #PWR0182
+L power:GND #PWR086
 U 1 1 61A38134
 P 5350 2900
-F 0 "#PWR0182" H 5350 2650 50  0001 C CNN
+F 0 "#PWR086" H 5350 2650 50  0001 C CNN
 F 1 "GND" H 5355 2727 50  0000 C CNN
 F 2 "" H 5350 2900 50  0001 C CNN
@@
 Connection ~ 6200 2600
 $Comp
-L Device:R R37
+L Device:R R43
 U 1 1 61A397D5
 P 7050 4750
-F 0 "R37" H 7120 4796 50  0000 L CNN
+F 0 "R43" H 7120 4796 50  0000 L CNN
 F 1 "12.4k 1%" H 7120 4705 50  0000 L CNN
 F 2 "Resistor_SMD:R_0402_1005Metric" V 6980 4750 50  0001 C CNN
@@
 Wire Wire Line
 	4900 3350 4350 3350
+Text GLabel 4350 3850 0    50   Input ~ 0
+HDMI_D2_P
+Text GLabel 4350 3950 0    50   Input ~ 0
+HDMI_D2_N
+Text GLabel 4350 3650 0    50   Input ~ 0
+HDMI_D1_P
+Text GLabel 4350 3750 0    50   Input ~ 0
+HDMI_D1_N
+Text GLabel 4350 3450 0    50   Input ~ 0
+HDMI_D0_P
+Text GLabel 4350 3550 0    50   Input ~ 0
+HDMI_D0_N
 Text GLabel 4350 3250 0    50   Input ~ 0
-HDMI_D2_P
+HDMI_CK_P
 Text GLabel 4350 3350 0    50   Input ~ 0
-HDMI_D2_N
-Text GLabel 4350 3450 0    50   Input ~ 0
-HDMI_D1_P
-Text GLabel 4350 3550 0    50   Input ~ 0
-HDMI_D1_N
-Text GLabel 4350 3650 0    50   Input ~ 0
-HDMI_D0_P
-Text GLabel 4350 3750 0    50   Input ~ 0
-HDMI_D0_N
-Text GLabel 4350 3850 0    50   Input ~ 0
-HDMI_CK_P
-Text GLabel 4350 3950 0    50   Input ~ 0
 HDMI_CK_N
 Wire Wire Line
@@
 	7750 4350 7750 4300
 $Comp
-L Device:R R31
+L Device:R R37
 U 1 1 61AEEAD1
 P 8050 4150
-F 0 "R31" H 8120 4196 50  0000 L CNN
+F 0 "R37" H 8120 4196 50  0000 L CNN
 F 1 "4.7k" H 8120 4105 50  0000 L CNN
 F 2 "Resistor_SMD:R_0402_1005Metric" V 7980 4150 50  0001 C CNN
@@
 $EndComp
 $Comp
-L Device:R R30
+L Device:R R36
 U 1 1 61AEDD4D
 P 7750 4150
-F 0 "R30" H 7820 4196 50  0000 L CNN
+F 0 "R36" H 7820 4196 50  0000 L CNN
 F 1 "4.7k" H 7820 4105 50  0000 L CNN
 F 2 "Resistor_SMD:R_0402_1005Metric" V 7680 4150 50  0001 C CNN
@@
 	8550 5150 8550 5200
 $Comp
-L power:GND #PWR0183
+L power:GND #PWR089
 U 1 1 61A6FC85
 P 8750 5200
-F 0 "#PWR0183" H 8750 4950 50  0001 C CNN
+F 0 "#PWR089" H 8750 4950 50  0001 C CNN
 F 1 "GND" H 8755 5027 50  0000 C CNN
 F 2 "" H 8750 5200 50  0001 C CNN
@@
 $EndComp
 $Comp
-L Connector:HDMI_A J8
+L Connector:HDMI_A_1.4 J8
 U 1 1 61A5E9CE
 P 8750 4050
 F 0 "J8" H 9180 4096 50  0000 L CNN
 F 1 "HDMI" H 9180 4005 50  0000 L CNN
-F 2 "Connector_HDMI:HDMI_A_Contact_Technology_HDMI-19APL2_Horizontal" H 8775 4050 50  0001 C CNN
+F 2 "imucam:CnC_2000-1-2-41-00-BK" H 8775 4050 50  0001 C CNN
 F 3 "https://en.wikipedia.org/wiki/HDMI" H 8775 4050 50  0001 C CNN
 	1    8750 4050
@@
 Wire Wire Line
 	7600 4150 6800 4150
-Wire Wire Line
-	6800 3250 8350 3250
-Wire Wire Line
-	6800 3350 8350 3350
-Wire Wire Line
-	6800 3450 8350 3450
-Wire Wire Line
-	6800 3550 8350 3550
-Wire Wire Line
-	6800 3650 8350 3650
-Wire Wire Line
-	6800 3750 8350 3750
-Wire Wire Line
-	6800 3850 8350 3850
-Wire Wire Line
-	6800 3950 8350 3950
 Wire Wire Line
 	7600 4750 8350 4750
@@
 HDMI_OE
 $Comp
-L Device:R R33
+L Device:R R39
 U 1 1 61B50DA8
 P 3400 4400
-F 0 "R33" H 3470 4446 50  0000 L CNN
+F 0 "R39" H 3470 4446 50  0000 L CNN
 F 1 "4.7k" H 3470 4355 50  0000 L CNN
 F 2 "Resistor_SMD:R_0402_1005Metric" V 3330 4400 50  0001 C CNN
@@
 $EndComp
 $Comp
-L Device:R R32
+L Device:R R38
 U 1 1 61B511BB
 P 3100 4400
-F 0 "R32" H 3170 4446 50  0000 L CNN
+F 0 "R38" H 3170 4446 50  0000 L CNN
 F 1 "4.7k" H 3170 4355 50  0000 L CNN
 F 2 "Resistor_SMD:R_0402_1005Metric" V 3030 4400 50  0001 C CNN
@@
 Connection ~ 3400 4750
 $Comp
-L power:+3.3V #PWR0184
+L power:+3.3V #PWR087
 U 1 1 61B620D7
 P 3100 4250
-F 0 "#PWR0184" H 3100 4100 50  0001 C CNN
+F 0 "#PWR087" H 3100 4100 50  0001 C CNN
 F 1 "+3.3V" H 3115 4423 50  0000 C CNN
 F 2 "" H 3100 4250 50  0001 C CNN
@@
 $EndComp
 $Comp
-L power:+5V #PWR0185
+L power:+5V #PWR083
 U 1 1 61B94788
 P 6550 2150
-F 0 "#PWR0185" H 6550 2000 50  0001 C CNN
+F 0 "#PWR083" H 6550 2000 50  0001 C CNN
 F 1 "+5V" H 6565 2323 50  0000 C CNN
 F 2 "" H 6550 2150 50  0001 C CNN
@@
 	6850 2150 6550 2150
 $Comp
-L power:GND #PWR0186
+L power:GND #PWR084
 U 1 1 61B984B1
 P 7200 2550
-F 0 "#PWR0186" H 7200 2300 50  0001 C CNN
+F 0 "#PWR084" H 7200 2300 50  0001 C CNN
 F 1 "GND" H 7205 2377 50  0000 C CNN
 F 2 "" H 7200 2550 50  0001 C CNN
@@
 Connection ~ 6550 2150
 $Comp
-L Device:R R35
+L Device:R R41
 U 1 1 61C43F79
 P 4300 4400
-F 0 "R35" H 4370 4446 50  0000 L CNN
+F 0 "R41" H 4370 4446 50  0000 L CNN
 F 1 "10k" H 4370 4355 50  0000 L CNN
 F 2 "Resistor_SMD:R_0402_1005Metric" V 4230 4400 50  0001 C CNN
@@
 $EndComp
 $Comp
-L Device:R R34
+L Device:R R40
 U 1 1 61C443EB
 P 4000 4400
-F 0 "R34" H 4070 4446 50  0000 L CNN
+F 0 "R40" H 4070 4446 50  0000 L CNN
 F 1 "10k" H 4070 4355 50  0000 L CNN
 F 2 "Resistor_SMD:R_0402_1005Metric" V 3930 4400 50  0001 C CNN
@@
 	3400 4250 4000 4250
 $Comp
-L Device:R R38
+L Device:R R44
 U 1 1 61FD3CEB
 P 3700 5400
-F 0 "R38" H 3770 5446 50  0000 L CNN
+F 0 "R44" H 3770 5446 50  0000 L CNN
 F 1 "10k" H 3770 5355 50  0000 L CNN
 F 2 "Resistor_SMD:R_0402_1005Metric" V 3630 5400 50  0001 C CNN
@@
 $EndComp
 $Comp
-L power:GND #PWR0187
+L power:GND #PWR090
 U 1 1 61FD40D4
 P 3700 5550
-F 0 "#PWR0187" H 3700 5300 50  0001 C CNN
+F 0 "#PWR090" H 3700 5300 50  0001 C CNN
 F 1 "GND" H 3705 5377 50  0000 C CNN
 F 2 "" H 3700 5550 50  0001 C CNN
@@
 Connection ~ 4300 5050
 $Comp
-L Device:R R36
+L Device:R R42
 U 1 1 6200261D
 P 4600 4400
-F 0 "R36" H 4670 4446 50  0000 L CNN
+F 0 "R42" H 4670 4446 50  0000 L CNN
 F 1 "10k" H 4670 4355 50  0000 L CNN
 F 2 "Resistor_SMD:R_0402_1005Metric" V 4530 4400 50  0001 C CNN
@@
 Text GLabel 3050 4950 0    50   Input ~ 0
 HDMI_DDC_EN
+Wire Wire Line
+	8350 3950 6800 3950
+Wire Wire Line
+	8350 3850 6800 3850
+Wire Wire Line
+	8350 3750 6800 3750
+Wire Wire Line
+	8350 3650 6800 3650
+Wire Wire Line
+	8350 3550 6800 3550
+Wire Wire Line
+	8350 3450 6800 3450
+Wire Wire Line
+	8350 3350 6800 3350
+Wire Wire Line
+	8350 3250 6800 3250
+Text Label 8150 3250 0    50   ~ 0
+D2_P
+Text Label 8150 3350 0    50   ~ 0
+D2_N
+Text Label 8150 3450 0    50   ~ 0
+D1_P
+Text Label 8150 3550 0    50   ~ 0
+D1_N
+Text Label 8150 3650 0    50   ~ 0
+D0_P
+Text Label 8150 3750 0    50   ~ 0
+D0_N
+Text Label 8150 3850 0    50   ~ 0
+CK_P
+Text Label 8150 3950 0    50   ~ 0
+CK_N
 $EndSCHEMATC

Commit message: More work on PCB
Connections:
- net labels added: 5V_HDMI
Changed lines of the file:
@@
 Text Label 8150 3950 0    50   ~ 0
 CK_N
+Text Label 7750 2150 0    50   ~ 0
+5V_HDMI
 $EndSCHEMATC
