File: kicad/imucam/hdmi.sch (KiCad schematic (older format))
At the start: 24 parts, among them J8 HDMI, U10 PTN3366, U9 AP2331

Commit message: Switched FSYNC to use TRIGGER, lots of PCB work
Parts:
- renumbered J8 to J7, R36 to R38, R37 to R39, R38 to R40, R39 to R41, R40 to R42, R41 to R43, R42 to R44, R43 to R45, R44 to R46
Changed lines of the file:
@@
 $EndComp
 $Comp
-L power:GND #PWR088
+L power:GND #PWR089
 U 1 1 61A343C7
 P 6200 5050
-F 0 "#PWR088" H 6200 4800 50  0001 C CNN
+F 0 "#PWR089" H 6200 4800 50  0001 C CNN
 F 1 "GND" H 6205 4877 50  0000 C CNN
 F 2 "" H 6200 5050 50  0001 C CNN
@@
 $EndComp
 $Comp
-L power:+3.3V #PWR085
+L power:+3.3V #PWR086
 U 1 1 61A34AA9
 P 6200 2600
-F 0 "#PWR085" H 6200 2450 50  0001 C CNN
+F 0 "#PWR086" H 6200 2450 50  0001 C CNN
 F 1 "+3.3V" H 6215 2773 50  0000 C CNN
 F 2 "" H 6200 2600 50  0001 C CNN
@@
 	5800 2900 5350 2900
 $Comp
-L power:GND #PWR086
+L power:GND #PWR087
 U 1 1 61A38134
 P 5350 2900
-F 0 "#PWR086" H 5350 2650 50  0001 C CNN
+F 0 "#PWR087" H 5350 2650 50  0001 C CNN
 F 1 "GND" H 5355 2727 50  0000 C CNN
 F 2 "" H 5350 2900 50  0001 C CNN
@@
 Connection ~ 6200 2600
 $Comp
-L Device:R R43
+L Device:R R45
 U 1 1 61A397D5
 P 7050 4750
-F 0 "R43" H 7120 4796 50  0000 L CNN
+F 0 "R45" H 7120 4796 50  0000 L CNN
 F 1 "12.4k 1%" H 7120 4705 50  0000 L CNN
 F 2 "Resistor_SMD:R_0402_1005Metric" V 6980 4750 50  0001 C CNN
@@
 	7750 4350 7750 4300
 $Comp
-L Device:R R37
+L Device:R R39
 U 1 1 61AEEAD1
 P 8050 4150
-F 0 "R37" H 8120 4196 50  0000 L CNN
+F 0 "R39" H 8120 4196 50  0000 L CNN
 F 1 "4.7k" H 8120 4105 50  0000 L CNN
 F 2 "Resistor_SMD:R_0402_1005Metric" V 7980 4150 50  0001 C CNN
@@
 $EndComp
 $Comp
-L Device:R R36
+L Device:R R38
 U 1 1 61AEDD4D
 P 7750 4150
-F 0 "R36" H 7820 4196 50  0000 L CNN
+F 0 "R38" H 7820 4196 50  0000 L CNN
 F 1 "4.7k" H 7820 4105 50  0000 L CNN
 F 2 "Resistor_SMD:R_0402_1005Metric" V 7680 4150 50  0001 C CNN
@@
 	8550 5150 8550 5200
 $Comp
-L power:GND #PWR089
+L power:GND #PWR090
 U 1 1 61A6FC85
 P 8750 5200
-F 0 "#PWR089" H 8750 4950 50  0001 C CNN
+F 0 "#PWR090" H 8750 4950 50  0001 C CNN
 F 1 "GND" H 8755 5027 50  0000 C CNN
 F 2 "" H 8750 5200 50  0001 C CNN
@@
 $EndComp
 $Comp
-L Connector:HDMI_A_1.4 J8
+L Connector:HDMI_A_1.4 J7
 U 1 1 61A5E9CE
 P 8750 4050
-F 0 "J8" H 9180 4096 50  0000 L CNN
+F 0 "J7" H 9180 4096 50  0000 L CNN
 F 1 "HDMI" H 9180 4005 50  0000 L CNN
 F 2 "imucam:CnC_2000-1-2-41-00-BK" H 8775 4050 50  0001 C CNN
@@
 HDMI_OE
 $Comp
-L Device:R R39
+L Device:R R41
 U 1 1 61B50DA8
 P 3400 4400
-F 0 "R39" H 3470 4446 50  0000 L CNN
+F 0 "R41" H 3470 4446 50  0000 L CNN
 F 1 "4.7k" H 3470 4355 50  0000 L CNN
 F 2 "Resistor_SMD:R_0402_1005Metric" V 3330 4400 50  0001 C CNN
@@
 $EndComp
 $Comp
-L Device:R R38
+L Device:R R40
 U 1 1 61B511BB
 P 3100 4400
-F 0 "R38" H 3170 4446 50  0000 L CNN
+F 0 "R40" H 3170 4446 50  0000 L CNN
 F 1 "4.7k" H 3170 4355 50  0000 L CNN
 F 2 "Resistor_SMD:R_0402_1005Metric" V 3030 4400 50  0001 C CNN
@@
 Connection ~ 3400 4750
 $Comp
-L power:+3.3V #PWR087
+L power:+3.3V #PWR088
 U 1 1 61B620D7
 P 3100 4250
-F 0 "#PWR087" H 3100 4100 50  0001 C CNN
+F 0 "#PWR088" H 3100 4100 50  0001 C CNN
 F 1 "+3.3V" H 3115 4423 50  0000 C CNN
 F 2 "" H 3100 4250 50  0001 C CNN
@@
 $EndComp
 $Comp
-L power:+5V #PWR083
+L power:+5V #PWR084
 U 1 1 61B94788
 P 6550 2150
-F 0 "#PWR083" H 6550 2000 50  0001 C CNN
+F 0 "#PWR084" H 6550 2000 50  0001 C CNN
 F 1 "+5V" H 6565 2323 50  0000 C CNN
 F 2 "" H 6550 2150 50  0001 C CNN
@@
 	6850 2150 6550 2150
 $Comp
-L power:GND #PWR084
+L power:GND #PWR085
 U 1 1 61B984B1
 P 7200 2550
-F 0 "#PWR084" H 7200 2300 50  0001 C CNN
+F 0 "#PWR085" H 7200 2300 50  0001 C CNN
 F 1 "GND" H 7205 2377 50  0000 C CNN
 F 2 "" H 7200 2550 50  0001 C CNN
@@
 Connection ~ 6550 2150
 $Comp
-L Device:R R41
+L Device:R R43
 U 1 1 61C43F79
 P 4300 4400
-F 0 "R41" H 4370 4446 50  0000 L CNN
+F 0 "R43" H 4370 4446 50  0000 L CNN
 F 1 "10k" H 4370 4355 50  0000 L CNN
 F 2 "Resistor_SMD:R_0402_1005Metric" V 4230 4400 50  0001 C CNN
@@
 $EndComp
 $Comp
-L Device:R R40
+L Device:R R42
 U 1 1 61C443EB
 P 4000 4400
-F 0 "R40" H 4070 4446 50  0000 L CNN
+F 0 "R42" H 4070 4446 50  0000 L CNN
 F 1 "10k" H 4070 4355 50  0000 L CNN
 F 2 "Resistor_SMD:R_0402_1005Metric" V 3930 4400 50  0001 C CNN
@@
 	3400 4250 4000 4250
 $Comp
-L Device:R R44
+L Device:R R46
 U 1 1 61FD3CEB
 P 3700 5400
-F 0 "R44" H 3770 5446 50  0000 L CNN
+F 0 "R46" H 3770 5446 50  0000 L CNN
 F 1 "10k" H 3770 5355 50  0000 L CNN
 F 2 "Resistor_SMD:R_0402_1005Metric" V 3630 5400 50  0001 C CNN
@@
 $EndComp
 $Comp
-L power:GND #PWR090
+L power:GND #PWR091
 U 1 1 61FD40D4
 P 3700 5550
-F 0 "#PWR090" H 3700 5300 50  0001 C CNN
+F 0 "#PWR091" H 3700 5300 50  0001 C CNN
 F 1 "GND" H 3705 5377 50  0000 C CNN
 F 2 "" H 3700 5550 50  0001 C CNN
@@
 Connection ~ 4300 5050
 $Comp
-L Device:R R42
+L Device:R R44
 U 1 1 6200261D
 P 4600 4400
-F 0 "R42" H 4670 4446 50  0000 L CNN
+F 0 "R44" H 4670 4446 50  0000 L CNN
 F 1 "10k" H 4670 4355 50  0000 L CNN
 F 2 "Resistor_SMD:R_0402_1005Metric" V 4530 4400 50  0001 C CNN

Commit message: Slightly more progress on current measurement
Parts:
- renumbered C69 to C66, C71 to C67, C73 to C68, C75 to C69, C72 to C71, C74 to C72, C76 to C73, C67 to C74, C68 to C75, C65 to C76, C66 to C77, R40 to R39, R41 to R40, R46 to R41, R38 to R46, R39 to R47, U9 to U11
Changed lines of the file:
@@
 $EndComp
 $Comp
-L power:GND #PWR089
+L power:GND #PWR091
 U 1 1 61A343C7
 P 6200 5050
-F 0 "#PWR089" H 6200 4800 50  0001 C CNN
+F 0 "#PWR091" H 6200 4800 50  0001 C CNN
 F 1 "GND" H 6205 4877 50  0000 C CNN
 F 2 "" H 6200 5050 50  0001 C CNN
@@
 $EndComp
 $Comp
-L power:+3.3V #PWR086
+L power:+3.3V #PWR090
 U 1 1 61A34AA9
 P 6200 2600
-F 0 "#PWR086" H 6200 2450 50  0001 C CNN
+F 0 "#PWR090" H 6200 2450 50  0001 C CNN
 F 1 "+3.3V" H 6215 2773 50  0000 C CNN
 F 2 "" H 6200 2600 50  0001 C CNN
@@
 $EndComp
 $Comp
-L Device:C C67
+L Device:C C74
 U 1 1 61A3662C
 P 5350 2750
-F 0 "C67" H 5465 2796 50  0000 L CNN
+F 0 "C74" H 5465 2796 50  0000 L CNN
 F 1 "10uF" H 5465 2705 50  0000 L CNN
 F 2 "Capacitor_SMD:C_0603_1608Metric" H 5388 2600 50  0001 C CNN
@@
 $EndComp
 $Comp
-L Device:C C68
+L Device:C C75
 U 1 1 61A3695C
 P 5800 2750
-F 0 "C68" H 5915 2796 50  0000 L CNN
+F 0 "C75" H 5915 2796 50  0000 L CNN
 F 1 "100nF" H 5915 2705 50  0000 L CNN
 F 2 "Capacitor_SMD:C_0402_1005Metric" H 5838 2600 50  0001 C CNN
@@
 	5800 2900 5350 2900
 $Comp
-L power:GND #PWR087
+L power:GND #PWR089
 U 1 1 61A38134
 P 5350 2900
-F 0 "#PWR087" H 5350 2650 50  0001 C CNN
+F 0 "#PWR089" H 5350 2650 50  0001 C CNN
 F 1 "GND" H 5355 2727 50  0000 C CNN
 F 2 "" H 5350 2900 50  0001 C CNN
@@
 HDMI_HPD
 $Comp
-L Device:C C69
+L Device:C C66
 U 1 1 61A78AD4
 P 4700 3250
-F 0 "C69" V 4650 3150 50  0000 C CNN
+F 0 "C66" V 4650 3150 50  0000 C CNN
 F 1 "100nF" V 4750 3100 50  0000 C CNN
 F 2 "Capacitor_SMD:C_0402_1005Metric" H 4738 3100 50  0001 C CNN
@@
 $EndComp
 $Comp
-L Device:C C71
+L Device:C C67
 U 1 1 61A7A48F
 P 4700 3450
-F 0 "C71" V 4650 3350 50  0000 C CNN
+F 0 "C67" V 4650 3350 50  0000 C CNN
 F 1 "100nF" V 4750 3300 50  0000 C CNN
 F 2 "Capacitor_SMD:C_0402_1005Metric" H 4738 3300 50  0001 C CNN
@@
 $EndComp
 $Comp
-L Device:C C72
+L Device:C C71
 U 1 1 61A7AA31
 P 5050 3550
-F 0 "C72" V 5000 3450 50  0000 C CNN
+F 0 "C71" V 5000 3450 50  0000 C CNN
 F 1 "100nF" V 5100 3400 50  0000 C CNN
 F 2 "Capacitor_SMD:C_0402_1005Metric" H 5088 3400 50  0001 C CNN
@@
 $EndComp
 $Comp
-L Device:C C73
+L Device:C C68
 U 1 1 61A7AEB6
 P 4700 3650
-F 0 "C73" V 4650 3550 50  0000 C CNN
+F 0 "C68" V 4650 3550 50  0000 C CNN
 F 1 "100nF" V 4750 3500 50  0000 C CNN
 F 2 "Capacitor_SMD:C_0402_1005Metric" H 4738 3500 50  0001 C CNN
@@
 $EndComp
 $Comp
-L Device:C C74
+L Device:C C72
 U 1 1 61A7B399
 P 5050 3750
-F 0 "C74" V 5000 3650 50  0000 C CNN
+F 0 "C72" V 5000 3650 50  0000 C CNN
 F 1 "100nF" V 5100 3600 50  0000 C CNN
 F 2 "Capacitor_SMD:C_0402_1005Metric" H 5088 3600 50  0001 C CNN
@@
 $EndComp
 $Comp
-L Device:C C75
+L Device:C C69
 U 1 1 61A7BB72
 P 4700 3850
-F 0 "C75" V 4650 3750 50  0000 C CNN
+F 0 "C69" V 4650 3750 50  0000 C CNN
 F 1 "100nF" V 4750 3700 50  0000 C CNN
 F 2 "Capacitor_SMD:C_0402_1005Metric" H 4738 3700 50  0001 C CNN
@@
 $EndComp
 $Comp
-L Device:C C76
+L Device:C C73
 U 1 1 61A7C0F4
 P 5050 3950
-F 0 "C76" V 5000 3850 50  0000 C CNN
+F 0 "C73" V 5000 3850 50  0000 C CNN
 F 1 "100nF" V 5100 3800 50  0000 C CNN
 F 2 "Capacitor_SMD:C_0402_1005Metric" H 5088 3800 50  0001 C CNN
@@
 	7750 4350 7750 4300
 $Comp
-L Device:R R39
+L Device:R R47
 U 1 1 61AEEAD1
 P 8050 4150
-F 0 "R39" H 8120 4196 50  0000 L CNN
+F 0 "R47" H 8120 4196 50  0000 L CNN
 F 1 "4.7k" H 8120 4105 50  0000 L CNN
 F 2 "Resistor_SMD:R_0402_1005Metric" V 7980 4150 50  0001 C CNN
@@
 $EndComp
 $Comp
-L Device:R R38
+L Device:R R46
 U 1 1 61AEDD4D
 P 7750 4150
-F 0 "R38" H 7820 4196 50  0000 L CNN
+F 0 "R46" H 7820 4196 50  0000 L CNN
 F 1 "4.7k" H 7820 4105 50  0000 L CNN
 F 2 "Resistor_SMD:R_0402_1005Metric" V 7680 4150 50  0001 C CNN
@@
 	8550 5150 8550 5200
 $Comp
-L power:GND #PWR090
+L power:GND #PWR094
 U 1 1 61A6FC85
 P 8750 5200
-F 0 "#PWR090" H 8750 4950 50  0001 C CNN
+F 0 "#PWR094" H 8750 4950 50  0001 C CNN
 F 1 "GND" H 8755 5027 50  0000 C CNN
 F 2 "" H 8750 5200 50  0001 C CNN
@@
 HDMI_OE
 $Comp
-L Device:R R41
+L Device:R R40
 U 1 1 61B50DA8
 P 3400 4400
-F 0 "R41" H 3470 4446 50  0000 L CNN
+F 0 "R40" H 3470 4446 50  0000 L CNN
 F 1 "4.7k" H 3470 4355 50  0000 L CNN
 F 2 "Resistor_SMD:R_0402_1005Metric" V 3330 4400 50  0001 C CNN
@@
 $EndComp
 $Comp
-L Device:R R40
+L Device:R R39
 U 1 1 61B511BB
 P 3100 4400
-F 0 "R40" H 3170 4446 50  0000 L CNN
+F 0 "R39" H 3170 4446 50  0000 L CNN
 F 1 "4.7k" H 3170 4355 50  0000 L CNN
 F 2 "Resistor_SMD:R_0402_1005Metric" V 3030 4400 50  0001 C CNN
@@
 Connection ~ 3400 4750
 $Comp
-L power:+3.3V #PWR088
+L power:+3.3V #PWR087
 U 1 1 61B620D7
 P 3100 4250
-F 0 "#PWR088" H 3100 4100 50  0001 C CNN
+F 0 "#PWR087" H 3100 4100 50  0001 C CNN
 F 1 "+3.3V" H 3115 4423 50  0000 C CNN
 F 2 "" H 3100 4250 50  0001 C CNN
@@
 	5150 4500 5150 4850
 $Comp
-L imucam:AP2331 U9
+L imucam:AP2331 U11
 U 1 1 61B93326
 P 7200 2250
-F 0 "U9" H 7200 2665 50  0000 C CNN
+F 0 "U11" H 7200 2665 50  0000 C CNN
 F 1 "AP2331" H 7200 2574 50  0000 C CNN
 F 2 "Package_TO_SOT_SMD:SOT-23" H 7200 1800 50  0001 C CNN
@@
 $EndComp
 $Comp
-L power:+5V #PWR084
+L power:+5V #PWR092
 U 1 1 61B94788
 P 6550 2150
-F 0 "#PWR084" H 6550 2000 50  0001 C CNN
+F 0 "#PWR092" H 6550 2000 50  0001 C CNN
 F 1 "+5V" H 6565 2323 50  0000 C CNN
 F 2 "" H 6550 2150 50  0001 C CNN
@@
 	6850 2150 6550 2150
 $Comp
-L power:GND #PWR085
+L power:GND #PWR093
 U 1 1 61B984B1
 P 7200 2550
-F 0 "#PWR085" H 7200 2300 50  0001 C CNN
+F 0 "#PWR093" H 7200 2300 50  0001 C CNN
 F 1 "GND" H 7205 2377 50  0000 C CNN
 F 2 "" H 7200 2550 50  0001 C CNN
@@
 	8050 2150 8050 2850
 $Comp
-L Device:C C65
+L Device:C C76
 U 1 1 61B9C87B
 P 6550 2350
-F 0 "C65" H 6665 2396 50  0000 L CNN
+F 0 "C76" H 6665 2396 50  0000 L CNN
 F 1 "100nF" H 6665 2305 50  0000 L CNN
 F 2 "Capacitor_SMD:C_0402_1005Metric" H 6588 2200 50  0001 C CNN
@@
 $EndComp
 $Comp
-L Device:C C66
+L Device:C C77
 U 1 1 61B9D2E1
 P 7650 2350
-F 0 "C66" H 7765 2396 50  0000 L CNN
+F 0 "C77" H 7765 2396 50  0000 L CNN
 F 1 "100nF" H 7765 2305 50  0000 L CNN
 F 2 "Capacitor_SMD:C_0402_1005Metric" H 7688 2200 50  0001 C CNN
@@
 	3400 4250 4000 4250
 $Comp
-L Device:R R46
+L Device:R R41
 U 1 1 61FD3CEB
 P 3700 5400
-F 0 "R46" H 3770 5446 50  0000 L CNN
+F 0 "R41" H 3770 5446 50  0000 L CNN
 F 1 "10k" H 3770 5355 50  0000 L CNN
 F 2 "Resistor_SMD:R_0402_1005Metric" V 3630 5400 50  0001 C CNN
@@
 $EndComp
 $Comp
-L power:GND #PWR091
+L power:GND #PWR088
 U 1 1 61FD40D4
 P 3700 5550
-F 0 "#PWR091" H 3700 5300 50  0001 C CNN
+F 0 "#PWR088" H 3700 5300 50  0001 C CNN
 F 1 "GND" H 3705 5377 50  0000 C CNN
 F 2 "" H 3700 5550 50  0001 C CNN

Commit message: Turns out, we need level translators
Parts:
- renumbered C76 to C70, C77 to C71, C74 to C72, C75 to C73, C66 to C74, C70 to C75, C67 to C76, C71 to C77, C68 to C78, C72 to C79, C69 to C80, C73 to C81, R46 to R30, R47 to R31, R39 to R32, R40 to R33, R42 to R34, R43 to R35, R44 to R36, R45 to R37, R41 to R38, U11 to U13, U10 to U14
Changed lines of the file:
@@
 $EndDescr
 $Comp
-L imucam:PTN3366 U10
+L imucam:PTN3366 U14
 U 1 1 61A33450
 P 6200 4150
-F 0 "U10" H 6650 5250 50  0000 C CNN
+F 0 "U14" H 6650 5250 50  0000 C CNN
 F 1 "PTN3366" H 5800 5250 50  0000 C CNN
 F 2 "Package_DFN_QFN:QFN-32-1EP_5x5mm_P0.5mm_EP3.6x3.6mm" H 6350 4250 50  0001 C CNN
@@
 $EndComp
 $Comp
-L power:GND #PWR091
+L power:GND #PWR098
 U 1 1 61A343C7
 P 6200 5050
-F 0 "#PWR091" H 6200 4800 50  0001 C CNN
+F 0 "#PWR098" H 6200 4800 50  0001 C CNN
 F 1 "GND" H 6205 4877 50  0000 C CNN
 F 2 "" H 6200 5050 50  0001 C CNN
@@
 $EndComp
 $Comp
-L power:+3.3V #PWR090
+L power:+3.3V #PWR095
 U 1 1 61A34AA9
 P 6200 2600
-F 0 "#PWR090" H 6200 2450 50  0001 C CNN
+F 0 "#PWR095" H 6200 2450 50  0001 C CNN
 F 1 "+3.3V" H 6215 2773 50  0000 C CNN
 F 2 "" H 6200 2600 50  0001 C CNN
@@
 $EndComp
 $Comp
-L Device:C C74
+L Device:C C72
 U 1 1 61A3662C
 P 5350 2750
-F 0 "C74" H 5465 2796 50  0000 L CNN
+F 0 "C72" H 5465 2796 50  0000 L CNN
 F 1 "10uF" H 5465 2705 50  0000 L CNN
 F 2 "Capacitor_SMD:C_0603_1608Metric" H 5388 2600 50  0001 C CNN
@@
 $EndComp
 $Comp
-L Device:C C75
+L Device:C C73
 U 1 1 61A3695C
 P 5800 2750
-F 0 "C75" H 5915 2796 50  0000 L CNN
+F 0 "C73" H 5915 2796 50  0000 L CNN
 F 1 "100nF" H 5915 2705 50  0000 L CNN
 F 2 "Capacitor_SMD:C_0402_1005Metric" H 5838 2600 50  0001 C CNN
@@
 	5800 2900 5350 2900
 $Comp
-L power:GND #PWR089
+L power:GND #PWR096
 U 1 1 61A38134
 P 5350 2900
-F 0 "#PWR089" H 5350 2650 50  0001 C CNN
+F 0 "#PWR096" H 5350 2650 50  0001 C CNN
 F 1 "GND" H 5355 2727 50  0000 C CNN
 F 2 "" H 5350 2900 50  0001 C CNN
@@
 Connection ~ 6200 2600
 $Comp
-L Device:R R45
+L Device:R R37
 U 1 1 61A397D5
 P 7050 4750
-F 0 "R45" H 7120 4796 50  0000 L CNN
+F 0 "R37" H 7120 4796 50  0000 L CNN
 F 1 "12.4k 1%" H 7120 4705 50  0000 L CNN
 F 2 "Resistor_SMD:R_0402_1005Metric" V 6980 4750 50  0001 C CNN
@@
 HDMI_HPD
 $Comp
-L Device:C C66
+L Device:C C74
 U 1 1 61A78AD4
 P 4700 3250
-F 0 "C66" V 4650 3150 50  0000 C CNN
+F 0 "C74" V 4650 3150 50  0000 C CNN
 F 1 "100nF" V 4750 3100 50  0000 C CNN
 F 2 "Capacitor_SMD:C_0402_1005Metric" H 4738 3100 50  0001 C CNN
@@
 $EndComp
 $Comp
-L Device:C C70
+L Device:C C75
 U 1 1 61A797BD
 P 5050 3350
-F 0 "C70" V 5000 3250 50  0000 C CNN
+F 0 "C75" V 5000 3250 50  0000 C CNN
 F 1 "100nF" V 5100 3200 50  0000 C CNN
 F 2 "Capacitor_SMD:C_0402_1005Metric" H 5088 3200 50  0001 C CNN
@@
 $EndComp
 $Comp
-L Device:C C67
+L Device:C C76
 U 1 1 61A7A48F
 P 4700 3450
-F 0 "C67" V 4650 3350 50  0000 C CNN
+F 0 "C76" V 4650 3350 50  0000 C CNN
 F 1 "100nF" V 4750 3300 50  0000 C CNN
 F 2 "Capacitor_SMD:C_0402_1005Metric" H 4738 3300 50  0001 C CNN
@@
 $EndComp
 $Comp
-L Device:C C71
+L Device:C C77
 U 1 1 61A7AA31
 P 5050 3550
-F 0 "C71" V 5000 3450 50  0000 C CNN
+F 0 "C77" V 5000 3450 50  0000 C CNN
 F 1 "100nF" V 5100 3400 50  0000 C CNN
 F 2 "Capacitor_SMD:C_0402_1005Metric" H 5088 3400 50  0001 C CNN
@@
 $EndComp
 $Comp
-L Device:C C68
+L Device:C C78
 U 1 1 61A7AEB6
 P 4700 3650
-F 0 "C68" V 4650 3550 50  0000 C CNN
+F 0 "C78" V 4650 3550 50  0000 C CNN
 F 1 "100nF" V 4750 3500 50  0000 C CNN
 F 2 "Capacitor_SMD:C_0402_1005Metric" H 4738 3500 50  0001 C CNN
@@
 $EndComp
 $Comp
-L Device:C C72
+L Device:C C79
 U 1 1 61A7B399
 P 5050 3750
-F 0 "C72" V 5000 3650 50  0000 C CNN
+F 0 "C79" V 5000 3650 50  0000 C CNN
 F 1 "100nF" V 5100 3600 50  0000 C CNN
 F 2 "Capacitor_SMD:C_0402_1005Metric" H 5088 3600 50  0001 C CNN
@@
 $EndComp
 $Comp
-L Device:C C69
+L Device:C C80
 U 1 1 61A7BB72
 P 4700 3850
-F 0 "C69" V 4650 3750 50  0000 C CNN
+F 0 "C80" V 4650 3750 50  0000 C CNN
 F 1 "100nF" V 4750 3700 50  0000 C CNN
 F 2 "Capacitor_SMD:C_0402_1005Metric" H 4738 3700 50  0001 C CNN
@@
 $EndComp
 $Comp
-L Device:C C73
+L Device:C C81
 U 1 1 61A7C0F4
 P 5050 3950
-F 0 "C73" V 5000 3850 50  0000 C CNN
+F 0 "C81" V 5000 3850 50  0000 C CNN
 F 1 "100nF" V 5100 3800 50  0000 C CNN
 F 2 "Capacitor_SMD:C_0402_1005Metric" H 5088 3800 50  0001 C CNN
@@
 	7750 4350 7750 4300
 $Comp
-L Device:R R47
+L Device:R R31
 U 1 1 61AEEAD1
 P 8050 4150
-F 0 "R47" H 8120 4196 50  0000 L CNN
+F 0 "R31" H 8120 4196 50  0000 L CNN
 F 1 "4.7k" H 8120 4105 50  0000 L CNN
 F 2 "Resistor_SMD:R_0402_1005Metric" V 7980 4150 50  0001 C CNN
@@
 $EndComp
 $Comp
-L Device:R R46
+L Device:R R30
 U 1 1 61AEDD4D
 P 7750 4150
-F 0 "R46" H 7820 4196 50  0000 L CNN
+F 0 "R30" H 7820 4196 50  0000 L CNN
 F 1 "4.7k" H 7820 4105 50  0000 L CNN
 F 2 "Resistor_SMD:R_0402_1005Metric" V 7680 4150 50  0001 C CNN
@@
 	8550 5150 8550 5200
 $Comp
-L power:GND #PWR094
+L power:GND #PWR099
 U 1 1 61A6FC85
 P 8750 5200
-F 0 "#PWR094" H 8750 4950 50  0001 C CNN
+F 0 "#PWR099" H 8750 4950 50  0001 C CNN
 F 1 "GND" H 8755 5027 50  0000 C CNN
 F 2 "" H 8750 5200 50  0001 C CNN
@@
 HDMI_OE
 $Comp
-L Device:R R40
+L Device:R R33
 U 1 1 61B50DA8
 P 3400 4400
-F 0 "R40" H 3470 4446 50  0000 L CNN
+F 0 "R33" H 3470 4446 50  0000 L CNN
 F 1 "4.7k" H 3470 4355 50  0000 L CNN
 F 2 "Resistor_SMD:R_0402_1005Metric" V 3330 4400 50  0001 C CNN
@@
 $EndComp
 $Comp
-L Device:R R39
+L Device:R R32
 U 1 1 61B511BB
 P 3100 4400
-F 0 "R39" H 3170 4446 50  0000 L CNN
+F 0 "R32" H 3170 4446 50  0000 L CNN
 F 1 "4.7k" H 3170 4355 50  0000 L CNN
 F 2 "Resistor_SMD:R_0402_1005Metric" V 3030 4400 50  0001 C CNN
@@
 Connection ~ 3400 4750
 $Comp
-L power:+3.3V #PWR087
+L power:+3.3V #PWR097
 U 1 1 61B620D7
 P 3100 4250
-F 0 "#PWR087" H 3100 4100 50  0001 C CNN
+F 0 "#PWR097" H 3100 4100 50  0001 C CNN
 F 1 "+3.3V" H 3115 4423 50  0000 C CNN
 F 2 "" H 3100 4250 50  0001 C CNN
@@
 	5150 4500 5150 4850
 $Comp
-L imucam:AP2331 U11
+L imucam:AP2331 U13
 U 1 1 61B93326
 P 7200 2250
-F 0 "U11" H 7200 2665 50  0000 C CNN
+F 0 "U13" H 7200 2665 50  0000 C CNN
 F 1 "AP2331" H 7200 2574 50  0000 C CNN
 F 2 "Package_TO_SOT_SMD:SOT-23" H 7200 1800 50  0001 C CNN
@@
 $EndComp
 $Comp
-L power:+5V #PWR092
+L power:+5V #PWR093
 U 1 1 61B94788
 P 6550 2150
-F 0 "#PWR092" H 6550 2000 50  0001 C CNN
+F 0 "#PWR093" H 6550 2000 50  0001 C CNN
 F 1 "+5V" H 6565 2323 50  0000 C CNN
 F 2 "" H 6550 2150 50  0001 C CNN
@@
 	6850 2150 6550 2150
 $Comp
-L power:GND #PWR093
+L power:GND #PWR094
 U 1 1 61B984B1
 P 7200 2550
-F 0 "#PWR093" H 7200 2300 50  0001 C CNN
+F 0 "#PWR094" H 7200 2300 50  0001 C CNN
 F 1 "GND" H 7205 2377 50  0000 C CNN
 F 2 "" H 7200 2550 50  0001 C CNN
@@
 	8050 2150 8050 2850
 $Comp
-L Device:C C76
+L Device:C C70
 U 1 1 61B9C87B
 P 6550 2350
-F 0 "C76" H 6665 2396 50  0000 L CNN
+F 0 "C70" H 6665 2396 50  0000 L CNN
 F 1 "100nF" H 6665 2305 50  0000 L CNN
 F 2 "Capacitor_SMD:C_0402_1005Metric" H 6588 2200 50  0001 C CNN
@@
 $EndComp
 $Comp
-L Device:C C77
+L Device:C C71
 U 1 1 61B9D2E1
 P 7650 2350
-F 0 "C77" H 7765 2396 50  0000 L CNN
+F 0 "C71" H 7765 2396 50  0000 L CNN
 F 1 "100nF" H 7765 2305 50  0000 L CNN
 F 2 "Capacitor_SMD:C_0402_1005Metric" H 7688 2200 50  0001 C CNN
@@
 Connection ~ 6550 2150
 $Comp
-L Device:R R43
+L Device:R R35
 U 1 1 61C43F79
 P 4300 4400
-F 0 "R43" H 4370 4446 50  0000 L CNN
+F 0 "R35" H 4370 4446 50  0000 L CNN
 F 1 "10k" H 4370 4355 50  0000 L CNN
 F 2 "Resistor_SMD:R_0402_1005Metric" V 4230 4400 50  0001 C CNN
@@
 $EndComp
 $Comp
-L Device:R R42
+L Device:R R34
 U 1 1 61C443EB
 P 4000 4400
-F 0 "R42" H 4070 4446 50  0000 L CNN
+F 0 "R34" H 4070 4446 50  0000 L CNN
 F 1 "10k" H 4070 4355 50  0000 L CNN
 F 2 "Resistor_SMD:R_0402_1005Metric" V 3930 4400 50  0001 C CNN
@@
 	3400 4250 4000 4250
 $Comp
-L Device:R R41
+L Device:R R38
 U 1 1 61FD3CEB
 P 3700 5400
-F 0 "R41" H 3770 5446 50  0000 L CNN
+F 0 "R38" H 3770 5446 50  0000 L CNN
 F 1 "10k" H 3770 5355 50  0000 L CNN
 F 2 "Resistor_SMD:R_0402_1005Metric" V 3630 5400 50  0001 C CNN
@@
 $EndComp
 $Comp
-L power:GND #PWR088
+L power:GND #PWR0100
 U 1 1 61FD40D4
 P 3700 5550
-F 0 "#PWR088" H 3700 5300 50  0001 C CNN
+F 0 "#PWR0100" H 3700 5300 50  0001 C CNN
 F 1 "GND" H 3705 5377 50  0000 C CNN
 F 2 "" H 3700 5550 50  0001 C CNN
@@
 Connection ~ 4300 5050
 $Comp
-L Device:R R44
+L Device:R R36
 U 1 1 6200261D
 P 4600 4400
-F 0 "R44" H 4670 4446 50  0000 L CNN
+F 0 "R36" H 4670 4446 50  0000 L CNN
 F 1 "10k" H 4670 4355 50  0000 L CNN
 F 2 "Resistor_SMD:R_0402_1005Metric" V 4530 4400 50  0001 C CNN
