File: kicad/imucam/imu.sch (KiCad schematic (older format))
At the start: 6 parts

Commit message: Cleaned up footprints
Parts:
- C? (x3): footprint Resistor_SMD:R_0402_1005Metric -> Capacitor_SMD:C_0402_1005Metric
- J?: footprint (none) -> Connector_PinHeader_2.54mm:PinHeader_1x03_P2.54mm_Vertical
- R?: footprint (none) -> Resistor_SMD:R_0402_1005Metric
- U?: footprint (none) -> Package_DFN_QFN:QFN-24-1EP_3x3mm_P0.4mm_EP1.75x1.6mm
Changed lines of the file:
@@
 F 0 "U?" H 3850 4000 50  0000 C CNN
 F 1 "ICM20948" H 4750 4000 50  0000 C CNN
-F 2 "" H 4350 3350 50  0001 C CNN
+F 2 "Package_DFN_QFN:QFN-24-1EP_3x3mm_P0.4mm_EP1.75x1.6mm" H 4350 3350 50  0001 C CNN
 F 3 "" H 4350 3350 50  0001 C CNN
 	1    4350 3350
@@
 F 0 "C?" H 4715 2246 50  0000 L CNN
 F 1 "100nF" H 4715 2155 50  0000 L CNN
-F 2 "Resistor_SMD:R_0402_1005Metric" H 4638 2050 50  0001 C CNN
+F 2 "Capacitor_SMD:C_0402_1005Metric" H 4638 2050 50  0001 C CNN
 F 3 "~" H 4600 2200 50  0001 C CNN
 	1    4600 2200
@@
 F 0 "C?" H 5165 2246 50  0000 L CNN
 F 1 "100nF" H 5165 2155 50  0000 L CNN
-F 2 "Resistor_SMD:R_0402_1005Metric" H 5088 2050 50  0001 C CNN
+F 2 "Capacitor_SMD:C_0402_1005Metric" H 5088 2050 50  0001 C CNN
 F 3 "~" H 5050 2200 50  0001 C CNN
 	1    5050 2200
@@
 F 0 "C?" H 5215 4246 50  0000 L CNN
 F 1 "100nF" H 5215 4155 50  0000 L CNN
-F 2 "Resistor_SMD:R_0402_1005Metric" H 5138 4050 50  0001 C CNN
+F 2 "Capacitor_SMD:C_0402_1005Metric" H 5138 4050 50  0001 C CNN
 F 3 "~" H 5100 4200 50  0001 C CNN
 	1    5100 4200
@@
 F 0 "J?" H 6580 3892 50  0000 L CNN
 F 1 "FSYNC_SEL" H 6580 3801 50  0000 L CNN
-F 2 "" H 6500 3850 50  0001 C CNN
+F 2 "Connector_PinHeader_2.54mm:PinHeader_1x03_P2.54mm_Vertical" H 6500 3850 50  0001 C CNN
 F 3 "~" H 6500 3850 50  0001 C CNN
 	1    6500 3850
@@
 F 0 "R?" H 5720 4246 50  0000 L CNN
 F 1 "10k" H 5720 4155 50  0000 L CNN
-F 2 "" V 5580 4200 50  0001 C CNN
+F 2 "Resistor_SMD:R_0402_1005Metric" V 5580 4200 50  0001 C CNN
 F 3 "~" H 5650 4200 50  0001 C CNN
 	1    5650 4200

Commit message: Annotated schematic
Parts:
- gave numbers to parts that had none: 6
Changed lines of the file:
@@
 $EndDescr
 $Comp
-L imucam:ICM20948 U?
+L imucam:ICM20948 U6
 U 1 1 61423402
 P 4350 3350
-F 0 "U?" H 3850 4000 50  0000 C CNN
+F 0 "U6" H 3850 4000 50  0000 C CNN
 F 1 "ICM20948" H 4750 4000 50  0000 C CNN
 F 2 "Package_DFN_QFN:QFN-24-1EP_3x3mm_P0.4mm_EP1.75x1.6mm" H 4350 3350 50  0001 C CNN
@@
 NoConn ~ 3700 3950
 $Comp
-L power:GND #PWR?
+L power:GND #PWR0158
 U 1 1 61424342
 P 4350 4150
-F 0 "#PWR?" H 4350 3900 50  0001 C CNN
+F 0 "#PWR0158" H 4350 3900 50  0001 C CNN
 F 1 "GND" H 4355 3977 50  0000 C CNN
 F 2 "" H 4350 4150 50  0001 C CNN
@@
 $EndComp
 $Comp
-L power:GND #PWR?
+L power:GND #PWR0159
 U 1 1 61424BD5
 P 3550 2950
-F 0 "#PWR?" H 3550 2700 50  0001 C CNN
+F 0 "#PWR0159" H 3550 2700 50  0001 C CNN
 F 1 "GND" H 3555 2777 50  0000 C CNN
 F 2 "" H 3550 2950 50  0001 C CNN
@@
 	3700 2950 3550 2950
 $Comp
-L power:+1V8 #PWR?
+L power:+1V8 #PWR0160
 U 1 1 61424F25
 P 4350 2000
-F 0 "#PWR?" H 4350 1850 50  0001 C CNN
+F 0 "#PWR0160" H 4350 1850 50  0001 C CNN
 F 1 "+1V8" H 4365 2173 50  0000 C CNN
 F 2 "" H 4350 2000 50  0001 C CNN
@@
 	4450 2650 4350 2650
 $Comp
-L Device:C C?
+L Device:C C54
 U 1 1 61425808
 P 4600 2200
-F 0 "C?" H 4715 2246 50  0000 L CNN
+F 0 "C54" H 4715 2246 50  0000 L CNN
 F 1 "100nF" H 4715 2155 50  0000 L CNN
 F 2 "Capacitor_SMD:C_0402_1005Metric" H 4638 2050 50  0001 C CNN
@@
 $EndComp
 $Comp
-L Device:C C?
+L Device:C C55
 U 1 1 614263DB
 P 5050 2200
-F 0 "C?" H 5165 2246 50  0000 L CNN
+F 0 "C55" H 5165 2246 50  0000 L CNN
 F 1 "100nF" H 5165 2155 50  0000 L CNN
 F 2 "Capacitor_SMD:C_0402_1005Metric" H 5088 2050 50  0001 C CNN
@@
 	4600 2350 5050 2350
 $Comp
-L power:GND #PWR?
+L power:GND #PWR0161
 U 1 1 61426F47
 P 5050 2350
-F 0 "#PWR?" H 5050 2100 50  0001 C CNN
+F 0 "#PWR0161" H 5050 2100 50  0001 C CNN
 F 1 "GND" H 5055 2177 50  0000 C CNN
 F 2 "" H 5050 2350 50  0001 C CNN
@@
 	5050 3450 5100 3450
 $Comp
-L Device:C C?
+L Device:C C56
 U 1 1 61429967
 P 5100 4200
-F 0 "C?" H 5215 4246 50  0000 L CNN
+F 0 "C56" H 5215 4246 50  0000 L CNN
 F 1 "100nF" H 5215 4155 50  0000 L CNN
 F 2 "Capacitor_SMD:C_0402_1005Metric" H 5138 4050 50  0001 C CNN
@@
 $EndComp
 $Comp
-L power:GND #PWR?
+L power:GND #PWR0162
 U 1 1 6142BF1F
 P 5100 4350
-F 0 "#PWR?" H 5100 4100 50  0001 C CNN
+F 0 "#PWR0162" H 5100 4100 50  0001 C CNN
 F 1 "GND" H 5105 4177 50  0000 C CNN
 F 2 "" H 5100 4350 50  0001 C CNN
@@
 	5050 3950 5200 3950
 $Comp
-L Connector_Generic:Conn_01x03 J?
+L Connector_Generic:Conn_01x03 J3
 U 1 1 61887C9A
 P 6500 3850
-F 0 "J?" H 6580 3892 50  0000 L CNN
+F 0 "J3" H 6580 3892 50  0000 L CNN
 F 1 "FSYNC_SEL" H 6580 3801 50  0000 L CNN
 F 2 "Connector_PinHeader_2.54mm:PinHeader_1x03_P2.54mm_Vertical" H 6500 3850 50  0001 C CNN
@@
 	5050 3850 5650 3850
 $Comp
-L Device:R R?
+L Device:R R18
 U 1 1 6188A3FB
 P 5650 4200
-F 0 "R?" H 5720 4246 50  0000 L CNN
+F 0 "R18" H 5720 4246 50  0000 L CNN
 F 1 "10k" H 5720 4155 50  0000 L CNN
 F 2 "Resistor_SMD:R_0402_1005Metric" V 5580 4200 50  0001 C CNN
@@
 $EndComp
 $Comp
-L power:GND #PWR?
+L power:GND #PWR0163
 U 1 1 6188AB2A
 P 5650 4350
-F 0 "#PWR?" H 5650 4100 50  0001 C CNN
+F 0 "#PWR0163" H 5650 4100 50  0001 C CNN
 F 1 "GND" H 5655 4177 50  0000 C CNN
 F 2 "" H 5650 4350 50  0001 C CNN

Commit message: Lots of schematic work
Connections:
- net labels added: CAM_SHUTTER
- net labels removed: CAM_TRIGGER
Changed lines of the file:
@@
 NoConn ~ 3700 3950
 $Comp
-L power:GND #PWR0158
+L power:GND #PWR061
 U 1 1 61424342
 P 4350 4150
-F 0 "#PWR0158" H 4350 3900 50  0001 C CNN
+F 0 "#PWR061" H 4350 3900 50  0001 C CNN
 F 1 "GND" H 4355 3977 50  0000 C CNN
 F 2 "" H 4350 4150 50  0001 C CNN
@@
 $EndComp
 $Comp
-L power:GND #PWR0159
+L power:GND #PWR060
 U 1 1 61424BD5
 P 3550 2950
-F 0 "#PWR0159" H 3550 2700 50  0001 C CNN
+F 0 "#PWR060" H 3550 2700 50  0001 C CNN
 F 1 "GND" H 3555 2777 50  0000 C CNN
 F 2 "" H 3550 2950 50  0001 C CNN
@@
 	3700 2950 3550 2950
 $Comp
-L power:+1V8 #PWR0160
+L power:+1V8 #PWR058
 U 1 1 61424F25
 P 4350 2000
-F 0 "#PWR0160" H 4350 1850 50  0001 C CNN
+F 0 "#PWR058" H 4350 1850 50  0001 C CNN
 F 1 "+1V8" H 4365 2173 50  0000 C CNN
 F 2 "" H 4350 2000 50  0001 C CNN
@@
 	4600 2350 5050 2350
 $Comp
-L power:GND #PWR0161
+L power:GND #PWR059
 U 1 1 61426F47
 P 5050 2350
-F 0 "#PWR0161" H 5050 2100 50  0001 C CNN
+F 0 "#PWR059" H 5050 2100 50  0001 C CNN
 F 1 "GND" H 5055 2177 50  0000 C CNN
 F 2 "" H 5050 2350 50  0001 C CNN
@@
 $EndComp
 $Comp
-L power:GND #PWR0162
+L power:GND #PWR062
 U 1 1 6142BF1F
 P 5100 4350
-F 0 "#PWR0162" H 5100 4100 50  0001 C CNN
+F 0 "#PWR062" H 5100 4100 50  0001 C CNN
 F 1 "GND" H 5105 4177 50  0000 C CNN
 F 2 "" H 5100 4350 50  0001 C CNN
@@
 $EndComp
 Text GLabel 6300 3750 0    50   Input ~ 0
-CAM_TRIGGER
+CAM_SHUTTER
 Text GLabel 6300 3950 0    50   Input ~ 0
 CAM_FLASH
@@
 $EndComp
 $Comp
-L power:GND #PWR0163
+L power:GND #PWR063
 U 1 1 6188AB2A
 P 5650 4350
-F 0 "#PWR0163" H 5650 4100 50  0001 C CNN
+F 0 "#PWR063" H 5650 4100 50  0001 C CNN
 F 1 "GND" H 5655 4177 50  0000 C CNN
 F 2 "" H 5650 4350 50  0001 C CNN

Commit message: More work on PCB
Parts:
- removed J3: FSYNC_SEL, Connector_PinHeader_2.54mm:PinHeader_1x03_P2.54mm_Vertical, symbol Connector_Generic:Conn_01x03
- added JP1: SolderJumper_3_Open, Jumper:SolderJumper-3_P1.3mm_Open_Pad1.0x1.5mm, symbol Jumper:SolderJumper_3_Open
Connections:
- wire segments 19 -> 21
Changed lines of the file:
@@
 Wire Wire Line
 	5050 3950 5200 3950
-$Comp
-L Connector_Generic:Conn_01x03 J3
-U 1 1 61887C9A
-P 6500 3850
-F 0 "J3" H 6580 3892 50  0000 L CNN
-F 1 "FSYNC_SEL" H 6580 3801 50  0000 L CNN
-F 2 "Connector_PinHeader_2.54mm:PinHeader_1x03_P2.54mm_Vertical" H 6500 3850 50  0001 C CNN
-F 3 "~" H 6500 3850 50  0001 C CNN
-	1    6500 3850
-	1    0    0    -1
-$EndComp
-Text GLabel 6300 3750 0    50   Input ~ 0
+Text GLabel 6550 3650 2    50   Input ~ 0
 CAM_SHUTTER
-Text GLabel 6300 3950 0    50   Input ~ 0
+Text GLabel 6550 4050 2    50   Input ~ 0
 CAM_FLASH
 Wire Wire Line
@@
 Wire Wire Line
 	5650 3850 6300 3850
+$Comp
+L Jumper:SolderJumper_3_Open JP1
+U 1 1 6140D595
+P 6450 3850
+F 0 "JP1" V 6450 3918 50  0000 L CNN
+F 1 "SolderJumper_3_Open" V 6495 3918 50  0001 L CNN
+F 2 "Jumper:SolderJumper-3_P1.3mm_Open_Pad1.0x1.5mm" H 6450 3850 50  0001 C CNN
+F 3 "~" H 6450 3850 50  0001 C CNN
+	1    6450 3850
+	0    1    1    0
+$EndComp
+Wire Wire Line
+	6550 3650 6450 3650
+Wire Wire Line
+	6550 4050 6450 4050
 $EndSCHEMATC

Commit message: Switched FSYNC to use TRIGGER, lots of PCB work
Parts:
- removed JP1: SolderJumper_3_Open, Jumper:SolderJumper-3_P1.3mm_Open_Pad1.0x1.5mm, symbol Jumper:SolderJumper_3_Open
- removed R18: 10k, Resistor_SMD:R_0402_1005Metric, symbol Device:R
Connections:
- net labels added: CAM_TRIGGER
- net labels removed: CAM_FLASH, CAM_SHUTTER
- wire segments 21 -> 17
Changed lines of the file:
@@
 Wire Wire Line
 	5050 3950 5200 3950
-Text GLabel 6550 3650 2    50   Input ~ 0
-CAM_SHUTTER
-Text GLabel 6550 4050 2    50   Input ~ 0
-CAM_FLASH
 Wire Wire Line
-	5050 3850 5650 3850
-$Comp
-L Device:R R18
-U 1 1 6188A3FB
-P 5650 4200
-F 0 "R18" H 5720 4246 50  0000 L CNN
-F 1 "10k" H 5720 4155 50  0000 L CNN
-F 2 "Resistor_SMD:R_0402_1005Metric" V 5580 4200 50  0001 C CNN
-F 3 "~" H 5650 4200 50  0001 C CNN
-	1    5650 4200
-	1    0    0    -1
-$EndComp
-$Comp
-L power:GND #PWR063
-U 1 1 6188AB2A
-P 5650 4350
-F 0 "#PWR063" H 5650 4100 50  0001 C CNN
-F 1 "GND" H 5655 4177 50  0000 C CNN
-F 2 "" H 5650 4350 50  0001 C CNN
-F 3 "" H 5650 4350 50  0001 C CNN
-	1    5650 4350
-	1    0    0    -1
-$EndComp
-Wire Wire Line
-	5650 3850 5650 4050
-Connection ~ 5650 3850
-Wire Wire Line
-	5650 3850 6300 3850
-$Comp
-L Jumper:SolderJumper_3_Open JP1
-U 1 1 6140D595
-P 6450 3850
-F 0 "JP1" V 6450 3918 50  0000 L CNN
-F 1 "SolderJumper_3_Open" V 6495 3918 50  0001 L CNN
-F 2 "Jumper:SolderJumper-3_P1.3mm_Open_Pad1.0x1.5mm" H 6450 3850 50  0001 C CNN
-F 3 "~" H 6450 3850 50  0001 C CNN
-	1    6450 3850
-	0    1    1    0
-$EndComp
-Wire Wire Line
-	6550 3650 6450 3650
-Wire Wire Line
-	6550 4050 6450 4050
+	5050 3850 5200 3850
+Text GLabel 5200 3850 2    50   Input ~ 0
+CAM_TRIGGER
 $EndSCHEMATC

Commit message: Turns out, we need level translators
Parts:
- renumbered C54 to C52, C55 to C53, C56 to C54
Changed lines of the file:
@@
 NoConn ~ 3700 3950
 $Comp
-L power:GND #PWR060
+L power:GND #PWR058
 U 1 1 61424342
 P 4350 4150
-F 0 "#PWR060" H 4350 3900 50  0001 C CNN
+F 0 "#PWR058" H 4350 3900 50  0001 C CNN
 F 1 "GND" H 4355 3977 50  0000 C CNN
 F 2 "" H 4350 4150 50  0001 C CNN
@@
 $EndComp
 $Comp
-L power:GND #PWR058
+L power:GND #PWR057
 U 1 1 61424BD5
 P 3550 2950
-F 0 "#PWR058" H 3550 2700 50  0001 C CNN
+F 0 "#PWR057" H 3550 2700 50  0001 C CNN
 F 1 "GND" H 3555 2777 50  0000 C CNN
 F 2 "" H 3550 2950 50  0001 C CNN
@@
 	3700 2950 3550 2950
 $Comp
-L power:+1V8 #PWR059
+L power:+1V8 #PWR055
 U 1 1 61424F25
 P 4350 2000
-F 0 "#PWR059" H 4350 1850 50  0001 C CNN
+F 0 "#PWR055" H 4350 1850 50  0001 C CNN
 F 1 "+1V8" H 4365 2173 50  0000 C CNN
 F 2 "" H 4350 2000 50  0001 C CNN
@@
 	4450 2650 4350 2650
 $Comp
-L Device:C C54
+L Device:C C52
 U 1 1 61425808
 P 4600 2200
-F 0 "C54" H 4715 2246 50  0000 L CNN
+F 0 "C52" H 4715 2246 50  0000 L CNN
 F 1 "100nF" H 4715 2155 50  0000 L CNN
 F 2 "Capacitor_SMD:C_0402_1005Metric" H 4638 2050 50  0001 C CNN
@@
 $EndComp
 $Comp
-L Device:C C55
+L Device:C C53
 U 1 1 614263DB
 P 5050 2200
-F 0 "C55" H 5165 2246 50  0000 L CNN
+F 0 "C53" H 5165 2246 50  0000 L CNN
 F 1 "100nF" H 5165 2155 50  0000 L CNN
 F 2 "Capacitor_SMD:C_0402_1005Metric" H 5088 2050 50  0001 C CNN
@@
 	4600 2350 5050 2350
 $Comp
-L power:GND #PWR061
+L power:GND #PWR056
 U 1 1 61426F47
 P 5050 2350
-F 0 "#PWR061" H 5050 2100 50  0001 C CNN
+F 0 "#PWR056" H 5050 2100 50  0001 C CNN
 F 1 "GND" H 5055 2177 50  0000 C CNN
 F 2 "" H 5050 2350 50  0001 C CNN
@@
 	5050 3450 5100 3450
 $Comp
-L Device:C C56
+L Device:C C54
 U 1 1 61429967
 P 5100 4200
-F 0 "C56" H 5215 4246 50  0000 L CNN
+F 0 "C54" H 5215 4246 50  0000 L CNN
 F 1 "100nF" H 5215 4155 50  0000 L CNN
 F 2 "Capacitor_SMD:C_0402_1005Metric" H 5138 4050 50  0001 C CNN
@@
 $EndComp
 $Comp
-L power:GND #PWR062
+L power:GND #PWR059
 U 1 1 6142BF1F
 P 5100 4350
-F 0 "#PWR062" H 5100 4100 50  0001 C CNN
+F 0 "#PWR059" H 5100 4100 50  0001 C CNN
 F 1 "GND" H 5105 4177 50  0000 C CNN
 F 2 "" H 5100 4350 50  0001 C CNN
