File: kicad/imucam/imu.sch (KiCad schematic (older format))
At the start: 4 parts, among them U6 ICM20948

Commit message: Ready to begin routing differential pairs
Parts:
- U6: footprint Package_DFN_QFN:QFN-24-1EP_3x3mm_P0.4mm_EP1.75x1.6mm -> imucam:QFN-24-1EP_3x3mm_P0.4mm_EP1.75x1.6mm_NoDiePad
Changed lines of the file:
@@
 Comment4 ""
 $EndDescr
-$Comp
-L imucam:ICM20948 U6
-U 1 1 61423402
-P 4350 3350
-F 0 "U6" H 3850 4000 50  0000 C CNN
-F 1 "ICM20948" H 4750 4000 50  0000 C CNN
-F 2 "Package_DFN_QFN:QFN-24-1EP_3x3mm_P0.4mm_EP1.75x1.6mm" H 4350 3350 50  0001 C CNN
-F 3 "" H 4350 3350 50  0001 C CNN
-	1    4350 3350
-	1    0    0    -1
-$EndComp
 NoConn ~ 3700 3050
 NoConn ~ 3700 3150
@@
 Text GLabel 5200 3850 2    50   Input ~ 0
 CAM_TRIGGER
+$Comp
+L imucam:ICM20948 U6
+U 1 1 61423402
+P 4350 3350
+F 0 "U6" H 3850 4000 50  0000 C CNN
+F 1 "ICM20948" H 4750 4000 50  0000 C CNN
+F 2 "imucam:QFN-24-1EP_3x3mm_P0.4mm_EP1.75x1.6mm_NoDiePad" H 4350 3350 50  0001 C CNN
+F 3 "" H 4350 3350 50  0001 C CNN
+	1    4350 3350
+	1    0    0    -1
+$EndComp
 $EndSCHEMATC

Commit message: More routing
Parts:
- U6: symbol imucam:ICM20948 -> imucam-rescue:ICM20948-imucam
Changed lines of the file:
@@
 CAM_TRIGGER
 $Comp
-L imucam:ICM20948 U6
+L imucam-rescue:ICM20948-imucam U6
 U 1 1 61423402
 P 4350 3350
