File: kicad/imucam/imucam.kicad_pcb (KiCad board)
At the start: 4 copper layers, 52.3 x 76.2 mm, 164 parts, among them J1 JTAG, J2 EXTCAM, J3 NUCLEO_CN8, J4 NUCLEO_CN7, J5 NUCLEO_CN9, J6 NUCLEO_CN10, J7 HDMI, Q1 BSS214NW, Q2 BSS214NW, Q3 BSS214NW, Q4 BSS214NW, Q5 BSS214NW, Q6 BSS214NW, U1 TLV73310PDBVT, U10 PTN3366, U2 LIFCL-17-xSG72, U3 AT25SF081-SSHD-X, U4 MIC5365-2.8YD5, U5 AR0330CM1C00, U6 ICM20948, U7 TPS562200, U8 TPS562200, U9 AP2331, X1 ECS-2520MV-xxx-xx

Commit message: Slightly more progress on current measurement
Parts:
- added C57: 100nF, Capacitor_SMD:C_0402_1005Metric, F.Cu at (54.6, 119.4)
- added R18: .05, Resistor_SMD:R_0805_2012Metric, F.Cu at (55.4, 116.9)
- added U7: INA219AxDCN, Package_TO_SOT_SMD:SOT-23-8, F.Cu at (50.8, 117.8)
- renumbered C6 to C1, C34 to C11, C1 to C12, C11 to C13, C24 to C14, C35 to C15, C36 to C16, C2 to C17, C12 to C18, C23 to C2, C25 to C20, C27 to C21, C29 to C22, C37 to C23, C3 to C24, C13 to C25, C20 to C26, C26 to C27, C30 to C29, C7 to C3, C14 to C30, C15 to C31, C16 to C32, C17 to C33, C18 to C34, C4 to C35, C5 to C36, C21 to C37, C53 to C38, C52 to C39, C31 to C4, C38 to C40, C43 to C41, C48 to C42, C39 to C43, C49 to C45, C40 to C46, C45 to C47, C50 to C48, C41 to C49, C8 to C5, C46 to C50, C42 to C52, C47 to C53, C62 to C59, C32 to C6, C59 to C60, C63 to C61, C57 to C62, C61 to C63, C60 to C64, C64 to C65, C69 to C66, C71 to C67, C73 to C68, C75 to C69, C9 to C7, C72 to C71, C74 to C72, C76 to C73, C67 to C74, C68 to C75, C65 to C76, C66 to C77, C22 to C8, C33 to C9, FB3 to FB1, FB4 to FB2, FB5 to FB3, FB2 to FB4, FB1 to FB5, J5 to J4, J4 to J5, R6 to R1, R1 to R11, R5 to R12, R11 to R13, R12 to R14, R13 to R15, R33 to R19, R34 to R20, R35 to R21, R36 to R22, R25 to R23, R30 to R24, R26 to R25, R31 to R26, R22 to R27, R27 to R28, R32 to R29, R7 to R3, R37 to R30, R18 to R31, R19 to R32, R20 to R33, R21 to R34, R23 to R35, R28 to R36, R24 to R37, R29 to R38, R40 to R39, R3 to R4, R41 to R40, R46 to R41, R38 to R46, R39 to R47, R8 to R5, R4 to R6, R9 to R7, R15 to R8, R14 to R9, U9 to U11, U7 to U8, U8 to U9
Connections:
- J1 pad 7: (no net) -> Net-(J1-Pad7)
- J2 pad 23: (no net) -> Net-(J2-Pad23)
- J2 pad 24: (no net) -> Net-(J2-Pad24)
- J3 pad 1: (no net) -> Net-(J3-Pad1)
- J3 pad 10: (no net) -> Net-(J3-Pad10)
- J3 pad 12: (no net) -> Net-(J3-Pad12)
- J3 pad 14: (no net) -> Net-(J3-Pad14)
- J3 pad 15: (no net) -> Net-(J3-Pad15)
- J3 pad 16: (no net) -> Net-(J3-Pad16)
- J3 pad 2: (no net) -> Net-(J3-Pad2)
- J3 pad 3: (no net) -> Net-(J3-Pad3)
- J3 pad 4: (no net) -> Net-(J3-Pad4)
- J3 pad 6: (no net) -> Net-(J3-Pad6)
- J3 pad 7: (no net) -> Net-(J3-Pad7)
- J3 pad 8: (no net) -> Net-(J3-Pad8)
- J3 pad 9: +5V -> /nucleo/5V_IN
- J4 pad 1: (no net) -> Net-(J4-Pad1)
- J4 pad 10: (no net) -> Net-(J4-Pad10)
- J4 pad 11: (no net) -> Net-(J4-Pad11)
- J4 pad 13: (no net) -> Net-(J4-Pad13)
- J4 pad 14: (no net) -> Net-(J4-Pad14)
- J4 pad 15: (no net) -> Net-(J4-Pad15)
- J4 pad 17: (no net) -> Net-(J4-Pad17)
- J4 pad 2: (no net) -> Net-(J4-Pad2)
- J4 pad 20: (no net) -> CAM_FLASH
- J4 pad 22: (no net) -> Net-(J4-Pad22)
- J4 pad 25: (no net) -> Net-(J4-Pad25)
- J4 pad 27: (no net) -> Net-(J4-Pad27)
- J4 pad 3: (no net) -> Net-(J4-Pad3)
- J4 pad 4: (no net) -> Net-(J4-Pad4)
- J4 pad 5: (no net) -> Net-(J4-Pad5)
- J4 pad 6: (no net) -> Net-(J4-Pad6)
- J4 pad 7: (no net) -> Net-(J4-Pad7)
- J4 pad 8: (no net) -> Net-(J4-Pad8)
- J4 pad 9: (no net) -> Net-(J4-Pad9)
- J5 pad 1: (no net) -> Net-(J5-Pad1)
- J5 pad 3: (no net) -> Net-(J5-Pad3)
- J5 pad 5: (no net) -> Net-(J5-Pad5)
- J5 pad 6: (no net) -> Net-(J5-Pad6)
- J5 pad 7: (no net) -> IMU_FSYNC_SEL
- J5 pad 9: (no net) -> IMU_FSYNC_EN
- J6 pad 1: (no net) -> Net-(J6-Pad1)
- J6 pad 10: (no net) -> /nucleo/CAM_TRIGGER_3V3
- J6 pad 11: (no net) -> Net-(J6-Pad11)
- J6 pad 12: (no net) -> Net-(J6-Pad12)
- J6 pad 13: (no net) -> Net-(J6-Pad13)
- J6 pad 14: (no net) -> Net-(J6-Pad14)
- J6 pad 15: (no net) -> Net-(J6-Pad15)
- J6 pad 16: (no net) -> Net-(J6-Pad16)
- J6 pad 18: (no net) -> Net-(J6-Pad18)
- J6 pad 2: (no net) -> Net-(J6-Pad2)
- J6 pad 20: (no net) -> Net-(J6-Pad20)
- J6 pad 24: (no net) -> Net-(J6-Pad24)
- J6 pad 25: (no net) -> Net-(J6-Pad25)
- J6 pad 26: (no net) -> Net-(J6-Pad26)
- J6 pad 28: (no net) -> Net-(J6-Pad28)
- J6 pad 29: (no net) -> Net-(J6-Pad29)
- J6 pad 3: (no net) -> Net-(J6-Pad3)
- J6 pad 30: (no net) -> Net-(J6-Pad30)
- J6 pad 31: (no net) -> Net-(J6-Pad31)
- J6 pad 32: (no net) -> Net-(J6-Pad32)
- J6 pad 33: (no net) -> Net-(J6-Pad33)
- J6 pad 34: (no net) -> Net-(J6-Pad34)
- J6 pad 7: (no net) -> Net-(J6-Pad7)
- J6 pad 8: (no net) -> Net-(J6-Pad8)
- J6 pad 9: (no net) -> Net-(J6-Pad9)
- J7 pad 13: (no net) -> Net-(J7-Pad13)
- J7 pad 14: (no net) -> Net-(J7-Pad14)
- R37 pad 1: (no net) -> /nucleo/IMU_CS_3V3
- U1 pad 4: (no net) -> Net-(U1-Pad4)
- U10 pad 23: (no net) -> Net-(U10-Pad23)
- U10 pad 24: (no net) -> Net-(U10-Pad24)
- U10 pad 3: (no net) -> Net-(U10-Pad3)
- U2 pad 39: (no net) -> Net-(U2-Pad39)
- U4 pad 4: (no net) -> Net-(U4-Pad4)
- U5 pad 10: (no net) -> Net-(U5-Pad10)
- U5 pad 11: (no net) -> Net-(U5-Pad11)
- U5 pad 12: (no net) -> Net-(U5-Pad12)
- U5 pad 13: (no net) -> Net-(U5-Pad13)
- U5 pad 14: (no net) -> Net-(U5-Pad14)
- U5 pad 15: (no net) -> Net-(U5-Pad15)
- U5 pad 16: (no net) -> Net-(U5-Pad16)
- U5 pad 3: (no net) -> Net-(U5-Pad3)
- U5 pad 35: (no net) -> Net-(U5-Pad35)
- U5 pad 7: (no net) -> Net-(U5-Pad7)
- U5 pad 8: (no net) -> Net-(U5-Pad8)
- U5 pad 9: (no net) -> Net-(U5-Pad9)
- U6 pad 1: (no net) -> Net-(U6-Pad1)
- U6 pad 14: (no net) -> Net-(U6-Pad14)
- U6 pad 15: (no net) -> Net-(U6-Pad15)
- U6 pad 16: (no net) -> Net-(U6-Pad16)
- U6 pad 17: (no net) -> Net-(U6-Pad17)
- U6 pad 19: (no net) -> Net-(U6-Pad19)
- U6 pad 2: (no net) -> Net-(U6-Pad2)
- U6 pad 3: (no net) -> Net-(U6-Pad3)
- U6 pad 4: (no net) -> Net-(U6-Pad4)
- U6 pad 5: (no net) -> Net-(U6-Pad5)
- U6 pad 6: (no net) -> Net-(U6-Pad6)
- X1 pad 1: (no net) -> Net-(X1-Pad1)

Commit message: Turns out, we need level translators
Parts:
- removed the C50 at (23.9, 31.8)
- removed the C51 at (29.5, 26.7)
- removed the C52 at (29.1, 32.1)
- removed the C53 at (27.7, 32.1)
- removed Q5, Q6: BSS214NW, Package_TO_SOT_SMD:SOT-323_SC-70
- removed the R23 at (-120.6, -16.1)
- removed the R24 at (-49.5, 104.4)
- removed the R25 at (-56.7, 112.1)
- removed the R26 at (-40.6, 95.5)
- removed the R27 at (-19.1, 3.81)
- removed the R28 at (-16.1, 5.80)
- removed the R29 at (-24.7, 32.7)
- removed the R30 at (-21.8, 32.7)
- removed the R35 at (-19.1, 5.80)
- removed the R36 at (-13.2, 3.81)
- removed the R37 at (-16.1, 3.81)
- removed the R38 at (-13.2, 5.80)
- added C38: 1uF, Capacitor_SMD:C_0402_1005Metric, F.Cu at (-55.5, -21.4)
- added C39: 100nF, Capacitor_SMD:C_0402_1005Metric, F.Cu at (-55.5, -19.4)
- added C55: 100nF, Capacitor_SMD:C_0402_1005Metric, F.Cu at (-65.4, -19.4)
- added C56: 100nF, Capacitor_SMD:C_0402_1005Metric, F.Cu at (-74.2, -10.9)
- added C57: 100nF, Capacitor_SMD:C_0402_1005Metric, F.Cu at (-62.5, -21.4)
- added C58: 100nF, Capacitor_SMD:C_0402_1005Metric, F.Cu at (-71.2, -12.9)
- added C59: 100nF, Capacitor_SMD:C_0402_1005Metric, F.Cu at (-68.3, -14.8)
- added C60: 100nF, Capacitor_SMD:C_0402_1005Metric, F.Cu at (-65.4, -17.4)
- added R18: 4.7k, Resistor_SMD:R_0402_1005Metric, F.Cu at (-65.4, -21.4)
- added R19: 4.7k, Resistor_SMD:R_0402_1005Metric, F.Cu at (-74.1, -12.8)
- added R20: 4.7k, Resistor_SMD:R_0402_1005Metric, F.Cu at (-71.2, -14.8)
- added U11: NTS0104PW, Package_SO:TSSOP-14_4.4x5mm_P0.65mm, F.Cu at (-71.2, -19.1)
- added U7: NTS0104PW, Package_SO:TSSOP-14_4.4x5mm_P0.65mm, F.Cu at (-80.0, -19.1)
- added U8: NTS0104PW, Package_SO:TSSOP-14_4.4x5mm_P0.65mm, F.Cu at (-80.0, -12.6)
- C40, C41, C45, C46, C47, C48: moved to F.Cu
- C42, C44: value 100nF -> 1uF; moved to F.Cu
- C43, C49: value 1uF -> 100nF; moved to F.Cu
- R26: renamed from R19; value 1k -> 100
- R27: renamed from R20; value 1k -> 100
- R28: renamed from R21; value 1k -> 100
- R29: renamed from R22; value 1k -> 100
- moved R17 132.9 mm to (-74.1, -14.8)
- moved C42 93.7 mm to (-52.6, -19.4), turned to 0 degrees
- moved C45 90.8 mm to (-49.8, -19.4), turned to 0 degrees
- moved C44 88.6 mm to (-52.6, -17.5), turned to 0 degrees
- moved C46 88.2 mm to (-46.9, -21.4), turned to 0 degrees
- moved C48 87.8 mm to (-46.9, -19.4), turned to 0 degrees
- moved C47 87.6 mm to (-49.8, -17.5), turned to 0 degrees
- moved C49 87.5 mm to (-46.9, -17.5)
- moved C43 87.4 mm to (-49.8, -21.4), turned to 0 degrees
- moved C41 86.9 mm to (-55.5, -17.5), turned to 0 degrees
- moved C40 85.7 mm to (-52.6, -21.4), turned to 0 degrees
- renumbered C12 to C1, C13 to C11, C18 to C12, C25 to C13, C30 to C14, C31 to C15, C32 to C16, C33 to C17, C34 to C18, C17 to C2, C26 to C20, C37 to C21, C8 to C22, C2 to C23, C14 to C24, C20 to C25, C27 to C26, C21 to C27, C22 to C29, C24 to C3, C29 to C30, C4 to C31, C6 to C32, C9 to C33, C11 to C34, C15 to C35, C16 to C36, C23 to C37, C35 to C4, C36 to C5, C39 to C50, C38 to C51, C54 to C52, C55 to C53, C56 to C54, C1 to C6, C63 to C61, C59 to C63, C61 to C64, C58 to C66, C60 to C67, C64 to C68, C57 to C69, C3 to C7, C76 to C70, C77 to C71, C74 to C72, C75 to C73, C66 to C74, C70 to C75, C67 to C76, C71 to C77, C68 to C78, C72 to C79, C5 to C8, C69 to C80, C73 to C81, C7 to C9, FB5 to FB1, FB4 to FB2, FB1 to FB3, FB2 to FB4, FB3 to FB5, J5 to J4, J4 to J5, L2 to L1, L1 to L2, STM_LED4 to PWR1, R11 to R1, R13 to R11, R14 to R12, R15 to R13, R9 to R14, R8 to R15, R33 to R21, R31 to R22, R34 to R23, R32 to R24, R18 to R25, R4 to R3, R46 to R30, R47 to R31, R39 to R32, R40 to R33, R42 to R34, R43 to R35, R44 to R36, R45 to R37, R41 to R38, R6 to R4, R12 to R5, R1 to R6, R3 to R7, R5 to R8, R7 to R9, U8 to U10, U7 to U12, U11 to U13, U10 to U14
Connections:
- C43 pad 1: +1V8 -> +2V8
- C44 pad 1: +1V8 -> +2V8
- C46 pad 1: +1V8 -> +2V8
- C47 pad 1: +1V8 -> +2V8
- C49 pad 1: +1V8 -> +2V8
- J1 pad 7: Net-(J1-Pad7) -> (no net)
- J2 pad 23: Net-(J2-Pad23) -> (no net)
- J2 pad 24: Net-(J2-Pad24) -> (no net)
- J3 pad 1: Net-(J3-Pad1) -> (no net)
- J3 pad 10: Net-(J3-Pad10) -> (no net)
- J3 pad 12: Net-(J3-Pad12) -> (no net)
- J3 pad 14: Net-(J3-Pad14) -> (no net)
- J3 pad 15: Net-(J3-Pad15) -> (no net)
- J3 pad 16: Net-(J3-Pad16) -> (no net)
- J3 pad 2: Net-(J3-Pad2) -> (no net)
- J3 pad 3: Net-(J3-Pad3) -> (no net)
- J3 pad 4: Net-(J3-Pad4) -> (no net)
- J3 pad 6: Net-(J3-Pad6) -> (no net)
- J3 pad 7: Net-(J3-Pad7) -> (no net)
- J3 pad 8: Net-(J3-Pad8) -> (no net)
- J4 pad 1: Net-(J5-Pad1) -> (no net)
- J4 pad 11: IMU_INT -> /nucleo/IMU_INT_3V3
- J4 pad 17: IMU_CS -> /nucleo/IMU_CS_3V3
- J4 pad 19: IMU_SO -> /nucleo/IMU_SO_3V3
- J4 pad 3: Net-(J5-Pad3) -> (no net)
- J4 pad 5: Net-(J5-Pad5) -> (no net)
- J4 pad 6: Net-(J5-Pad6) -> (no net)
- J4 pad 7: IMU_FSYNC_SEL -> (no net)
- J4 pad 9: IMU_FSYNC_EN -> (no net)
- J5 pad 1: Net-(J4-Pad1) -> (no net)
- J5 pad 10: Net-(J4-Pad10) -> (no net)
- J5 pad 11: Net-(J4-Pad11) -> (no net)
- J5 pad 13: Net-(J4-Pad13) -> (no net)
- J5 pad 14: Net-(J4-Pad14) -> (no net)
- J5 pad 15: Net-(J4-Pad15) -> (no net)
- J5 pad 16: CAM_RESET_BAR -> /nucleo/CAM_RESET_BAR_3V3
- J5 pad 17: Net-(J4-Pad17) -> (no net)
- J5 pad 18: CAM_TRIGGER -> /nucleo/CAM_SHUTTER_3V3
- J5 pad 2: Net-(J4-Pad2) -> (no net)
- J5 pad 20: CAM_FLASH -> /nucleo/CAM_FLASH_3V3
- J5 pad 22: Net-(J4-Pad22) -> (no net)
- J5 pad 25: Net-(J4-Pad25) -> (no net)
- J5 pad 27: Net-(J4-Pad27) -> (no net)
- J5 pad 3: Net-(J4-Pad3) -> (no net)
- J5 pad 4: Net-(J4-Pad4) -> (no net)
- J5 pad 5: Net-(J4-Pad5) -> (no net)
- J5 pad 6: Net-(J4-Pad6) -> (no net)
- J5 pad 7: Net-(J4-Pad7) -> (no net)
- J5 pad 8: Net-(J4-Pad8) -> (no net)
- J5 pad 9: Net-(J4-Pad9) -> (no net)
- J6 pad 1: Net-(J6-Pad1) -> (no net)
- J6 pad 11: Net-(J6-Pad11) -> (no net)
- J6 pad 12: Net-(J6-Pad12) -> (no net)
- J6 pad 13: Net-(J6-Pad13) -> (no net)
- J6 pad 14: Net-(J6-Pad14) -> (no net)
- J6 pad 15: Net-(J6-Pad15) -> (no net)
- J6 pad 16: Net-(J6-Pad16) -> (no net)
- J6 pad 18: Net-(J6-Pad18) -> (no net)
- J6 pad 2: Net-(J6-Pad2) -> (no net)
- J6 pad 20: Net-(J6-Pad20) -> (no net)
- J6 pad 24: Net-(J6-Pad24) -> (no net)
- J6 pad 25: Net-(J6-Pad25) -> (no net)
- J6 pad 26: Net-(J6-Pad26) -> (no net)
- J6 pad 28: Net-(J6-Pad28) -> (no net)
- J6 pad 29: Net-(J6-Pad29) -> (no net)
- J6 pad 3: Net-(J6-Pad3) -> (no net)
- J6 pad 30: Net-(J6-Pad30) -> (no net)
- J6 pad 31: Net-(J6-Pad31) -> (no net)
- J6 pad 32: Net-(J6-Pad32) -> (no net)
- J6 pad 33: Net-(J6-Pad33) -> (no net)
- J6 pad 34: Net-(J6-Pad34) -> (no net)
- J6 pad 7: Net-(J6-Pad7) -> (no net)
- J6 pad 8: Net-(J6-Pad8) -> (no net)
- J6 pad 9: Net-(J6-Pad9) -> (no net)
- J7 pad 13: Net-(J7-Pad13) -> (no net)
- J7 pad 14: Net-(J7-Pad14) -> (no net)
- R17 pad 1: +1V8 -> +3V3
- R17 pad 2: CAM_RESET_BAR -> SDA_3V3
- U1 pad 4: Net-(U1-Pad4) -> (no net)
- U14 pad 23: Net-(U10-Pad23) -> (no net)
- U14 pad 24: Net-(U10-Pad24) -> (no net)
- U14 pad 3: Net-(U10-Pad3) -> (no net)
- U2 pad 39: Net-(U2-Pad39) -> (no net)
- U4 pad 4: Net-(U4-Pad4) -> (no net)
- U5 pad 10: Net-(U5-Pad10) -> (no net)
- U5 pad 11: Net-(U5-Pad11) -> (no net)
- U5 pad 12: Net-(U5-Pad12) -> (no net)
- U5 pad 13: Net-(U5-Pad13) -> (no net)
- U5 pad 14: Net-(U5-Pad14) -> (no net)
- U5 pad 15: Net-(U5-Pad15) -> (no net)
- U5 pad 16: Net-(U5-Pad16) -> (no net)
- U5 pad 17: +1V8 -> +2V8
- U5 pad 23: +1V8 -> +2V8
- U5 pad 3: Net-(U5-Pad3) -> CAM_FLASH
- U5 pad 35: Net-(U5-Pad35) -> CAM_SHUTTER
- U5 pad 7: Net-(U5-Pad7) -> (no net)
- U5 pad 8: Net-(U5-Pad8) -> (no net)
- U5 pad 9: Net-(U5-Pad9) -> (no net)
- U6 pad 1: Net-(U6-Pad1) -> (no net)
- U6 pad 14: Net-(U6-Pad14) -> (no net)
- U6 pad 15: Net-(U6-Pad15) -> (no net)
- U6 pad 16: Net-(U6-Pad16) -> (no net)
- U6 pad 17: Net-(U6-Pad17) -> (no net)
- U6 pad 19: Net-(U6-Pad19) -> (no net)
- U6 pad 2: Net-(U6-Pad2) -> (no net)
- U6 pad 3: Net-(U6-Pad3) -> (no net)
- U6 pad 4: Net-(U6-Pad4) -> (no net)
- U6 pad 5: Net-(U6-Pad5) -> (no net)
- U6 pad 6: Net-(U6-Pad6) -> (no net)
- X1 pad 1: Net-(X1-Pad1) -> (no net)

Commit message: WIP of remapping nucleo pinout for pcb routing
Parts:
- removed C78, C79, C80, C81: 100nF, Capacitor_SMD:C_0402_1005Metric
- removed U13: AP2331, Package_TO_SOT_SMD:SOT-23
- removed U14: PTN3366, Package_DFN_QFN:QFN-32-1EP_5x5mm_P0.5mm_EP3.6x3.6mm
- added R39: 4.7k, Resistor_SMD:R_0402_1005Metric, F.Cu at (-26.7, 38.1)
- C1, C18, C27, C29, C3, C33, C35, C63, C66, C72: value 10uF -> 100nF; footprint Capacitor_SMD:C_0603_1608Metric -> Capacitor_SMD:C_0402_1005Metric
- C12, C14, C15, C17, C21, C34, C55, C60, C74, C9: value 100nF -> 10uF; footprint Capacitor_SMD:C_0402_1005Metric -> Capacitor_SMD:C_0603_1608Metric
- C2: value 10uF -> 1uF; footprint Capacitor_SMD:C_0603_1608Metric -> Capacitor_SMD:C_0402_1005Metric
- C22: value 1uF -> 10uF; footprint Capacitor_SMD:C_0402_1005Metric -> Capacitor_SMD:C_0603_1608Metric
- C23, C42, C46, C51: value 1uF -> 100nF
- C31: value 2.2uF -> 100nF
- C36, C39, C41, C45, C8: value 100nF -> 1uF
- C4: value 1uF -> 2.2uF
- C59, C64: value 100nF -> 22uF; footprint Capacitor_SMD:C_0402_1005Metric -> Capacitor_SMD:C_0603_1608Metric
- C65, C68: value 22uF -> 100nF; footprint Capacitor_SMD:C_0603_1608Metric -> Capacitor_SMD:C_0402_1005Metric
- J4: value NUCLEO_CN7 -> NUCLEO_CN9; footprint Connector_PinHeader_2.54mm:PinHeader_2x10_P2.54mm_Vertical -> Connector_PinHeader_2.54mm:PinHeader_2x15_P2.54mm_Vertical
- J5: value NUCLEO_CN9 -> NUCLEO_CN7; footprint Connector_PinHeader_2.54mm:PinHeader_2x15_P2.54mm_Vertical -> Connector_PinHeader_2.54mm:PinHeader_2x10_P2.54mm_Vertical
- R11, R20, R33: value 4.7k -> 10k
- R12: value 4.7k -> 1k
- R13, R38: value 10k -> 4.7k
- R14, R26, R29: value 100 -> 4.7k
- R18: value 4.7k -> .05; footprint Resistor_SMD:R_0402_1005Metric -> Resistor_SMD:R_0805_2012Metric
- R19: value 4.7k -> 12.4k
- R21: value 12.4k -> 100
- R22: value 30.9k -> 100
- R23, R24, R6: value 10k -> 100
- R25: value .05 -> 4.7k; footprint Resistor_SMD:R_0805_2012Metric -> Resistor_SMD:R_0402_1005Metric
- R27: value 100 -> 30.9k
- R28, R3: value 100 -> 10k
- R5: value 1k -> 10k
- R7: value 10k -> 1k
- R9: value 1k -> 100
- U10: value TPS562200 -> NTS0308E; footprint Package_TO_SOT_SMD:SOT-23-6 -> Package_SO:TSSOP-20_4.4x6.5mm_P0.65mm
- U11: value NTS0104PW -> PTN3366; footprint Package_SO:TSSOP-14_4.4x5mm_P0.65mm -> Package_DFN_QFN:QFN-32-1EP_5x5mm_P0.5mm_EP3.6x3.6mm_ThermalVias
- U12: value INA219AxDCN -> AP2331; footprint Package_TO_SOT_SMD:SOT-23-8 -> Package_TO_SOT_SMD:SOT-23
- U7: value NTS0104PW -> TPS562200; footprint Package_SO:TSSOP-14_4.4x5mm_P0.65mm -> Package_TO_SOT_SMD:SOT-23-6
- U8: value NTS0104PW -> INA219AxDCN; footprint Package_SO:TSSOP-14_4.4x5mm_P0.65mm -> Package_TO_SOT_SMD:SOT-23-8
- moved U11 125.0 mm to (34.6, 47.5), turned to 180 degrees
- moved C74 57.4 mm to (89.7, 51.1)
- moved J4 55.5 mm to (0.00, 35.6)
- moved DONE1 51.8 mm to (61.7, 5.08)
- moved FPGA_LED1 51.8 mm to (61.7, 7.37)
- moved FPGA_LED2 51.8 mm to (61.7, 9.65)
- moved FPGA_LED3 51.8 mm to (61.7, 11.9)
- moved C75 51.5 mm to (83.6, 56.1)
- moved C76 51.5 mm to (83.6, 59.1)
- moved C77 51.5 mm to (83.6, 58.1)
- moved C52 48.6 mm to (-21.8, 30.0)
- moved J6 46.0 mm to (45.7, 30.5)
- moved C73 44.7 mm to (84.3, 46.2)
- moved C53 42.9 mm to (-11.7, 28.2)
- moved C54 42.3 mm to (-14.2, 31.2)
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Connections:
- C11 pad 1: +1V0 -> Net-(C11-Pad1)
- C14 pad 1: Net-(C14-Pad1) -> +1V8
- C15 pad 1: Net-(C14-Pad1) -> Net-(C15-Pad1)
- C16 pad 1: Net-(C14-Pad1) -> Net-(C15-Pad1)
- C17 pad 1: Net-(C14-Pad1) -> +1V0
- C18 pad 1: Net-(C14-Pad1) -> +1V0
- C2 pad 1: +1V0 -> +1V8
- C22 pad 1: +1V0 -> +3V3
- C23 pad 1: +1V8 -> Net-(C15-Pad1)
- C24 pad 1: +1V8 -> +1V0
- C25 pad 1: +1V8 -> +1V0
- C27 pad 1: +3V3 -> +1V8
- C30 pad 1: +3V3 -> Net-(C30-Pad1)
- C31 pad 1: Net-(C31-Pad1) -> Net-(C30-Pad1)
- C32 pad 1: Net-(C31-Pad1) -> Net-(C30-Pad1)
- C33 pad 1: Net-(C33-Pad1) -> Net-(C30-Pad1)
- C34 pad 1: Net-(C33-Pad1) -> Net-(C30-Pad1)
- C35 pad 1: Net-(C35-Pad1) -> +3V3
- C36 pad 1: Net-(C35-Pad1) -> Net-(C36-Pad1)
- C37 pad 1: Net-(C35-Pad1) -> Net-(C36-Pad1)
- C38 pad 1: +1V8 -> +3V3
- C39 pad 1: +1V8 -> +2V8
- C41 pad 1: +1V8 -> +2V8
- C42 pad 1: +2V8 -> +1V8
- C44 pad 1: +2V8 -> +1V8
- C46 pad 1: +2V8 -> +1V8
- C5 pad 1: Net-(C4-Pad1) -> +1V0
- C51 pad 1: +3V3 -> +2V8
- C55 pad 1: GND -> +5V
- C55 pad 2: +3V3 -> GND
- C56 pad 1: +1V8 -> +5V
- C57 pad 1: GND -> Net-(C57-Pad1)
- C57 pad 2: +3V3 -> Net-(C57-Pad2)
- C58 pad 1: +1V8 -> +3V3
- C59 pad 1: GND -> +1V8
- C59 pad 2: +3V3 -> GND
- C6 pad 1: +1V0 -> Net-(C4-Pad1)
- C60 pad 1: +1V8 -> +5V
- C61 pad 1: Net-(C61-Pad1) -> +5V
- C61 pad 2: Net-(C61-Pad2) -> GND
- C62 pad 1: Net-(C62-Pad1) -> GND
- C62 pad 2: Net-(C62-Pad2) -> +1V8
- C63 pad 1: +5V -> Net-(C63-Pad1)
- C63 pad 2: GND -> Net-(C63-Pad2)
- C64 pad 1: +5V -> +3V3
- C65 pad 1: +1V8 -> +3V3
- C66 pad 1: +5V -> Net-(C66-Pad1)
- C66 pad 2: GND -> HDMI_CK_P
- C67 pad 1: +5V -> Net-(C67-Pad1)
- C67 pad 2: GND -> HDMI_D0_P
- C68 pad 1: +3V3 -> Net-(C68-Pad1)
- C68 pad 2: GND -> HDMI_D1_P
- C69 pad 1: +3V3 -> Net-(C69-Pad1)
- C69 pad 2: GND -> HDMI_D2_P
- C70 pad 1: +5V -> Net-(C70-Pad1)
- C70 pad 2: GND -> HDMI_CK_N
- C71 pad 1: /hdmi/5V_HDMI -> Net-(C71-Pad1)
- C71 pad 2: GND -> HDMI_D0_N
- C72 pad 1: +3V3 -> Net-(C72-Pad1)
- C72 pad 2: GND -> HDMI_D1_N
- C73 pad 1: +3V3 -> Net-(C73-Pad1)
- C73 pad 2: GND -> HDMI_D2_N
- C74 pad 1: Net-(C74-Pad1) -> +3V3
- C74 pad 2: HDMI_CK_P -> GND
- C75 pad 1: Net-(C75-Pad1) -> +3V3
- C75 pad 2: HDMI_CK_N -> GND
- C76 pad 1: Net-(C76-Pad1) -> +5V
- C76 pad 2: HDMI_D0_P -> GND
- C77 pad 1: Net-(C77-Pad1) -> /hdmi/5V_HDMI
- C77 pad 2: HDMI_D0_N -> GND
- C9 pad 1: +1V0 -> Net-(C11-Pad1)
- FB1 pad 1: +1V8 -> +1V0
- FB2 pad 2: Net-(C14-Pad1) -> Net-(C11-Pad1)
- FB3 pad 2: Net-(C31-Pad1) -> Net-(C15-Pad1)
- FB4 pad 2: Net-(C33-Pad1) -> Net-(C30-Pad1)
- FB5 pad 1: +1V0 -> +1V8
- FB5 pad 2: Net-(C35-Pad1) -> Net-(C36-Pad1)
- J4 pad 10: FPGA_SCK -> (no net)
- J4 pad 11: /nucleo/IMU_INT_3V3 -> (no net)
- J4 pad 12: FPGA_SO -> GND
- J4 pad 13: /nucleo/IMU_SI_3V3 -> (no net)
- J4 pad 14: FPGA_SI -> (no net)
- J4 pad 15: /nucleo/IMU_SCK_3V3 -> (no net)
- J4 pad 16: FPGA_CS -> CAM_RESET_BAR
- J4 pad 17: /nucleo/IMU_CS_3V3 -> (no net)
- J4 pad 18: FPGA_INT -> (no net)
- J4 pad 19: /nucleo/IMU_SO_3V3 -> HDMI_SCL
- J4 pad 2: SCL_3V3 -> (no net)
- J4 pad 20: FPGA_DONE -> (no net)
- J4 pad 4: SDA_3V3 -> (no net)
- J4 pad 8: GND -> (no net)
- J5 pad 10: (no net) -> FPGA_SCK
- J5 pad 11: (no net) -> /nucleo/IMU_INT_3V3
- J5 pad 12: GND -> FPGA_SO
- J5 pad 13: (no net) -> /nucleo/IMU_SI_3V3
- J5 pad 14: (no net) -> FPGA_SI
- J5 pad 15: (no net) -> /nucleo/IMU_SCK_3V3
- J5 pad 16: /nucleo/CAM_RESET_BAR_3V3 -> FPGA_CS
- J5 pad 17: (no net) -> /nucleo/IMU_CS_3V3
- J5 pad 18: /nucleo/CAM_SHUTTER_3V3 -> FPGA_INT
- J5 pad 19: HDMI_SCL -> /nucleo/IMU_SO_3V3
- J5 pad 2: (no net) -> SCL_3V3
- J5 pad 20: /nucleo/CAM_FLASH_3V3 -> FPGA_DONE
- J5 pad 4: (no net) -> SDA_3V3
- J5 pad 8: (no net) -> GND
- L1 pad 2: Net-(C61-Pad1) -> Net-(C57-Pad1)
- L2 pad 2: Net-(C62-Pad1) -> Net-(C63-Pad1)
- R1 pad 1: +3V3 -> /FPGA/LED1
- R1 pad 2: /FPGA/FLASH_CS -> GND
- R11 pad 2: /FPGA/JTAG_TDO -> /FPGA/FLASH_CS
- R12 pad 1: +3V3 -> /FPGA/FLASH_SCK
- R12 pad 2: /FPGA/JTAG_TMS -> GND
- R13 pad 2: /FPGA/JTAG_RESET -> /FPGA/JTAG_TDO
- R14 pad 2: Net-(DONE1-Pad2) -> /FPGA/JTAG_TMS
- R15 pad 2: FPGA_DONE -> /FPGA/JTAG_RESET
- R17 pad 1: +3V3 -> +1V8
- R17 pad 2: SDA_3V3 -> CAM_RESET_BAR
- R18 pad 1: +3V3 -> +5V
- R18 pad 2: SCL_3V3 -> /nucleo/5V_IN
- R19 pad 1: SCL_1V8 -> +1V8
- R19 pad 2: +1V8 -> Net-(R19-Pad2)
- R20 pad 1: SDA_1V8 -> Net-(R19-Pad2)
- R20 pad 2: +1V8 -> GND
- R21 pad 1: +1V8 -> /nucleo/LED1
- R22 pad 1: +3V3 -> /nucleo/LED2
- R23 pad 1: Net-(R21-Pad2) -> /nucleo/LED3
- R23 pad 2: GND -> Net-(R23-Pad2)
- R24 pad 1: Net-(R22-Pad2) -> +3V3
- R24 pad 2: GND -> Net-(PWR1-Pad2)
- R25 pad 1: +5V -> SDA_1V8
- R25 pad 2: /nucleo/5V_IN -> +1V8
- R26 pad 1: /nucleo/LED1 -> SCL_1V8
- R26 pad 2: Net-(R26-Pad2) -> +1V8
- R27 pad 1: /nucleo/LED2 -> +3V3
- R28 pad 1: /nucleo/LED3 -> Net-(R27-Pad2)
- R28 pad 2: Net-(R28-Pad2) -> GND
- R29 pad 2: Net-(PWR1-Pad2) -> SCL_3V3
- R3 pad 1: +3V3 -> /FPGA/LED2
- R3 pad 2: Net-(FPGA_LED2-Pad2) -> GND
- R30 pad 1: /hdmi/5V_HDMI -> +3V3
- R30 pad 2: Net-(J7-Pad15) -> SDA_3V3
- R31 pad 1: /hdmi/5V_HDMI -> +3V3
- R31 pad 2: Net-(J7-Pad16) -> HDMI_SCL
- R32 pad 2: HDMI_SCL -> HDMI_SDA
- R33 pad 1: +3V3 -> HDMI_OE
- R33 pad 2: HDMI_SDA -> GND
- R38 pad 1: HDMI_OE -> /hdmi/5V_HDMI
- R38 pad 2: GND -> Net-(J7-Pad15)
- R4 pad 2: Net-(FPGA_LED3-Pad2) -> Net-(FPGA_LED2-Pad2)
- R5 pad 1: /FPGA/FLASH_SCK -> /FPGA/LED3
- R6 pad 1: /FPGA/LED1 -> +3V3
- R6 pad 2: GND -> Net-(FPGA_LED3-Pad2)
- R7 pad 1: /FPGA/LED2 -> +3V3
- R7 pad 2: GND -> Net-(R7-Pad2)
- R8 pad 1: /FPGA/LED3 -> +3V3
- R8 pad 2: GND -> FPGA_DONE
- R9 pad 2: Net-(R9-Pad2) -> Net-(DONE1-Pad2)
- STM_LED1 pad 2: Net-(R26-Pad2) -> Net-(R21-Pad2)
- STM_LED2 pad 2: Net-(R27-Pad2) -> Net-(R22-Pad2)
- STM_LED3 pad 2: Net-(R28-Pad2) -> Net-(R23-Pad2)
- U10 pad 1: GND -> SCL_1V8
- U10 pad 2: Net-(C62-Pad1) -> +1V8
- U10 pad 3: +5V -> SDA_1V8
- U10 pad 4: Net-(R22-Pad2) -> IMU_INT
- U10 pad 5: +5V -> IMU_SCK
- U10 pad 6: Net-(C62-Pad2) -> IMU_CS
- U11 pad 1: +1V8 -> +3V3
- U11 pad 10: /nucleo/IMU_SI_3V3 -> /hdmi/CK_N
- U11 pad 11: /nucleo/IMU_SO_3V3 -> /hdmi/D0_P
- U11 pad 12: /nucleo/IMU_CS_3V3 -> /hdmi/D0_N
- U11 pad 13: /nucleo/IMU_SCK_3V3 -> /hdmi/D1_P
- U11 pad 14: +3V3 -> /hdmi/D1_N
- U11 pad 2: IMU_SCK -> HDMI_EQ1
- U11 pad 3: IMU_CS -> (no net)
- U11 pad 4: IMU_SO -> Net-(R37-Pad1)
- U11 pad 5: IMU_SI -> HDMI_HPD
- U11 pad 6: (no net) -> HDMI_SDA
- U11 pad 7: GND -> HDMI_SCL
- U11 pad 8: +1V8 -> HDMI_EQ0
- U11 pad 9: (no net) -> /hdmi/CK_P
- U12 pad 1: /nucleo/5V_IN -> GND
- U12 pad 2: +5V -> /hdmi/5V_HDMI
- U12 pad 3: GND -> +5V
- U2 pad 17: Net-(C14-Pad1) -> Net-(C30-Pad1)
- U2 pad 29: Net-(C14-Pad1) -> Net-(C30-Pad1)
- U2 pad 47: Net-(C14-Pad1) -> Net-(C30-Pad1)
- U2 pad 50: Net-(R9-Pad2) -> Net-(R7-Pad2)
- U2 pad 63: Net-(C31-Pad1) -> Net-(C4-Pad1)
- U2 pad 7: Net-(C14-Pad1) -> Net-(C30-Pad1)
- U2 pad 70: Net-(C35-Pad1) -> Net-(C15-Pad1)
- U2 pad 71: Net-(C33-Pad1) -> Net-(C11-Pad1)
- U2 pad 72: Net-(C35-Pad1) -> Net-(C15-Pad1)
- U5 pad 3: CAM_FLASH -> (no net)
- U5 pad 35: CAM_SHUTTER -> (no net)
- U7 pad 1: +1V8 -> GND
- U7 pad 2: SCL_1V8 -> Net-(C57-Pad1)
- U7 pad 3: SDA_1V8 -> +5V
- U7 pad 4: IMU_INT -> Net-(R19-Pad2)
- U7 pad 5: GND -> +5V
- U7 pad 6: (no net) -> Net-(C57-Pad2)
- U8 pad 1: +1V8 -> /nucleo/5V_IN
- U8 pad 2: CAM_RESET_BAR -> +5V
- U8 pad 3: CAM_SHUTTER -> GND
- U8 pad 4: CAM_FLASH -> +3V3
- U8 pad 5: CAM_TRIGGER -> SCL_3V3
- U8 pad 6: (no net) -> SDA_3V3
- U8 pad 8: +1V8 -> GND
- U9 pad 2: Net-(C61-Pad1) -> Net-(C63-Pad1)
- U9 pad 4: Net-(R21-Pad2) -> Net-(R27-Pad2)
- U9 pad 6: Net-(C61-Pad2) -> Net-(C63-Pad2)
- X1 pad 4: Net-(C4-Pad1) -> Net-(C36-Pad1)
Routing:
- net GND: track 0.06 -> 0.00 mm, vias 19 -> 0
Other:
- outline, holes or cut-outs redrawn
